File: PROJ/SPAR/18159/STAN/01/src/eagleBoard.brd (EAGLE design)
At the start: 74.9 x 73.7 mm, 327 parts, among them J1 VDC-IN, J10 TRIG2, J11 TRIG1, J14 AUDIO I/O, J15 MIDI, J16 USB-C, J17 AGND, J2 GND-IN, J3 DEBUG, J4 QWIIC, J6 3.3VA, J7 3.3V, J8 PLAYING, J9 CORTEX_JTAG_DEBUG_PTH_NS, Q1 3.1A/30V/105mΩ, U1 LM1117, U3 ATSAMS70N20A-AN, U4 LMV324, U5 LM1117, U6 6N138M, U7 ADAU1328, U8 74AHC1G125W5-7, Y1 11.2896 MHz

Commit message: Added projects.
Parts:
- U3: value ATSAMS70N20A-AN -> ATSAMS70NXXA-AN
Changed lines of the file:
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@@
 <drawing>
 <settings>
-<setting alwaysvectorfont="no"/>
+<setting alwaysvectorfont="yes"/>
 <setting keepoldvectorfont="yes"/>
 <setting verticaltext="up"/>
@@
 <layer number="98" name="Guide" color="6" fill="1" visible="no" active="no"/>
 <layer number="99" name="SpiceOrder" color="7" fill="1" visible="no" active="no"/>
-<layer number="100" name="Muster" color="7" fill="1" visible="no" active="yes"/>
+<layer number="100" name="Muster" color="7" fill="1" visible="yes" active="yes"/>
 <layer number="101" name="Patch_Top" color="12" fill="4" visible="no" active="yes"/>
 <layer number="102" name="Vscore" color="7" fill="1" visible="no" active="yes"/>
@@
 </autorouter>
 <elements>
-<element name="U3" library="SparkFun-IC-Microcontroller" package="LQFP100" value="ATSAMS70N20A-AN" x="26.67" y="20.32" smashed="yes" rot="R270">
+<element name="U3" library="SparkFun-IC-Microcontroller" package="LQFP100" value="ATSAMS70NXXA-AN" x="26.67" y="20.32" smashed="yes" rot="R270">
 <attribute name="NAME" x="35.7901" y="26.715" size="1.27" layer="25" rot="R270"/>
 <attribute name="PROD_ID" value="IC-13238" x="26.67" y="20.32" size="1.778" layer="27" rot="R270" display="off"/>
