File: PROJ/ADAF/3463/STAN/01/src/kicadBoard.kicad_sch (KiCad schematic)
At the start: 29 parts

Commit message: Quickly Adding Everything
Parts:
- removed C1, C2, C3, C4, C5, C6, C7: (no value), symbol eagleSchem-eagle-import:CAP_CERAMIC0805-NOOUTLINE
- removed D1: (no value), symbol eagleSchem-eagle-import:DIODESOD-323
- removed FID1, FID2, FID3: (no value), symbol eagleSchem-eagle-import:FIDUCIAL_1MM
- removed JP1: (no value), symbol eagleSchem-eagle-import:HEADER-1X670MIL
- removed JP2: (no value), symbol eagleSchem-eagle-import:HEADER-1X4ROUND
- removed Q1, Q2, Q3: (no value), symbol eagleSchem-eagle-import:MOSFET-NWIDE
- removed R1, R2, R3, R4, R5, R6: (no value), symbol eagleSchem-eagle-import:RESISTOR0805_NOOUTLINE
- removed U$1, U$2, U$3, U$4: (no value), symbol eagleSchem-eagle-import:MOUNTINGHOLE2.5
- removed U1: (no value), symbol eagleSchem-eagle-import:VREG_SOT23-5
- removed U2: (no value), symbol eagleSchem-eagle-import:ACCEL_MAG_FXOS8700CQ
- removed U4: (no value), symbol eagleSchem-eagle-import:GYRO_FXAS21002C
- added C1, C2, C3, C4, C5, C6, C7: (no value), symbol schematicEagle-eagle-import:CAP_CERAMIC0805-NOOUTLINE
- added D1: (no value), symbol schematicEagle-eagle-import:DIODESOD-323
- added FID1, FID2, FID3: (no value), symbol schematicEagle-eagle-import:FIDUCIAL_1MM
- added JP1: (no value), symbol schematicEagle-eagle-import:HEADER-1X670MIL
- added JP2: (no value), symbol schematicEagle-eagle-import:HEADER-1X4ROUND
- added Q1, Q2, Q3: (no value), symbol schematicEagle-eagle-import:MOSFET-NWIDE
- added R1, R2, R3, R4, R5, R6: (no value), symbol schematicEagle-eagle-import:RESISTOR0805_NOOUTLINE
- added U$1, U$2, U$3, U$4: (no value), symbol schematicEagle-eagle-import:MOUNTINGHOLE2.5
- added U1: (no value), symbol schematicEagle-eagle-import:VREG_SOT23-5
- added U2: (no value), symbol schematicEagle-eagle-import:ACCEL_MAG_FXOS8700CQ
- added U4: (no value), symbol schematicEagle-eagle-import:GYRO_FXAS21002C
Connections:
- net 3.3V: now also C3.1, C4.1, C6.1, JP1.5, Q1.1 (G), Q2.1 (G), R1.2, R2.2, R5.1, R6.2, U1.5 (OUT), U2.1 (VDDIO), U2.10 (SA1/CS), U2.14 (VDD), U2.7 (SA0/MISO), U4.13 (SA0/MISO), U4.15 (VDD), U4.17 (SPI_CS), U4.18 (VDDIO)
- net ACC_RST: now also Q3.3 (D), R5.2, U2.16 (RST)
- net AINT1: now also JP2.3, U2.11 (INT1)
- net AINT2: now also JP2.4, U2.9 (INT2)
- net GINT1: now also JP2.1, U4.3 (INT1)
- net GINT2: now also JP2.2, U4.2 (INT2)
- net GND: now also C1.2, C2.2, C3.2, C4.2, C5.2, C6.2, C7.2, JP1.4, Q3.2 (S), U1.2 (GND), U2.12 (GND), U2.13 (RESERVED), U2.3 (RESERVED), U2.5 (GND), U4.1 (GND), U4.10 (RSVD(GND)), U4.14 (GND), U4.19 (GND), U4.20 (RSVD(GND)), U4.21 (RSVD(GND)), U4.22 (RSVD(GND)), U4.23 (RSVD(GND)), U4.24 (RSVD(GND)), U4.5 (GND), U4.6 (RSVD(GND)), U4.7 (RSVD(GND)), U4.8 (I2C/SPI), U4.9 (RSVD(GND))
- net RST: now also D1.C, JP1.1
- net RST_3V: now also D1.A, Q3.1 (G), R6.1, U4.4 (RST)
- net SCL: now also JP1.3, Q2.3 (D), R4.1
- net SCL_3V: now also Q2.2 (S), R2.1, U2.4 (SCL/SCLK), U4.11 (SCL/SCLK)
- net SDA: now also JP1.2, Q1.3 (D), R3.1
- net SDA_3V: now also Q1.2 (S), R1.1, U2.6 (SDA/MOSI), U4.12 (SDA/MOSI/SPI_DATA)
- net VIN: now also C1.1, JP1.6, R3.2, R4.2, U1.1 (IN), U1.3 (EN)
- new net: C5.1, U2.2 (BYP)
- new net: C7.1, U2.8 (CRST)
- new net: C2.1, U4.16 (VREGD)
