File: PROJ/ADAF/3660/STAN/01/src/kicadBoard.kicad_sch (KiCad schematic)
At the start: 14 parts

Commit message: Quickly Adding Everything
Parts:
- removed C1, C3: (no value), symbol eagleSchem-eagle-import:CAP_CERAMIC0805-NOOUTLINE
- removed D2: (no value), symbol eagleSchem-eagle-import:DIODESOD-323
- removed JP2: (no value), symbol eagleSchem-eagle-import:HEADER-1X770MIL
- removed Q1: (no value), symbol eagleSchem-eagle-import:MOSFET-N_DUAL
- removed R1, R4: (no value), symbol eagleSchem-eagle-import:RESISTOR_0603_NOOUT
- removed R3: (no value), symbol eagleSchem-eagle-import:RESISTOR_4PACK
- removed U$15, U$5: (no value), symbol eagleSchem-eagle-import:FIDUCIAL_1MM
- removed U$7, U$8: (no value), symbol eagleSchem-eagle-import:MOUNTINGHOLE2.0
- removed U1: (no value), symbol eagleSchem-eagle-import:BME680
- removed U2: (no value), symbol eagleSchem-eagle-import:VREG_SOT23-5
- added C1: (no value), symbol schematicEagle-eagle-import:CAP_CERAMIC0603_NO
- added C2, C3: (no value), symbol schematicEagle-eagle-import:CAP_CERAMIC0805-NOOUTLINE
- added CONN3, CONN4: (no value), symbol schematicEagle-eagle-import:STEMMA_I2C_QT
- added D1: (no value), symbol schematicEagle-eagle-import:LED0603_NOOUTLINE
- added D2: (no value), symbol schematicEagle-eagle-import:DIODESOD-323
- added FID3, FID4: (no value), symbol schematicEagle-eagle-import:FIDUCIAL_1MM
- added IC1: (no value), symbol schematicEagle-eagle-import:BME680
- added JP1: (no value), symbol schematicEagle-eagle-import:HEADER-1X770MIL
- added Q2: (no value), symbol schematicEagle-eagle-import:MOSFET-N_DUAL
- added R1, R4, R5: (no value), symbol schematicEagle-eagle-import:RESISTOR_0603_NOOUT
- added R3: (no value), symbol schematicEagle-eagle-import:RESISTOR_4PACK
- added SJ1: (no value), symbol schematicEagle-eagle-import:SOLDERJUMPER
- added U$1, U$17: (no value), symbol schematicEagle-eagle-import:MOUNTINGHOLE2.5
- added U2: (no value), symbol schematicEagle-eagle-import:VREG_SOT23-5
Connections:
- net 3.3V: now also C1.1, C3.1, IC1.6 (VDDIO), IC1.8 (VDD), JP1.2, Q2.2 (G), Q2.5 (G), R1.1, R3.2 (1), R3.4 (1), R4.2, R5.2, U2.5 (OUT)
- net CS: now also D2.C, JP1.7
- net CS_3V: now also D2.A, IC1.2 (CSB), R5.1
- net GND: now also C1.2, C2.2, C3.2, CONN3.1 (GND), CONN4.1 (GND), D1.C, IC1.1 (GND), IC1.7 (GND), JP1.3, SJ1.2, U2.2 (GND)
- net SCK/SCL: now also CONN3.4 (SCL), CONN4.4 (SCL), JP1.4, Q2.6 (D), R3.8 (2)
- net SCK_3V: now also IC1.4 (SCK), Q2.1 (S), R3.7 (2)
- net SDI/SDA: now also CONN3.3 (SDA), CONN4.3 (SDA), JP1.6, Q2.3 (D), R3.6 (2)
- net SDI_3V: now also IC1.3 (SDI), Q2.4 (S), R3.5 (2)
- net SDO/ADR: now also IC1.5 (SDO), JP1.5, R4.1, SJ1.1
- new net: D1.A, R1.2
- new net VCC: C2.1, CONN3.2 (V+), CONN4.2 (V+), JP1.1, R3.1, R3.3 (1), U2.1 (IN), U2.3 (EN)
Other:
- note added: "I2C Pullups"
- note added: "I2C Pullups & Shift"
- note added: "ON LED"
- note added: "Power supply"
- note added: "STEMMA/I2C Headers"
- note removed: "For I2C leave CSB pulled high (default value) SDI=SDA, SCK=SCL"
- note removed: "For SPI set CSB low at startup SDO=MISO, SDI=MOSI, SCK=SCK, CSB=CS/SSEL"
- note removed: "LEVEL SHIFTING (5V <--> 3V)"
