File: PROJ/ADAF/3900/STAN/01/src/kicadBoard.kicad_sch (KiCad schematic)
At the start: 65 parts

Commit message: Quickly Adding Everything
Parts:
- removed C1, C13, C14, C2, C4, C7, C9: (no value), symbol eagleSchem-eagle-import:CAP_CERAMIC0603_NO
- removed C10, C15, C3, C5, C6: (no value), symbol eagleSchem-eagle-import:CAP_CERAMIC0805-NOOUTLINE
- removed C11, C8: (no value), symbol eagleSchem-eagle-import:CAP_CERAMIC0805_10MGAP
- removed CHG0, L0: (no value), symbol eagleSchem-eagle-import:LED0805_NOOUTLINE
- removed D1, D2: (no value), symbol eagleSchem-eagle-import:DIODE-ZENERSOD323
- removed D4: (no value), symbol eagleSchem-eagle-import:DIODE-SCHOTTKYSOD-123
- removed I2C0: (no value), symbol eagleSchem-eagle-import:STEMMA_I2C_RASMT
- removed IC4: (no value), symbol eagleSchem-eagle-import:ACCEL_LIS3DHTR
- removed LED1: (no value), symbol eagleSchem-eagle-import:WS2812B3535
- removed MS1: (no value), symbol eagleSchem-eagle-import:FEATHERWING_SMTDUALNOHOLES
- removed NEOPIXEL0, PIR0: (no value), symbol eagleSchem-eagle-import:CON_JST_PH_3PIN
- removed Q1, Q2: (no value), symbol eagleSchem-eagle-import:MOSFET-P
- removed Q3: (no value), symbol eagleSchem-eagle-import:MOSFET-NWIDE
- removed R1, R4, R9: (no value), symbol eagleSchem-eagle-import:RESISTOR_4PACK
- removed R12, R13, R2, R3, R5, R6, R7, R8: (no value), symbol eagleSchem-eagle-import:RESISTOR_0603_NOOUT
- removed SJ1: (no value), symbol eagleSchem-eagle-import:SOLDERJUMPER_2WAY
- removed SW1: (no value), symbol eagleSchem-eagle-import:SPST_TACT-KMR2
- removed SW2: (no value), symbol eagleSchem-eagle-import:SWITCH_DPDTEG1390
- removed TFT0: (no value), symbol eagleSchem-eagle-import:DISP_LCD_ST7735_1.44IN
- removed TP1, TP2, TP5: (no value), symbol eagleSchem-eagle-import:TESTPOINTROUND1.5MM
- removed TP28, TP4: (no value), symbol eagleSchem-eagle-import:SEWTAPPCB_ALLIGATOR
- removed TP29, TP3: (no value), symbol eagleSchem-eagle-import:SEWTAP_ALLILONG
- removed U$13: (no value), symbol eagleSchem-eagle-import:CON_MOLEX_2P
- removed U$31, U$32: (no value), symbol eagleSchem-eagle-import:MOUNTINGHOLE2.5
- removed U$34, U$35: (no value), symbol eagleSchem-eagle-import:FIDUCIAL_1MM
- removed U$4: (no value), symbol eagleSchem-eagle-import:ATSAMD21G_QFN
- removed U1: (no value), symbol eagleSchem-eagle-import:SPIFLASH_8PIN208MIL
- removed U2: (no value), symbol eagleSchem-eagle-import:VREG_SOT23-5
- removed U3: (no value), symbol eagleSchem-eagle-import:MCP73831/2
- removed U4: (no value), symbol eagleSchem-eagle-import:PHOTOTRANSISTOR_PT26-21C
- removed U5: (no value), symbol eagleSchem-eagle-import:AUDIOAMP_PAM8302A
- removed VR2: (no value), symbol eagleSchem-eagle-import:TRIMPOT3303W/X
- removed X1: (no value), symbol eagleSchem-eagle-import:CON_JST_PH_2PIN
- removed X3: (no value), symbol eagleSchem-eagle-import:USB_MICRO_20329_V2
- removed X6: (no value), symbol eagleSchem-eagle-import:CON_JST_PH_2PIN_MTPH2
- added C1, C13, C14, C2, C4, C7, C9: (no value), symbol schematicEagle-eagle-import:CAP_CERAMIC0603_NO
- added C10, C15, C3, C5, C6: (no value), symbol schematicEagle-eagle-import:CAP_CERAMIC0805-NOOUTLINE
- added C11, C8: (no value), symbol schematicEagle-eagle-import:CAP_CERAMIC0805_10MGAP
- added CHG0, L0: (no value), symbol schematicEagle-eagle-import:LED0805_NOOUTLINE
- added D1, D2: (no value), symbol schematicEagle-eagle-import:DIODE-ZENERSOD323
- added D4: (no value), symbol schematicEagle-eagle-import:DIODE-SCHOTTKYSOD-123
- added I2C0: (no value), symbol schematicEagle-eagle-import:STEMMA_I2C_RASMT
- added IC4: (no value), symbol schematicEagle-eagle-import:ACCEL_LIS3DHTR
- added LED1: (no value), symbol schematicEagle-eagle-import:WS2812B3535
- added MS1: (no value), symbol schematicEagle-eagle-import:FEATHERWING_SMTDUALNOHOLES
- added NEOPIXEL0, PIR0: (no value), symbol schematicEagle-eagle-import:CON_JST_PH_3PIN
- added Q1, Q2: (no value), symbol schematicEagle-eagle-import:MOSFET-P
- added Q3: (no value), symbol schematicEagle-eagle-import:MOSFET-NWIDE
- added R1, R4, R9: (no value), symbol schematicEagle-eagle-import:RESISTOR_4PACK
- added R12, R13, R2, R3, R5, R6, R7, R8: (no value), symbol schematicEagle-eagle-import:RESISTOR_0603_NOOUT
- added SJ1: (no value), symbol schematicEagle-eagle-import:SOLDERJUMPER_2WAY
- added SW1: (no value), symbol schematicEagle-eagle-import:SPST_TACT-KMR2
- added SW2: (no value), symbol schematicEagle-eagle-import:SWITCH_DPDTEG1390
- added TFT0: (no value), symbol schematicEagle-eagle-import:DISP_LCD_ST7735_1.44IN
- added TP1, TP2, TP5: (no value), symbol schematicEagle-eagle-import:TESTPOINTROUND1.5MM
- added TP28, TP4: (no value), symbol schematicEagle-eagle-import:SEWTAPPCB_ALLIGATOR
- added TP29, TP3: (no value), symbol schematicEagle-eagle-import:SEWTAP_ALLILONG
- added U$13: (no value), symbol schematicEagle-eagle-import:CON_MOLEX_2P
- added U$31, U$32: (no value), symbol schematicEagle-eagle-import:MOUNTINGHOLE2.5
- added U$34, U$35: (no value), symbol schematicEagle-eagle-import:FIDUCIAL_1MM
- added U$4: (no value), symbol schematicEagle-eagle-import:ATSAMD21G_QFN
- added U1: (no value), symbol schematicEagle-eagle-import:SPIFLASH_8PIN208MIL
- added U2: (no value), symbol schematicEagle-eagle-import:VREG_SOT23-5
- added U3: (no value), symbol schematicEagle-eagle-import:MCP73831/2
- added U4: (no value), symbol schematicEagle-eagle-import:PHOTOTRANSISTOR_PT26-21C
- added U5: (no value), symbol schematicEagle-eagle-import:AUDIOAMP_PAM8302A
- added VR2: (no value), symbol schematicEagle-eagle-import:TRIMPOT3303W/X
- added X1: (no value), symbol schematicEagle-eagle-import:CON_JST_PH_2PIN
- added X3: (no value), symbol schematicEagle-eagle-import:USB_MICRO_20329_V2
- added X6: (no value), symbol schematicEagle-eagle-import:CON_JST_PH_2PIN_MTPH2
Connections:
- net +3V3: now also C11.1, C2.1, C4.1, C5.1, C7.1, C8.1, IC4.1 (VDDIO), IC4.13 (ADC3), IC4.14 (VDD), IC4.15 (ADC2), IC4.16 (ADC1), IC4.8 (CS), LED1.2 (VDD), MS1.2 (3V), MS1.2' (3V), R4.3 (1), R4.5 (2), R4.6 (2), R4.7 (2), R4.8 (2), R9.1, R9.2 (1), R9.4 (1), R9.8 (2), SJ1.3, TFT0.10 (VCC), TFT0.11 (VCC@1), TFT0.4 (LEDA), U$4.17 (VDDIO), U$4.36 (VDDIO), U$4.44 (VDDIN), U$4.6 (VDDA), U1.3 (WP#/IO2), U1.7 (HOLD#/IO3), U1.8 (VCC), U2.5 (OUT), U4.2_C (C)
- net A0: now also MS1.5 (GPIOA0), MS1.5' (GPIOA0), U$4.3 (PA02/EINT2/AIN0/Y0/VOUT), VR2.3 (E)
- net A1: now also MS1.6 (GPIOA1), MS1.6' (GPIOA1), R3.2, U$4.7 (PB08/I8/AIN2/SERCOM4.0), U4.1_E (E)
- net A2: now also MS1.7 (GPIOA2), MS1.7' (GPIOA2), TP3.P$1 (SEW), U$4.8 (PB09/I9/AIN3/SERCOM4.1)
- net A3: now also MS1.8 (GPIOA3), MS1.8' (GPIOA3), TP4.P$1 (SEW), U$4.9 (PA04/EINT4/VREFB/AIN4/SERCOM0.0)
- net A4: now also MS1.9 (GPIOA4), MS1.9' (GPIOA4), TP28.P$1 (SEW), U$4.10 (PA05/EINT5/AIN5/SERCOM0.1)
- net A5: now also MS1.10 (GPIOA5), MS1.10' (GPIOA5), TP29.P$1 (SEW), U$4.11 (PA06/EINT6/AIN6/SERCOM0.2)
- net AREF: now also C14.1, MS1.3 (AREF), MS1.3' (AREF), U$4.4 (PA03/EINT3/VREFA/AIN1)
- net BACKLITE: now also Q3.1 (G), R9.6 (2), U$4.1 (PA00/EINT0/SERCOM1.0)
- net D+: now also U$4.34 (PA25/I13/SERCOM3+5.3/D+), X3.D+
- net D-: now also U$4.33 (PA24/I12/SERCOM3+5.2/D-), X3.D-
- net D10: now also MS1.22 (GPIO10), MS1.22' (GPIO10), U$4.29 (PA20/I4/SERCOM3+5.2/I2SSC)
- net D11: now also MS1.23 (GPIO11), MS1.23' (GPIO11), U$4.30 (PA21/I5/SERCOM3+5.3/I2SFS0)
- net D12: now also MS1.24 (GPIO12), MS1.24' (GPIO12), U$4.31 (PA22/I2C/I6/SERCOM3+5.0)
- net D13: now also MS1.25 (GPIO13), MS1.25' (GPIO13), R7.1, U$4.32 (PA23/I2C/I7/SERCOM3+5.1/SOF)
- net D2: now also IC4.11 (INT1), U$4.23 (PA14/I14/SERCOM2+4.2)
- net D3: now also D2.C, R6.2, U$4.16 (PA11/I11/AIN19/SERCOM0+2.3/I2SF0)
- net D4: now also D1.C, R5.2, U$4.13 (PA08/I2C/AIN16/SERCOM0+2.0/I2SD1)
- net D5: now also MS1.19 (GPIO5), MS1.19' (GPIO5), U$4.24 (PA15/I15/SERCOM2+4.3)
- net D6: now also MS1.20 (GPIO6), MS1.20' (GPIO6), U$4.27 (PA18/I2/SERCOM1+3.2)
- net D8_NEOPIX: now also LED1.1 (DI), U$4.21 (PA12/I12/I2C/SERCOM2+4.0)
- net D9: now also MS1.21 (GPIO9), MS1.21' (GPIO9), U$4.28 (PA19/I3/SERCOM1+3.3/I2SD0)
- net EN: now also MS1.27 (EN), MS1.27' (EN), R1.4 (1), SW2.P1, U2.3 (EN)
- net FLASHMISO: now also U$4.22 (PA13/I13/I2C/SERCOM2+4.1), U1.2 (MISO)
- net FLASHMOSI: now also U$4.19 (PB10/I10/SERCOM4.2/I2SMC), U1.5 (MOSI)
- net FLASHSCK: now also U$4.20 (PB11/I11/SERCOM4.3/I2SCL), U1.6 (SCK)
- net FLASH_CS: now also R4.2 (1), U$4.12 (PA07/I7/AIN7/SERCOM0.3/I2SD0), U1.1 (SSEL)
- net GND: now also C1.2, C10.2, C11.2, C14.2, C15.2, C2.2, C3.2, C4.2, C5.2, C6.2, C7.2, C8.2, C9.2, D1.A, D2.A, I2C0.1 (GND), I2C0.NC1 (MT), I2C0.NC2 (MT), IC4.10 (RES(GND)), IC4.12 (GND@2), IC4.5 (GND@1), IC4.7 (SDO), L0.C, LED1.4 (GND), MS1.16 (NC), MS1.16' (NC), MS1.4 (GND), MS1.4' (GND), NEOPIXEL0.1, PIR0.1, Q3.2 (S), R1.6 (2), R1.7 (2), R3.1, R8.2, R9.3 (1), SW1.2 (S), SW1.4 (S1), SW2.O2, SW2.S1, TFT0.1 (GND), TFT0.13 (GND@3), TFT0.14 (GND@4), TFT0.2 (GND@1), TFT0.5 (GND@2), U$4.18 (GND), U$4.35 (GND), U$4.42 (GND), U$4.5 (GNDA), U$4.THERMAL (GND), U1.4 (VSS), U2.2 (GND), U3.2 (VSS), U5.7 (GND), VR2.1 (A), X1.1, X3.BASE@1 (GND), X3.BASE@2 (GND), X3.GND, X3.SPRT@1 (GND), X3.SPRT@2 (GND), X3.SPRT@3 (GND), X3.SPRT@4 (GND)
- net MISO: now also MS1.13 (GPIOMISO), MS1.13' (GPIOMISO), U$4.48 (PB03/I3/AIN11/SERCOM5.1)
- net MOSI: now also MS1.12 (GPIOMOSI), MS1.12' (GPIOMOSI), TFT0.8 (DATA), U$4.37 (PB22/I6/SERCOM5.2)
- net ON/OFF: now also Q2.1 (G), SW2.P2
- net RX: now also MS1.14 (GPIORX), MS1.14' (GPIORX), U$4.14 (PA09/I2C/I9/AIN17/SERCOM0+2.1/I2SMC)
- net SCK: now also MS1.11 (GPIOSCK), MS1.11' (GPIOSCK), TFT0.9 (CLOCK), U$4.38 (PB23/I7/SERCOM5.3)
- net SCL: now also I2C0.4 (SCL), IC4.4 (SCL), MS1.18 (GPIOSCL), MS1.18' (GPIOSCL), R4.4 (1), U$4.26 (PA17/I2C/I1/SERCOM1+3.1)
- net SDA: now also I2C0.3 (SDA), IC4.6 (SDA), MS1.17 (GPIOSDA), MS1.17' (GPIOSDA), R4.1, U$4.25 (PA16/I2C/I0/SERCOM1+3.0)
- net SPKR+: now also U$13.1, U5.5 (VO_P), X6.2
- net SPKR-: now also U$13.2, U5.8 (VO_N), X6.1
- net SWCLK: now also R9.7 (2), TP1.P$1, U$4.45 (PA30/I10/SECOM1.2/SWCLK)
- net SWDIO: now also TP2.P$1, U$4.46 (PA31/I11/SECOM1.3/SWDIO)
- net TFT_CS: now also R9.5 (2), TFT0.12 (CS), U$4.2 (PA01/EINT1/SERCOM1.1)
- net TFT_DC: now also TFT0.7 (RS/DC), U$4.41 (PA28/I8)
- net TFT_RESET: now also TFT0.6 (RESET), U$4.39 (PA27/I15)
- net TX: now also MS1.15 (GPIOTX), MS1.15' (GPIOTX), U$4.15 (PA10/I10/AIN18/SERCOM0+2.2/I2SCK)
- net V+: now also C15.1, C6.1, PIR0.2, Q2.3 (D), R1.5 (2), SJ1.1, U2.1 (IN), U5.1 (/SD), U5.6 (VDD)
- net VBAT: now also C3.1, MS1.28 (VBAT), MS1.28' (VBAT), Q1.3 (D), R1.8 (2), U3.3 (VBAT), X1.2
- net VBATT: now also R1.1, R1.2 (1), U$4.47 (PB02/I2/AIN10/SERCOM5.0)
- net VBUS: now also CHG0.A, D4.A, MS1.26 (USB), MS1.26' (USB), Q1.1 (G), R1.3 (1), U3.4 (VDD), X3.VBUS
- net VCC: now also C10.1, I2C0.2 (V+), NEOPIXEL0.2, SJ1.2
- net ~{RESET}: now also MS1.1 (~{RESET}), MS1.1' (~{RESET}), SW1.1 (P), SW1.3 (P1), TP5.P$1, U$4.40 (/RESET)
- new net: Q3.3 (D), TFT0.3 (LEDK)
- new net: D4.C, Q1.2 (S), Q2.2 (S), SW2.S2
- new net: L0.A, R7.2
- new net: C9.1, R12.1
- new net: R12.2, U5.4 (IN_N)
- new net: C1.1, U$4.43 (VDDCORE)
- new net: NEOPIXEL0.3, R6.1
- new net: C13.1, R13.1
- new net: C13.2, VR2.2 (S)
- new net: R8.1, U3.5 (PROG)
- new net: R2.2, U3.1 (STAT)
- new net: PIR0.3, R5.1
- new net: R13.2, U5.3 (IN_P)
- new net: CHG0.C, R2.1
