File: PROJ/ADAF/4383/STAN/01/src/kicadBoard.kicad_sch (KiCad schematic)
At the start: 18 parts

Commit message: Quickly Adding Everything
Parts:
- removed C1, C2, C3: (no value), symbol eagleSchem-eagle-import:CAP_CERAMIC0805-NOOUTLINE
- removed CN1: (no value), symbol eagleSchem-eagle-import:MICROSD
- removed DISP1: (no value), symbol eagleSchem-eagle-import:DISP_LCD_GENERIC_SPI_1.14IN_240X135_WRAPUNDER
- removed FID1, FID2: (no value), symbol eagleSchem-eagle-import:FIDUCIAL_1MM
- removed IC5: (no value), symbol eagleSchem-eagle-import:AXP083-SAG
- removed JP1: (no value), symbol eagleSchem-eagle-import:HEADER-1X11
- removed Q1: (no value), symbol eagleSchem-eagle-import:TRANSISTOR_NPNWIDE
- removed R2, R5, R7, R8: (no value), symbol eagleSchem-eagle-import:RESISTOR_0603_NOOUT
- removed U$10, U$9: (no value), symbol eagleSchem-eagle-import:MOUNTINGHOLE2.5
- removed U2: (no value), symbol eagleSchem-eagle-import:VREG_SOT23-5
- removed U3: (no value), symbol eagleSchem-eagle-import:74HC4050D
- added C1, C2, C3: (no value), symbol schematicEagle-eagle-import:CAP_CERAMIC0805-NOOUTLINE
- added CN1: (no value), symbol schematicEagle-eagle-import:MICROSD
- added DISP1: (no value), symbol schematicEagle-eagle-import:DISP_LCD_GENERIC_SPI_1.14IN_240X135_WRAPUNDER
- added FID1, FID2: (no value), symbol schematicEagle-eagle-import:FIDUCIAL_1MM
- added IC5: (no value), symbol schematicEagle-eagle-import:AXP083-SAG
- added JP1: (no value), symbol schematicEagle-eagle-import:HEADER-1X11
- added Q1: (no value), symbol schematicEagle-eagle-import:TRANSISTOR_NPNWIDE
- added R2, R5, R7, R8: (no value), symbol schematicEagle-eagle-import:RESISTOR_0603_NOOUT
- added U$10, U$9: (no value), symbol schematicEagle-eagle-import:MOUNTINGHOLE2.5
- added U2: (no value), symbol schematicEagle-eagle-import:VREG_SOT23-5
- added U3: (no value), symbol schematicEagle-eagle-import:74HC4050D
Connections:
- net 3.3V: now also C1.1, C3.1, CN1.4 (SD_VDD), DISP1.10 (VDD), DISP1.12 (LEDA), IC5.3 (VCC), JP1.2, R2.2, R8.2, U2.5 (OUT), U3.1 (VCC)
- net BACKLIGHT: now also JP1.11, R7.1, R8.1
- net DC: now also JP1.9, U3.14 (6A)
- net DC_3V: now also DISP1.5 (RS/DC), U3.15 (6Y)
- net GND: now also C1.2, C2.2, C3.2, CN1.6 (GND@3), CN1.MT1 (GND@2), CN1.MT2 (GND@1), DISP1.13 (GND), DISP1.8 (GND), IC5.1 (GND), JP1.3, Q1.2 (E), U2.2 (GND), U3.8 (GND)
- net LED_K: now also DISP1.11 (LEDK), R5.2
- net MISO_3V: now also CN1.7 (DATA_OUT), JP1.5
- net MOSI: now also JP1.6, U3.7 (3A)
- net MOSI_3V: now also CN1.3 (DATA_IN), DISP1.3 (DATA), U3.6 (3Y)
- net SCK: now also JP1.4, U3.5 (2A)
- net SCK_3V: now also CN1.5 (SCLK), DISP1.4 (CLOCK), U3.4 (2Y)
- net SDCS: now also JP1.10, U3.9 (4A)
- net SDCS_3V: now also CN1.2 (CS), U3.10 (4Y)
- net TFTCS: now also JP1.7, U3.3 (1A)
- net TFTCS_3V: now also DISP1.7 (CS), U3.2 (1Y)
- net VIN: now also C2.1, JP1.1, U2.1 (IN), U2.3 (EN)
- net ~{TFTRST_3V}: now also DISP1.6 (RESET), U3.12 (5Y)
- net ~{TFTRST}: now also IC5.2 (/RESET), JP1.8, R2.1, U3.11 (5A)
- new net: Q1.1 (B), R7.2
- new net: Q1.3 (C), R5.1
