File: PROJ/ADAF/4756/STAN/01/src/kicadBoard.kicad_sch (KiCad schematic)
At the start: 14 parts

Commit message: Quickly Adding Everything
Parts:
- removed C1: (no value), symbol eagleSchem-eagle-import:CAP_CERAMIC0603_NO
- removed C3: (no value), symbol eagleSchem-eagle-import:CAP_CERAMIC0805-NOOUTLINE
- removed CONN3, CONN4: (no value), symbol eagleSchem-eagle-import:STEMMA_I2C_QT
- removed D1: (no value), symbol eagleSchem-eagle-import:LED0603_NOOUTLINE
- removed FID3, FID4: (no value), symbol eagleSchem-eagle-import:FIDUCIAL_1MM
- removed IC1: (no value), symbol eagleSchem-eagle-import:LTC4311_SC70
- removed JP2: (no value), symbol eagleSchem-eagle-import:HEADER-1X570MIL
- removed R3: (no value), symbol eagleSchem-eagle-import:RESISTOR_4PACK
- removed U$1, U$17, U$19, U$21: (no value), symbol eagleSchem-eagle-import:MOUNTINGHOLE2.5
- added C1: (no value), symbol schematicEagle-eagle-import:CAP_CERAMIC0603_NO
- added C3: (no value), symbol schematicEagle-eagle-import:CAP_CERAMIC0805-NOOUTLINE
- added CONN3, CONN4: (no value), symbol schematicEagle-eagle-import:STEMMA_I2C_QT
- added D1: (no value), symbol schematicEagle-eagle-import:LED0603_NOOUTLINE
- added FID3, FID4: (no value), symbol schematicEagle-eagle-import:FIDUCIAL_1MM
- added IC1: (no value), symbol schematicEagle-eagle-import:LTC4311_SC70
- added JP2: (no value), symbol schematicEagle-eagle-import:HEADER-1X570MIL
- added R3: (no value), symbol schematicEagle-eagle-import:RESISTOR_4PACK
- added U$1, U$17, U$19, U$21: (no value), symbol schematicEagle-eagle-import:MOUNTINGHOLE2.5
Connections:
- net EN: now also IC1.3 (EN), JP2.5, R3.6 (2)
- net GND: now also C1.2, C3.2, CONN3.1 (GND), CONN4.1 (GND), D1.C, IC1.2 (GND), IC1.5 (GND), JP2.2
- net SCL: now also CONN3.4 (SCL), CONN4.4 (SCL), IC1.6 (BUS1), JP2.3, R3.2 (1)
- net SDA: now also CONN3.3 (SDA), CONN4.3 (SDA), IC1.4 (BUS2), JP2.4, R3.1
- net VCC: now also C1.1, C3.1, CONN3.2 (V+), CONN4.2 (V+), IC1.1 (VCC), JP2.1, R3.3 (1), R3.4 (1), R3.7 (2), R3.8 (2)
- new net: D1.A, R3.5 (2)
