File: PROJ/ADAF/4863/STAN/01/src/kicadBoard.kicad_sch (KiCad schematic)
At the start: 16 parts

Commit message: Quickly Adding Everything
Parts:
- removed C1, C34: (no value), symbol eagleSchem-eagle-import:CAP_CERAMIC0805-NOOUTLINE
- removed CONN1, CONN3: (no value), symbol eagleSchem-eagle-import:STEMMA_I2C_QT
- removed D1, D2: (no value), symbol eagleSchem-eagle-import:DIODE-ZENERSOD323
- removed FID1, FID2, FID3: (no value), symbol eagleSchem-eagle-import:FIDUCIAL_1MM
- removed NEOPIX0, SENSE0: (no value), symbol eagleSchem-eagle-import:CON_JST_PH_3PIN
- removed R7, R8: (no value), symbol eagleSchem-eagle-import:RESISTOR_0603_NOOUT
- removed RPI1: (no value), symbol eagleSchem-eagle-import:RASPBERRYPI_BPLUS_IDC
- removed RPI2: (no value), symbol eagleSchem-eagle-import:RASPBERRYPI_BPLUS_2X20_THMSMT_TOP
- removed SJ1: (no value), symbol eagleSchem-eagle-import:SOLDERJUMPER_2WAY
- added C1, C34: (no value), symbol schematicEagle-eagle-import:CAP_CERAMIC0805-NOOUTLINE
- added CONN1, CONN3: (no value), symbol schematicEagle-eagle-import:STEMMA_I2C_QT
- added D1, D2: (no value), symbol schematicEagle-eagle-import:DIODE-ZENERSOD323
- added FID1, FID2, FID3: (no value), symbol schematicEagle-eagle-import:FIDUCIAL_1MM
- added NEOPIX0, SENSE0: (no value), symbol schematicEagle-eagle-import:CON_JST_PH_3PIN
- added R7, R8: (no value), symbol schematicEagle-eagle-import:RESISTOR_0603_NOOUT
- added RPI1: (no value), symbol schematicEagle-eagle-import:RASPBERRYPI_BPLUS_IDC
- added RPI3: (no value), symbol schematicEagle-eagle-import:RASPBERRYPI_BPLUS_2X20_THMSMT_TOP
- added SJ1: (no value), symbol schematicEagle-eagle-import:SOLDERJUMPER_2WAY
Connections:
- net 13S: now also R8.1, SENSE0.3
- net 18S: now also NEOPIX0.3, R7.1
- net 3.3V: now also CONN1.2 (V+), CONN3.2 (V+), RPI1.1 (3.3V), RPI3.1 (3.3V), RPI3.S1 (3.3V), SJ1.3
- net 3.3V@1: now also RPI1.17 (3.3V@1), RPI3.17 (3.3V@1), RPI3.S17 (3.3V@1)
- net 5.0V: now also RPI1.2 (5.0V), RPI1.4 (5.0V@1), RPI3.2 (5.0V), RPI3.4 (5.0V@1), RPI3.S2 (5.0V), RPI3.S4 (5.0V@1), SJ1.1
- net EECLK: now also RPI1.28 (EECLK), RPI3.28 (EECLK), RPI3.S28 (EECLK)
- net EEDATA: now also RPI1.27 (EEDATA), RPI3.27 (EEDATA), RPI3.S27 (EEDATA)
- net GND: now also C1.2, C34.2, CONN1.1 (GND), CONN3.1 (GND), D1.A, D2.A, NEOPIX0.1, RPI1.14 (GND@1), RPI1.20 (GND@2), RPI1.25 (GND@3), RPI1.30 (GND@6), RPI1.34 (GND@7), RPI1.39 (GND@5), RPI1.6 (GND), RPI1.9 (GND@4), RPI3.14 (GND@1), RPI3.20 (GND@2), RPI3.25 (GND@3), RPI3.30 (GND@6), RPI3.34 (GND@7), RPI3.39 (GND@5), RPI3.6 (GND), RPI3.9 (GND@4), RPI3.S14 (GND@1), RPI3.S20 (GND@2), RPI3.S25 (GND@3), RPI3.S30 (GND@6), RPI3.S34 (GND@7), RPI3.S39 (GND@5), RPI3.S6 (GND), RPI3.S9 (GND@4), SENSE0.1
- net GPIO12: now also RPI1.32 (GPIO12), RPI3.32 (GPIO12), RPI3.S32 (GPIO12)
- net GPIO13: now also D2.C, R8.2, RPI1.33 (GPIO13), RPI3.33 (GPIO13), RPI3.S33 (GPIO13)
- net GPIO16: now also RPI1.36 (GPIO16), RPI3.36 (GPIO16), RPI3.S36 (GPIO16)
- net GPIO17: now also RPI1.11 (GPIO17), RPI3.11 (GPIO17), RPI3.S11 (GPIO17)
- net GPIO18: now also D1.C, R7.2, RPI1.12 (GPIO18), RPI3.12 (GPIO18), RPI3.S12 (GPIO18)
- net GPIO19: now also RPI1.35 (GPIO19), RPI3.35 (GPIO19), RPI3.S35 (GPIO19)
- net GPIO20: now also RPI1.38 (GPIO20), RPI3.38 (GPIO20), RPI3.S38 (GPIO20)
- net GPIO21: now also RPI1.40 (GPIO21), RPI3.40 (GPIO21), RPI3.S40 (GPIO21)
- net GPIO22: now also RPI1.15 (GPIO22), RPI3.15 (GPIO22), RPI3.S15 (GPIO22)
- net GPIO23: now also RPI1.16 (GPIO23), RPI3.16 (GPIO23), RPI3.S16 (GPIO23)
- net GPIO24: now also RPI1.18 (GPIO24), RPI3.18 (GPIO24), RPI3.S18 (GPIO24)
- net GPIO25: now also RPI1.22 (GPIO25), RPI3.22 (GPIO25), RPI3.S22 (GPIO25)
- net GPIO26: now also RPI1.37 (GPIO26), RPI3.37 (GPIO26), RPI3.S37 (GPIO26)
- net GPIO27: now also RPI1.13 (GPIO27), RPI3.13 (GPIO27), RPI3.S13 (GPIO27)
- net GPIO4: now also RPI1.7 (GPIO4), RPI3.7 (GPIO4), RPI3.S7 (GPIO4)
- net GPIO5: now also RPI1.29 (GPIO5), RPI3.29 (GPIO5), RPI3.S29 (GPIO5)
- net GPIO6: now also RPI1.31 (GPIO6), RPI3.31 (GPIO6), RPI3.S31 (GPIO6)
- net RXD: now also RPI1.10 (RXD), RPI3.10 (RXD), RPI3.S10 (RXD)
- net SCL: now also CONN1.4 (SCL), CONN3.4 (SCL), RPI1.5 (SCL), RPI3.5 (SCL), RPI3.S5 (SCL)
- net SDA: now also CONN1.3 (SDA), CONN3.3 (SDA), RPI1.3 (SDA), RPI3.3 (SDA), RPI3.S3 (SDA)
- net SPI_CE0: now also RPI1.24 (#SPI_CE0), RPI3.24 (#SPI_CE0), RPI3.S24 (#SPI_CE0)
- net SPI_CE1: now also RPI1.26 (#SPI_CE1), RPI3.26 (#SPI_CE1), RPI3.S26 (#SPI_CE1)
- net SPI_MISO: now also RPI1.21 (SPI_MISO), RPI3.21 (SPI_MISO), RPI3.S21 (SPI_MISO)
- net SPI_MOSI: now also RPI1.19 (SPI_MOSI), RPI3.19 (SPI_MOSI), RPI3.S19 (SPI_MOSI)
- net SPI_SCLK: now also RPI1.23 (SPI_SCLK), RPI3.23 (SPI_SCLK), RPI3.S23 (SPI_SCLK)
- net TXD: now also RPI1.8 (TXD), RPI3.8 (TXD), RPI3.S8 (TXD)
- net VCC: now also C1.1, C34.1, NEOPIX0.2, SENSE0.2, SJ1.2
