File: PROJ/ADAF/5027/STAN/01/src/kicadBoard.kicad_sch (KiCad schematic)
At the start: 12 parts

Commit message: Quickly Adding Everything
Parts:
- removed C1: (no value), symbol eagleSchem-eagle-import:CAP_CERAMIC_0805MP
- removed FID1, FID2: (no value), symbol eagleSchem-eagle-import:FIDUCIAL{dblquote}{dblquote}
- removed IC1: (no value), symbol eagleSchem-eagle-import:MCP9808-E/MS
- removed JP2: (no value), symbol eagleSchem-eagle-import:HEADER-1X870MIL
- removed R1, R2, R3, R4, R5: (no value), symbol eagleSchem-eagle-import:RESISTOR0805_NOOUTLINE
- removed U$3, U$5: (no value), symbol eagleSchem-eagle-import:MOUNTINGHOLE2.5
- added C1: (no value), symbol schematicEagle-eagle-import:CAP_CERAMIC0603_NO
- added C2: (no value), symbol schematicEagle-eagle-import:CAP_CERAMIC0805-NOOUTLINE
- added CONN3, CONN4: (no value), symbol schematicEagle-eagle-import:STEMMA_I2C_QT
- added D1: (no value), symbol schematicEagle-eagle-import:LED0603_NOOUTLINE
- added FID3, FID4: (no value), symbol schematicEagle-eagle-import:FIDUCIAL_1MM
- added IC1: (no value), symbol schematicEagle-eagle-import:MCP9808-E/MS
- added JP1: (no value), symbol schematicEagle-eagle-import:HEADER-1X670MIL
- added LED0: (no value), symbol schematicEagle-eagle-import:SOLDERJUMPERCLOSED
- added R2, R3: (no value), symbol schematicEagle-eagle-import:RESISTOR_4PACK
- added SJ1, SJ2, SJ3: (no value), symbol schematicEagle-eagle-import:SOLDERJUMPER
- added U$1, U$17, U$19, U$21: (no value), symbol schematicEagle-eagle-import:MOUNTINGHOLE2.5
Connections:
- net A0: now also IC1.7 (A0), JP1.6, R2.6 (2), SJ1.1
- net A1: now also IC1.6 (A1), R2.7 (2), SJ2.1
- net A2: now also IC1.5 (A2), R2.8 (2), SJ3.1
- net ALERT: now also IC1.3 (ALERT), JP1.5
- net GND: now also C1.2, C2.2, CONN3.1 (GND), CONN3.MT1 (MT), CONN3.MT2 (MT), CONN4.1 (GND), CONN4.MT1 (MT), CONN4.MT2 (MT), D1.C, IC1.4 (GND), JP1.2, R2.1, R2.2 (1), R2.3 (1)
- net SCL: now also CONN3.4 (SCL), CONN4.4 (SCL), IC1.2 (SCL), JP1.3, R3.6 (2)
- net SDA: now also CONN3.3 (SDA), CONN4.3 (SDA), IC1.1 (SDA), JP1.4, R3.7 (2)
- new net: D1.A, LED0.1
- new net: LED0.2, R3.1
- new net VCC: C1.1, C2.1, CONN3.2 (V+), CONN4.2 (V+), IC1.8 (VDD), JP1.1, R3.2 (1), R3.3 (1), R3.8 (2), SJ1.2, SJ2.2, SJ3.2
Other:
- note added: "I2C Pullups & Shift"
- note added: "ON LED"
- note added: "Power supply"
- note added: "STEMMA/I2C Headers"
