File: PROJ/ADAF/5159/STAN/01/src/kicadBoard.kicad_sch (KiCad schematic)
At the start: 15 parts

Commit message: Quickly Adding Everything
Parts:
- removed C2: (no value), symbol eagleSchem-eagle-import:CAP_CERAMIC0603_NO
- removed CONN3, CONN4: (no value), symbol eagleSchem-eagle-import:STEMMA_I2C_QT
- removed D2: (no value), symbol eagleSchem-eagle-import:LED0603_NOOUTLINE
- removed FID3, FID4: (no value), symbol eagleSchem-eagle-import:FIDUCIAL_1MM
- removed IC1: (no value), symbol eagleSchem-eagle-import:TCA4307
- removed JP2: (no value), symbol eagleSchem-eagle-import:HEADER-1X4ROUND
- removed JP3: (no value), symbol eagleSchem-eagle-import:HEADER-1X670MIL
- removed R1, R2: (no value), symbol eagleSchem-eagle-import:RESISTOR_4PACK
- removed U$1, U$17, U$19, U$21: (no value), symbol eagleSchem-eagle-import:MOUNTINGHOLE2.5
- added C2: (no value), symbol schematicEagle-eagle-import:CAP_CERAMIC0603_NO
- added CONN3, CONN4: (no value), symbol schematicEagle-eagle-import:STEMMA_I2C_QT
- added D2: (no value), symbol schematicEagle-eagle-import:LED0603_NOOUTLINE
- added FID3, FID4: (no value), symbol schematicEagle-eagle-import:FIDUCIAL_1MM
- added IC1: (no value), symbol schematicEagle-eagle-import:TCA4307
- added JP2: (no value), symbol schematicEagle-eagle-import:HEADER-1X4ROUND
- added JP3: (no value), symbol schematicEagle-eagle-import:HEADER-1X670MIL
- added R1, R2: (no value), symbol schematicEagle-eagle-import:RESISTOR_4PACK
- added U$1, U$17, U$19, U$21: (no value), symbol schematicEagle-eagle-import:MOUNTINGHOLE2.5
Connections:
- net EN: now also IC1.1 (EN), JP3.2, R1.7 (2)
- net GND: now also C2.2, CONN3.1 (GND), CONN4.1 (GND), D2.C, IC1.4 (GND), JP2.2, JP3.5
- net READY: now also IC1.5 (READY), JP3.1, R2.8 (2)
- net SCL_IN: now also CONN3.4 (SCL), IC1.3 (SCL_IN), JP3.4, R1.4 (1)
- net SCL_OUT: now also CONN4.4 (SCL), IC1.2 (SCL_OUT), JP2.3, R2.3 (1)
- net SDA_IN: now also CONN3.3 (SDA), IC1.6 (SDA_IN), JP3.3, R1.3 (1)
- net SDA_OUT: now also CONN4.3 (SDA), IC1.7 (SDA_OUT), JP2.4, R2.2 (1)
- net VCC: now also C2.1, CONN3.2 (V+), CONN4.2 (V+), IC1.8 (VCC), JP2.1, JP3.6, R1.2 (1), R1.5 (2), R1.6 (2), R1.8 (2), R2.1, R2.6 (2), R2.7 (2)
- new net: D2.A, R1.1
