File: PROJ/DANP/0001/STAN/1C/src/kicadBoard.kicad_sch (KiCad schematic)
At the start: 195 parts

Commit message: Quickly Adding Everything
Parts:
- removed C100, C101, C102, C103, C106, C108, C109, C110, C111, C112, C113, C114, C200, C201, C202, C203, C204, C205, C302, C303, C308, C400, C401, C402, C403, C404, C405, C406, C407, C408, C409, C410, C411, C412, C413, C414, C415, C416, C417, C418, C419, C420, C421, C422, C423, C501, C602, C702, C703, C704, C705, C707, C708, C709, C710, C711, C712, C713, C714, C715: (no value), symbol eagleSchem-eagle-import:CAPACITOR_NPOL-0402
- removed C104, C800: (no value), symbol eagleSchem-eagle-import:CAPACITOR_POL-SMC_A
- removed C105, C107, C115, C116, C300, C301, C304, C305, C306, C307, C500, C600, C601, C700, C701, C706: (no value), symbol eagleSchem-eagle-import:CAPACITOR_NPOL-0603
- removed D200: (no value), symbol eagleSchem-eagle-import:DIODE-SOD-123
- removed J1: (no value), symbol eagleSchem-eagle-import:USB-C-12
- removed J2: (no value), symbol eagleSchem-eagle-import:CON_HEADER_1X04
- removed J3: (no value), symbol eagleSchem-eagle-import:CON_HEADER_1X10-RIGHT_ANGLED_PTH_SHROUDED
- removed J4: (no value), symbol eagleSchem-eagle-import:CON-FPC_X05B20L10T
- removed L800: (no value), symbol eagleSchem-eagle-import:WE-KIL_0805
- removed LED900, LED901, LED902, LED903, LED904, LED905, LED906, LED907: (no value), symbol eagleSchem-eagle-import:LED-0805
- removed LOGO1: (no value), symbol eagleSchem-eagle-import:LOGO_CC-0
- removed PCB1: (no value), symbol eagleSchem-eagle-import:PCB_DP_RECTANGLE-50X100
- removed Q300: (no value), symbol eagleSchem-eagle-import:TRANSISTOR_FET_TSM2301CX
- removed Q301: (no value), symbol eagleSchem-eagle-import:TRANSISTOR-BJT_DMMT3906W
- removed R100, R101, R200, R201, R202, R203, R204, R300, R301, R307, R308, R309, R310, R311, R400, R401, R402, R403, R404, R405, R406, R407, R408, R409, R410, R411, R412, R413, R414, R415, R416, R417, R418, R419, R420, R421, R422, R423, R424, R425, R426, R427, R428, R429, R430, R431, R700, R701, R702, R800, R801, R802, R803, R804, R805, R806: (no value), symbol eagleSchem-eagle-import:RESISTOR-0402
- removed R302, R303, R304, R305, R306, R900, R901, R902, R903: (no value), symbol eagleSchem-eagle-import:RESISTOR-0603
- removed RN500, RN501: (no value), symbol eagleSchem-eagle-import:RNETWORK
- removed U100: (no value), symbol eagleSchem-eagle-import:IC_UC_STM32F103ZX
- removed U101: (no value), symbol eagleSchem-eagle-import:IC_MEM_W25X40CL
- removed U200: (no value), symbol eagleSchem-eagle-import:IC_74HCT4067
- removed U201, U301: (no value), symbol eagleSchem-eagle-import:IC_OP-AMP_MCP6001
- removed U202: (no value), symbol eagleSchem-eagle-import:IC_ADC_ADS7041
- removed U300: (no value), symbol eagleSchem-eagle-import:IC_MCP1824_ADJ
- removed U302: (no value), symbol eagleSchem-eagle-import:IC_MCP1700
- removed U303: (no value), symbol eagleSchem-eagle-import:MIC5205
- removed U400, U401, U404, U405, U408, U409, U412, U413: (no value), symbol eagleSchem-eagle-import:IC_BUFF_SN74LVC1T45DBV-SC-70-6
- removed U402, U403, U406, U407, U410, U411, U414, U415: (no value), symbol eagleSchem-eagle-import:IC_BUFF_74LVC1G07
- removed U500, U501: (no value), symbol eagleSchem-eagle-import:IC_74HCT4066PW
- removed U600, U601: (no value), symbol eagleSchem-eagle-import:IC_MEM_23LC1024
- removed U602: (no value), symbol eagleSchem-eagle-import:IC_BUFF_74LVC245A-TSSOP20
- removed U700: (no value), symbol eagleSchem-eagle-import:IC_FPGA_ICE40HX4K
- removed XTAL100: (no value), symbol eagleSchem-eagle-import:OSC-XTAL-12M
- added C100, C101, C102, C103, C106, C108, C109, C110, C111, C112, C113, C114, C200, C201, C202, C203, C204, C205, C302, C303, C308, C400, C401, C402, C403, C404, C405, C406, C407, C408, C409, C410, C411, C412, C413, C414, C415, C416, C417, C418, C419, C420, C421, C422, C423, C501, C602, C702, C703, C704, C705, C707, C708, C709, C710, C711, C712, C713, C714, C715: (no value), symbol schematicEagle-eagle-import:CAPACITOR_NPOL-0402
- added C104, C800: (no value), symbol schematicEagle-eagle-import:CAPACITOR_POL-SMC_A
- added C105, C107, C115, C116, C300, C301, C304, C305, C306, C307, C500, C600, C601, C700, C701, C706: (no value), symbol schematicEagle-eagle-import:CAPACITOR_NPOL-0603
- added D200: (no value), symbol schematicEagle-eagle-import:DIODE-SOD-123
- added J1: (no value), symbol schematicEagle-eagle-import:USB-C-12
- added J2: (no value), symbol schematicEagle-eagle-import:CON_HEADER_1X04
- added J3: (no value), symbol schematicEagle-eagle-import:CON_HEADER_1X10-RIGHT_ANGLED_PTH_SHROUDED
- added J4: (no value), symbol schematicEagle-eagle-import:CON-FPC_X05B20L10T
- added L800: (no value), symbol schematicEagle-eagle-import:WE-KIL_0805
- added LED900, LED901, LED902, LED903, LED904, LED905, LED906, LED907: (no value), symbol schematicEagle-eagle-import:LED-0805
- added LOGO1: (no value), symbol schematicEagle-eagle-import:LOGO_CC-0
- added PCB1: (no value), symbol schematicEagle-eagle-import:PCB_DP_RECTANGLE-50X100
- added Q300: (no value), symbol schematicEagle-eagle-import:TRANSISTOR_FET_TSM2301CX
- added Q301: (no value), symbol schematicEagle-eagle-import:TRANSISTOR-BJT_DMMT3906W
- added R100, R101, R200, R201, R202, R203, R204, R300, R301, R307, R308, R309, R310, R311, R400, R401, R402, R403, R404, R405, R406, R407, R408, R409, R410, R411, R412, R413, R414, R415, R416, R417, R418, R419, R420, R421, R422, R423, R424, R425, R426, R427, R428, R429, R430, R431, R700, R701, R702, R800, R801, R802, R803, R804, R805, R806: (no value), symbol schematicEagle-eagle-import:RESISTOR-0402
- added R302, R303, R304, R305, R306, R900, R901, R902, R903: (no value), symbol schematicEagle-eagle-import:RESISTOR-0603
- added RN500, RN501: (no value), symbol schematicEagle-eagle-import:RNETWORK
- added U100: (no value), symbol schematicEagle-eagle-import:IC_UC_STM32F103ZX
- added U101: (no value), symbol schematicEagle-eagle-import:IC_MEM_W25X40CL
- added U200: (no value), symbol schematicEagle-eagle-import:IC_74HCT4067
- added U201, U301: (no value), symbol schematicEagle-eagle-import:IC_OP-AMP_MCP6001
- added U202: (no value), symbol schematicEagle-eagle-import:IC_ADC_ADS7041
- added U300: (no value), symbol schematicEagle-eagle-import:IC_MCP1824_ADJ
- added U302: (no value), symbol schematicEagle-eagle-import:IC_MCP1700
- added U303: (no value), symbol schematicEagle-eagle-import:MIC5205
- added U400, U401, U404, U405, U408, U409, U412, U413: (no value), symbol schematicEagle-eagle-import:IC_BUFF_SN74LVC1T45DBV-SC-70-6
- added U402, U403, U406, U407, U410, U411, U414, U415: (no value), symbol schematicEagle-eagle-import:IC_BUFF_74LVC1G07
- added U500, U501: (no value), symbol schematicEagle-eagle-import:IC_74HCT4066PW
- added U600, U601: (no value), symbol schematicEagle-eagle-import:IC_MEM_23LC1024
- added U602: (no value), symbol schematicEagle-eagle-import:IC_BUFF_74LVC245A-TSSOP20
- added U700: (no value), symbol schematicEagle-eagle-import:IC_FPGA_ICE40HX4K
- added XTAL100: (no value), symbol schematicEagle-eagle-import:OSC-XTAL-12M
Connections:
- net +3V3: now also C102.1, C103.1, C104.+, C105.1, C106.1, C107.1, C108.1, C109.1, C110.1, C111.1, C112.1, C113.1, C114.1, C115.1, C116.1, C200.2, C201.1, C202.1, C204.1, C205.1, C300.1, C302.2, C303.2, C305.2, C306.2, C307.2, C308.2, C400.2, C402.2, C404.2, C406.2, C408.2, C410.2, C412.2, C414.2, C416.2, C417.2, C418.2, C419.2, C420.2, C421.2, C422.2, C423.2, C500.2, C501.2, C600.2, C601.2, C602.2, C700.1, C701.1, C702.1, C703.1, C704.1, C705.1, C706.1, C707.1, C708.1, C709.1, C710.1, C711.1, C712.1, C713.1, C714.1, C715.1, C800.+, D200.C, J2.1, J4.9, L800.1 (2), R100.2, R402.2, R403.2, R408.2, R409.2, R414.2, R415.2, R420.2, R421.2, R700.2, R701.2, R805.1, R900.2, U100.108 (VDD_2), U100.121 (VDD_10), U100.131 (VDD_11), U100.144 (VDD_3), U100.17 (VDD_5), U100.32 (VREF+), U100.33 (VDDA), U100.35 (PA1/USART2_RTS('0')/ADC123_IN1/TIM5_CH2/TIM2_CH2('00')), U100.39 (VDD_4), U100.52 (VDD_6), U100.6 (VBAT), U100.62 (VDD_7), U100.72 (VDD_1), U100.84 (VDD_8), U100.95 (VDD_9), U101.3 (~{WP}), U101.7 (~{HOLD}), U101.8 (VCC), U200.24 (V+), U201.5 (V+), U202.1 (DVDD), U202.7 (AVDD), U300.1 (VIN), U301.5 (V+), U302.2 (VIN), U302.3 (VOUT), U303.1 (IN), U303.3 (EN), U303.5 (OUT), U400.1 (VCCA), U401.1 (VCCA), U402.5 (V+), U403.5 (V+), U404.1 (VCCA), U405.1 (VCCA), U406.5 (V+), U407.5 (V+), U408.1 (VCCA), U409.1 (VCCA), U410.5 (V+), U411.5 (V+), U412.1 (VCCA), U413.1 (VCCA), U414.5 (V+), U415.5 (V+), U500.14 (V+), U501.14 (V+), U600.8 (V+), U601.8 (V+), U602.20 (V+), U700.100 (VCCIO_1@1), U700.108 (VPP_2V5), U700.111 (VCC@0), U700.123 (VCCIO_0@0), U700.126 (VCCPLL1), U700.131 (VCCIO_0@1), U700.27 (VCC@0), U700.30 (VCCIO_3@1), U700.40 (VCC@0), U700.46 (VCCIO_2@0), U700.54 (VCCPLL0), U700.57 (VCCIO_2@1), U700.6 (VCCIO_3@0), U700.72 (VCC_SPI), U700.89 (VCCIO_1@0), U700.92 (VCC@0)
- net ADC_CLOCK: now also U202.2 (SCLK), U700.48 (IOB_80)
- net ADC_CS: now also U202.4 (CS), U700.45 (IOB_73)
- net ADC_DATA: now also U202.3 (SDO), U700.47 (IOB_79)
- net ADC_MUX_EN: now also U200.15 (~{E}), U700.55 (IOB_91)
- net ADC_MUX_S0: now also U200.10 (S0), U700.80 (IOR_116)
- net ADC_MUX_S1: now also U200.11 (S1), U700.81 (IOR_117)
- net ADC_MUX_S2: now also U200.14 (S2), U700.82 (IOR_118)
- net ADC_MUX_S3: now also U200.13 (S3), U700.83 (IOR_119)
- net BPIO0: now also J3.1, R424.1, RN500.1, U200.9 (Y0), U602.18 (B0)
- net BPIO1: now also J3.2, R425.1, RN500.2 (1), U200.8 (Y1), U602.17 (B1)
- net BPIO2: now also J3.3, R426.1, RN500.3 (1), U200.7 (Y2), U602.16 (B2)
- net BPIO3: now also J3.4, R427.1, RN500.4 (1), U200.6 (Y3), U602.15 (B3)
- net BPIO4: now also J3.5, R428.1, RN501.5 (2), U200.5 (Y4), U602.14 (B4)
- net BPIO5: now also J3.6, R429.1, RN501.6 (2), U200.4 (Y5), U602.13 (B5)
- net BPIO6: now also J3.7, R430.1, RN501.7 (2), U200.3 (Y6), U602.12 (B6)
- net BPIO7: now also J3.8, R431.1, RN501.8 (2), U200.2 (Y7), U602.11 (B7)
- net BUFDIR0: now also R400.2, U400.5 (DIR), U700.107 (IOR_167)
- net BUFDIR1: now also R406.2, U404.5 (DIR), U700.113 (IOT_170)
- net BUFDIR2: now also R412.2, U408.5 (DIR), U700.99 (IOR_152)
- net BUFDIR3: now also R418.2, U412.5 (DIR), U700.104 (IOR_164)
- net BUFDIR4: now also R401.2, U401.5 (DIR), U700.79 (IOR_115)
- net BUFDIR5: now also R407.2, U405.5 (DIR), U700.75 (IOR_111)
- net BUFDIR6: now also R413.2, U409.5 (DIR), U700.64 (CBSEL1/IOB_104)
- net BUFDIR7: now also R419.2, U413.5 (DIR), U700.61 (IOB_96)
- net BUFIO0: now also U400.3 (A), U700.106 (IOR_166)
- net BUFIO1: now also U404.3 (A), U700.112 (IOT_169)
- net BUFIO2: now also U408.3 (A), U700.98 (IOR_148)
- net BUFIO3: now also U412.3 (A), U700.102 (IOR_161)
- net BUFIO4: now also U401.3 (A), U700.78 (IOR_114)
- net BUFIO5: now also U405.3 (A), U700.74 (IOR_110)
- net BUFIO6: now also U409.3 (A), U700.63 (CBSEL0/IOB_103)
- net BUFIO7: now also U413.3 (A), U700.60 (IOB_95)
- net BUFOD0: now also R402.1, U402.2 (I), U700.105 (IOR_165)
- net BUFOD1: now also R408.1, U406.2 (I), U700.110 (IOT_168)
- net BUFOD2: now also R414.1, U410.2 (I), U700.97 (IOR_147)
- net BUFOD3: now also R420.1, U414.2 (I), U700.101 (IOR_160)
- net BUFOD4: now also R403.1, U403.2 (I), U700.76 (IOR_112)
- net BUFOD5: now also R409.1, U407.2 (I), U700.73 (IOR_109)
- net BUFOD6: now also R415.1, U411.2 (I), U700.62 (IOB_102)
- net BUFOD7: now also R421.1, U415.2 (I), U700.56 (IOB_94)
- net DISPLAY_AUX1: now also J4.2, U100.47 (ADC12_IN9/TIM3_CH4('00'OR'10')/TIM8_CH3N/TIM1_CH3N('01')/PB1)
- net DISPLAY_CS: now also J4.5, U100.44 (ADC12_IN14/PC4)
- net DISPLAY_D/P: now also J4.4, U100.45 (ADC12_IN15/PC5)
- net DISPLAY_PWM: now also J4.3, U100.46 (ADC12_IN8/TIM3_CH3('00'OR'10')/TIM8_CH2N/TIM1_CH2N('01')/PB0)
- net DISPLAY_RESET: now also J4.1, R101.2, U100.48 (BOOT1/FT/PB2)
- net DISPLAY_SPI_CLOCK: now also J4.8, U100.41 (PA5/SPI1_SCK('0')/ADC12_IN5)
- net DISPLAY_SPI_MISO: now also J4.7, U100.42 (PA6/SPI1_MISO('0')/TIM8_BKIN/ADC12_IN6/TIM3_CH1('00')/TIM1_BKIN('01'))
- net DISPLAY_SPI_MOSI: now also J4.6, U100.43 (PA7/SPI1_MOSI('0')/TIM8_CH1N/ADC12_IN7/TIM3_CH2('00')/TIM1_CH1N('01'))
- net FLASH_CS: now also U100.132 (PG15/FT), U101.1 (~{CS})
- net FLASH_MISO: now also U100.134 (SPI3_MISO('0')/TIM3_CH1('10')/SPI1_MISO('1')/NJTRST/FT/PB4), U101.2 (SO)
- net FLASH_MOSI: now also U100.135 (I2C1_SMBA/SPI3_MOSI('0')/TIM3_CH2('10')/SPI1_MOSI('1')/PB5), U101.5 (SI)
- net FLASH_SCK: now also U100.133 (SPI3_SCK('0')/TIM2_CH2('01')/SPI1_SCK('1')/JTDO/FT//PB3), U101.6 (SCK)
- net FPGA_CDONE: now also R700.1, U100.69 (I2C2_SCL/USART3_TX('00')/TIM2_CH3('10'OR'11')/FT/PB10), U700.65 (CDONE)
- net FPGA_CRESET: now also R701.1, U100.70 (I2C2_SDA/USART3_RX('00')/TIM2_CH4('10'OR'11')/FT/PB11), U700.66 (CRESET_B)
- net FPGA_PROG_CLOCK: now also U100.74 (SPI2_SCK/USART3_CTS('00'OR'01')/TIM1_CH1N('00')/FT/PB13), U700.70 (IOB_107/SCK)
- net FPGA_PROG_CS: now also R702.2, U100.73 (SPI2_NSS/I2C2_SMBA/USART3_CK(00)/TIM1_BKIN('00')/FT/PB12), U700.71 (IOB_108/SS)
- net FPGA_PROG_MISO: now also U100.75 (SPI2_MISO/USART3_RTS('00'OR'01')/TIM1_CH2N('00')/FT/PB14), U700.67 (IOB_105/SDO)
- net FPGA_PROG_MOSI: now also U100.76 (SPI2_MOSI/TIM1_CH3N('00')/FT/PB15), U700.68 (IOB_106/SDI)
- net FSMC_A0: now also U100.10 (FSMC_A0/FT/PF0), U700.3 (IOL_3A)
- net FSMC_A1: now also U100.11 (FSMC_A1/FT/PF1), U700.4 (IOL_3B)
- net FSMC_A10: now also U100.56 (PG0/FT/FSMC_A10), U700.38 (IOB_57)
- net FSMC_A2: now also U100.12 (FSMC_A2/FT/PF2), U700.7 (IOL_4A)
- net FSMC_A3: now also U100.13 (FSMC_A3/FT/PF3), U700.8 (IOL_4B)
- net FSMC_A4: now also U100.14 (FSMC_A4/FT/PF4), U700.9 (IOL_5A)
- net FSMC_A5: now also U100.15 (FSMC_A5/FT/PF5), U700.10 (IOL_5B)
- net FSMC_A6: now also U100.50 (FSMC_A6/FT/PF12), U700.42 (IOB_64)
- net FSMC_A7: now also U100.53 (FSMC_A7/FT/PF13), U700.37 (IOB_56)
- net FSMC_A8: now also U100.54 (FSMC_A8/FT/PF14), U700.39 (IOB_61)
- net FSMC_A9: now also U100.55 (FSMC_A9/FT/PF15), U700.41 (IOB_63)
- net FSMC_D0: now also U100.85 (PD14/FT/FSMC_D0/TIM4_CH3('1')), U700.24 (IOL_17B)
- net FSMC_D1: now also U100.86 (PD15/FT/FSMC_D1/TIM4_CH4('1')), U700.23 (IOL_17A)
- net FSMC_D10: now also U100.66 (PE13/FT/FSMC_D10/TIM1_CH3('11')), U700.26 (IOL_18B)
- net FSMC_D11: now also U100.67 (PE14/FT/FSMC_D11/TIM1_CH4('11')), U700.28 (IOL_23A)
- net FSMC_D12: now also U100.68 (PE15/FT/FSMC_D12/TIM1_BKIN('11')), U700.29 (IOL_23B)
- net FSMC_D13: now also U100.77 (PD8/FT/FSMC_D13/USART3_TX('11')), U700.33 (IOL_25A)
- net FSMC_D14: now also U100.78 (PD9/FT/FSMC_D14/USART3_RX('11')), U700.32 (IOL_24B)
- net FSMC_D15: now also U100.79 (PD10/FT/FSMC_D15/USART3_CK('11')), U700.31 (IOL_24A)
- net FSMC_D2: now also U100.114 (PD0/FT/FSMC_D2), U700.1 (IOL_2A)
- net FSMC_D3: now also U100.115 (PD1/FT/FSMC_D3), U700.2 (IOL_2B)
- net FSMC_D4: now also U100.58 (PE7/FT/FSMC_D4/TIM1_ETR('11')), U700.15 (IOL_10A)
- net FSMC_D5: now also U100.59 (PE8/FT/FSMC_D5/TIM1_CH1N('11')), U700.16 (IOL_10B)
- net FSMC_D6: now also U100.60 (PE9/FT/FSMC_D6/TIM1_CH1('11')), U700.17 (IOL_12A)
- net FSMC_D7: now also U100.63 (PE10/FT/FSMC_D7/TIM1_CH2N('11')), U700.18 (IOL_12B)
- net FSMC_D8: now also U100.64 (PE11/FT/FSMC_D8/TIM1_CH2('11')), U700.19 (IOL_13A)
- net FSMC_D9: now also U100.65 (PE12/FT/FSMC_D9/TIM1_CH3N('11')), U700.25 (IOL_18A)
- net FSMC_NE3_CE: now also U100.125 (PG10/FT/FSMC_NCE4_1/FSMC_NE3), U700.22 (IOL_14B)
- net FSMC_NOE_OE: now also U100.118 (PD4/FT/FSMC_NOE/USART2_RTS(1)), U700.11 (IOL_8A)
- net FSMC_NWE_WE: now also U100.119 (PD5/FT/FSMC_NWE/USART2_TX('1')), U700.12 (IOL_8B)
- net GND: now also C100.2, C101.2, C102.2, C103.2, C104.-, C105.2, C106.2, C107.2, C108.2, C109.2, C110.2, C111.2, C112.2, C113.2, C114.2, C115.2, C116.2, C200.1, C201.2, C202.2, C203.2, C204.2, C205.2, C300.2, C301.2, C302.1, C303.1, C304.1, C305.1, C306.1, C307.1, C308.1, C400.1, C401.2, C402.1, C403.2, C404.1, C405.2, C406.1, C407.2, C408.1, C409.2, C410.1, C411.2, C412.1, C413.2, C414.1, C415.2, C416.1, C417.1, C418.1, C419.1, C420.1, C421.1, C422.1, C423.1, C500.1, C501.1, C600.1, C601.1, C602.1, C700.2, C701.2, C702.2, C703.2, C704.2, C705.2, C706.2, C707.2, C708.2, C709.2, C710.2, C711.2, C712.2, C713.2, C714.2, C715.2, C800.-, J1.GND@1 (GND), J1.GND@2 (GND), J1.P$1 (CHASSIS), J1.P$2 (CHASSIS), J1.P$3 (CHASSIS), J1.P$4 (CHASSIS), J1.P$5 (CHASSIS), J1.P$6 (CHASSIS), J1.P$7 (CHASSIS), J1.P$8 (CHASSIS), J2.2, J3.10, J4.10, LED900.C, LED901.C, LED902.C, LED903.C, LED904.C, LED905.C, LED906.C, LED907.C, R101.1, R204.2, R301.2, R303.1, R304.1, R305.2, R308.2, R311.2, R400.1, R401.1, R404.1, R405.1, R406.1, R407.1, R410.1, R411.1, R412.1, R413.1, R416.1, R417.1, R418.1, R419.1, R422.1, R423.1, R702.1, R803.2, R804.2, R806.1, U100.107 (VSS_2), U100.120 (VSS_10), U100.130 (VSS_11), U100.138 (BOOT0), U100.143 (VSS_3), U100.16 (VSS_5), U100.30 (VSSA), U100.31 (VREF-), U100.38 (VSS_4), U100.51 (VSS_6), U100.61 (VSS_7), U100.71 (VSS_1), U100.83 (VSS_8), U100.94 (VSS_9), U101.4 (GND), U200.12 (GND), U201.2 (V-), U202.5 (AINM), U202.8 (GND), U300.2 (GND), U301.2 (V-), U302.1 (GND), U303.2 (GND), U400.2 (GND), U401.2 (GND), U402.3 (GND), U403.3 (GND), U404.2 (GND), U405.2 (GND), U406.3 (GND), U407.3 (GND), U408.2 (GND), U409.2 (GND), U410.3 (GND), U411.3 (GND), U412.2 (GND), U413.2 (GND), U414.3 (GND), U415.3 (GND), U500.7 (GND), U501.7 (GND), U600.4 (GND), U601.4 (GND), U602.10 (GND), U700.103 (GND@1), U700.127 (GNDPLL1), U700.13 (GND@1), U700.132 (GND@0), U700.14 (GND@2), U700.140 (GND@1), U700.5 (GND@0), U700.53 (GNDPLL0), U700.59 (GND@0), U700.69 (GND@0), U700.86 (GND@0)
- net LAT0: now also U602.2 (A0), U700.94 (GBIN2/IOR_141)
- net LAT1: now also U602.3 (A1), U700.93 (GBIN3/IOR_140)
- net LAT2: now also U602.4 (A2), U700.91 (IOR_139)
- net LAT3: now also U602.5 (A3), U700.90 (IOR_138)
- net LAT4: now also U602.6 (A4), U700.88 (IOR_137)
- net LAT5: now also U602.7 (A5), U700.87 (IOR_136)
- net LAT6: now also U602.8 (A6), U700.85 (IOR_128)
- net LAT7: now also U602.9 (A7), U700.84 (IOR_120)
- net LAT_DIR: now also U602.1 (DIR), U700.95 (IOR_144)
- net LAT_OE: now also U602.19 (~{OE}), U700.96 (IOR_146)
- net LD1: now also R901.2, U100.110 (PA15/FT/JTDI/SPI3_NSS('0')/TIM2_CH1_ETR('11')/SPI1_NSS('1'))
- net MASTER_RESET: now also U100.93 (PG8/FT), U700.21 (GBIN6/IOL_14A)
- net MCU_ADC0: now also R310.2, R311.1, U100.34 (PA0/WKUP/USART2_CTS('0')/ADC123_IN0/TIM2_CH1_ETR/TIM5_CH1/TIM8_ETR)
- net MCU_ADC2: now also R302.2, R305.1, U100.36 (PA2/USART2_TX('0')/TIM5_CH3/ADC123_IN2/TIM2_CH3('00'OR'01))
- net MCU_ADC3: now also R805.2, R806.2, U100.37 (PA3/USART2_RX('0')/TIM5_CH4/ADC123_IN3/TIM2_CH4('00'OR'01'))
- net MCU_AUX0: now also U100.99 (TIM8_CH4/TIM3_CH4('11')/FT/PC9), U700.115 (IOT_172)
- net MCU_AUX1: now also U100.111 (UART4_TX/USART3_TX('01')/FT/PC10), U700.137 (IOT_215)
- net MCU_AUX2: now also U100.112 (UART4_RX/USART3_RX('01')/FT/PC11), U700.136 (IOT_214)
- net MCU_AUX3: now also U100.113 (UART5_TX/USART3_CK('01')/FT/PC12), U700.135 (IOT_213)
- net MCU_AUX4: now also U100.139 (TIM4_CH3('0')/I2C1_SCL('1')/FT/PB8), U700.130 (IOT_206)
- net MCU_AUX5: now also U100.140 (TIM4_CH4('0')/I2C1_SDA('1')/FT/PB9), U700.125 (IOT_192)
- net MCU_INT0: now also U100.141 (PE0/FT/TIM4_ETR/FSMC_NBL0), U700.124 (IOT_191)
- net MCU_INT1: now also U100.142 (PE1/FT/FSMC_NBL1), U700.122 (IOT_190)
- net MCU_INT2: now also U100.57 (PG1/FT/FSMC_A11), U700.114 (IOT_171)
- net MCU_INT3: now also U100.116 (PD2/FT/TIM3_ETR/UART5_RX), U700.134 (IOT_212)
- net MCU_MCO: now also U100.100 (PA8/FT/USART1_CK/TIM1_CH1('00'OR'01')/MCO), U700.128 (GBIN1/IOT_197)
- net MCU_PWM0: now also U100.102 (PA10/FT/USART1_RX('0')/TIM1_CH3('00'OR'01')), U700.129 (GBIN0/IOT_198)
- net MCU_PWM1: now also U100.96 (TIM8_CH1/TIM3_CH1('11')/FT/PC6), U700.49 (GBIN5/IOB_81)
- net MCU_VPU: now also U100.101 (PA9/FT/USART1_TX('0')/TIM1_CH2('00'OR'01')), U500.12 (E), U500.13 (E), U500.5 (E), U500.6 (E), U501.12 (E), U501.13 (E), U501.5 (E), U501.6 (E)
- net RST: now also R100.1, U100.25 (NRST)
- net SRAM0_CLOCK: now also U600.6 (SCK), U700.141 (IOT_219)
- net SRAM0_CS: now also U600.1 (~{CS}), U700.144 (IOT_222)
- net SRAM0_SIO0: now also U600.5 (SI/SIO0), U700.138 (IOT_216)
- net SRAM0_SIO1: now also U600.2 (SO/SIO1), U700.142 (IOT_220)
- net SRAM0_SIO2: now also U600.3 (SIO2), U700.139 (IOT_217)
- net SRAM0_SIO3: now also U600.7 (~{HOLD/SIO3}), U700.143 (IOT_221)
- net SRAM1_CLOCK: now also U601.6 (SCK), U700.118 (IOT_177)
- net SRAM1_CS: now also U601.1 (~{CS}), U700.121 (IOT_181)
- net SRAM1_SIO0: now also U601.5 (SI/SIO0), U700.116 (IOT_173)
- net SRAM1_SIO1: now also U601.2 (SO/SIO1), U700.119 (IOT_178)
- net SRAM1_SIO2: now also U601.3 (SIO2), U700.117 (IOT_174)
- net SRAM1_SIO3: now also U601.7 (~{HOLD/SIO3}), U700.120 (IOT_179)
- net SWCLK: now also J2.4, U100.109 (PA14/FT/JTCK-SWCLK)
- net SWDIO: now also J2.3, U100.105 (PA13/FT/JTMS-SWDIO)
- net USBLED: now also R903.2, U100.117 (PD3/FT/FSMC_CLK/USART2_CTS(1))
- net USB_D+: now also R801.1, U100.104 (PA12/FT/USART1_RTS/USBDP/TIM1_ETR('00'OR'01'))
- net USB_D-: now also R802.1, U100.103 (PA11/FT/USART1_CTS/USBDM/TIM1_CH4('00'OR'01'))
- net USB_DET: now also R800.2, U100.5 (PE6/FT/FSMC_A22)
- net VPP_FAST: now also U700.109 (VPP_FAST)
- net VREF/VOUT: now also C401.1, C403.1, C405.1, C407.1, C409.1, C411.1, C413.1, C415.1, J3.9, Q300.2 (S), Q301.5 (E), R302.1, U200.23 (Y8), U400.6 (VCCB), U401.6 (VCCB), U404.6 (VCCB), U405.6 (VCCB), U408.6 (VCCB), U409.6 (VCCB), U412.6 (VCCB), U413.6 (VCCB), U500.10 (Z), U500.2 (Z), U500.3 (Z), U500.9 (Z), U501.10 (Z), U501.2 (Z), U501.3 (Z), U501.9 (Z)
- net VREGEN: now also R301.1, R902.2, U100.4 (PE5/FT/FSMC_A21), U300.3 (~{SHDN})
- net VREG_DAC: now also R306.1, U100.40 (PA4/SPI1_NSS('0')/USART2_CK('0')/ADC12_IN4)
- new net: R411.2, R429.2, U405.4 (B), U407.4 (O)
- new net: Q301.1 (B), Q301.2 (B), Q301.3 (C), R303.2
- new net: Q300.1 (G), Q301.6 (C), R304.2
- new net: R417.2, R430.2, U409.4 (B), U411.4 (O)
- new net: LED901.A, LED905.A, R901.1
- new net: C304.2, R306.2, U301.3 (+)
- new net: J1.DP1, J1.DP2, R800.1, R801.2
- new net: R405.2, R428.2, U401.4 (B), U403.4 (O)
- new net: RN501.2 (1), U501.11 (Y)
- new net: C203.1, R203.2, U202.6 (AINP)
- new net: R201.1, U201.1 (OUT), U201.4 (-)
- new net: R201.2, R202.1
- new net: R202.2, R203.1, R204.1
- new net: J1.DN1, J1.DN2, R802.2
- new net: RN500.6 (2), U500.11 (Y)
- new net: LED903.A, LED907.A, R903.1
- new net: R404.2, R424.2, U400.4 (B), U402.4 (O)
- new net: R200.1, U200.1 (Z)
- new net: D200.A, R200.2, U201.3 (+)
- new net: R300.1, R307.2, R308.1, U300.4 (ADJ)
- new net: C301.1, Q300.3 (D), Q301.4 (E), R300.2, R310.1, U300.5 (OUT)
- new net: R423.2, R431.2, U413.4 (B), U415.4 (O)
- new net: LED900.A, LED904.A, R900.1
- new net: LED902.A, LED906.A, R902.1
- new net: RN500.8 (2), U500.4 (Y)
- new net: R422.2, R427.2, U412.4 (B), U414.4 (O)
- new net: R410.2, R425.2, U404.4 (B), U406.4 (O)
- new net: R416.2, R426.2, U408.4 (B), U410.4 (O)
- new net: RN500.5 (2), U500.8 (Y)
- new net: R307.1, R309.2, U301.1 (OUT)
- new net: RN500.7 (2), U500.1 (Y)
- new net: C101.1, U100.23 (OSC_IN), XTAL100.2
- new net: C100.1, U100.24 (OSC_OUT), XTAL100.1
- new net: J1.CC1, R803.1
- new net: R309.1, U301.4 (-)
- new net: J1.CC2, R804.1
- new net: RN501.3 (1), U501.1 (Y)
- new net: J1.VBUS@1 (VBUS), J1.VBUS@2 (VBUS), L800.2 (1)
- new net: RN501.1, U501.8 (Y)
- new net: RN501.4 (1), U501.4 (Y)
- new net: U700.133 (NC), U700.35 (NC), U700.36 (NC), U700.50 (NC), U700.51 (NC), U700.58 (NC), U700.77 (NC)
