File: PROJ/SPAR/10653/STAN/01/src/kicadBoard.kicad_sch (KiCad schematic)
At the start: 34 parts

Commit message: Quickly Adding Everything
Parts:
- removed C1, C10, C2, C3, C8, C9: (no value), symbol eagleSchem-eagle-import:CAP0603-CAP
- removed C4, C5, C6, C7: (no value), symbol eagleSchem-eagle-import:CAP_POL1206
- removed JP1: (no value), symbol eagleSchem-eagle-import:LOGO-SFENEW
- removed JP10, JP11, JP12, JP6: (no value), symbol eagleSchem-eagle-import:STAND-OFF
- removed JP13: (no value), symbol eagleSchem-eagle-import:LOGO-SFENW2
- removed JP2, JP3: (no value), symbol eagleSchem-eagle-import:FIDUCIAL1X2
- removed JP4, JP5, JP8: (no value), symbol eagleSchem-eagle-import:M02PTH
- removed JP7: (no value), symbol eagleSchem-eagle-import:M08
- removed JP9: (no value), symbol eagleSchem-eagle-import:M06SIP
- removed LED1: (no value), symbol eagleSchem-eagle-import:LED0603
- removed R1, R2, R3, R4: (no value), symbol eagleSchem-eagle-import:RESISTOR0603-RES
- removed S1: (no value), symbol eagleSchem-eagle-import:SWITCH-SPSTSMD
- removed U$10: (no value), symbol eagleSchem-eagle-import:CREATIVE_COMMONS
- removed U$14: (no value), symbol eagleSchem-eagle-import:OSHW-LOGOL
- removed U1: (no value), symbol eagleSchem-eagle-import:ISD1900ISD1932
- removed U2: (no value), symbol eagleSchem-eagle-import:MICELECTRET_SMD
- removed U3: (no value), symbol eagleSchem-eagle-import:AUDIO-JACK2SMD
- added C1, C10, C2, C3, C8, C9: (no value), symbol schematicEagle-eagle-import:CAP0603-CAP
- added C4, C5, C6, C7: (no value), symbol schematicEagle-eagle-import:CAP_POL1206
- added JP1: (no value), symbol schematicEagle-eagle-import:LOGO-SFENEW
- added JP10, JP11, JP12, JP6: (no value), symbol schematicEagle-eagle-import:STAND-OFF
- added JP13: (no value), symbol schematicEagle-eagle-import:LOGO-SFENW2
- added JP2, JP3: (no value), symbol schematicEagle-eagle-import:FIDUCIAL1X2
- added JP4, JP5, JP8: (no value), symbol schematicEagle-eagle-import:M02PTH
- added JP7: (no value), symbol schematicEagle-eagle-import:M08
- added JP9: (no value), symbol schematicEagle-eagle-import:M06SIP
- added LED1: (no value), symbol schematicEagle-eagle-import:LED0603
- added R1, R2, R3, R4: (no value), symbol schematicEagle-eagle-import:RESISTOR0603-RES
- added S1: (no value), symbol schematicEagle-eagle-import:SWITCH-SPSTSMD
- added U$10: (no value), symbol schematicEagle-eagle-import:CREATIVE_COMMONS
- added U$14: (no value), symbol schematicEagle-eagle-import:OSHW-LOGOL
- added U1: (no value), symbol schematicEagle-eagle-import:ISD1900ISD1932
- added U2: (no value), symbol schematicEagle-eagle-import:MICELECTRET_SMD
- added U3: (no value), symbol schematicEagle-eagle-import:AUDIO-JACK2SMD
Connections:
- net 5V: now also C1.1, C2.1, C3.1, C4.A (+), C5.A (+), C6.A (+), JP4.2, LED1.A, R2.2, S1.3 (S), U1.14 (VCCP), U1.21 (VCCA), U1.28 (VCCD)
- net AGC: now also C7.A (+), JP9.2, U1.17 (AGC)
- net E0: now also JP7.8, U1.7 (E0/_M5)
- net E1: now also JP7.7, U1.9 (E1/_M6)
- net E2: now also JP7.6, U1.10 (E2/_M7)
- net E3: now also JP7.5, U1.11 (E3/_M8)
- net FMC1: now also JP9.6, U1.6 (_PLAYL/FMC1)
- net FMC2: now also JP9.5, U1.23 (_PLAYE/FMC2)
- net FT: now also JP9.1, U1.26 (_FT)
- net GND: now also C1.2, C10.2, C2.2, C3.2, C4.C (-), C5.C (-), C6.C (-), C7.C (-), JP4.1, S1.1 (O), U1.1 (VSSD), U1.12 (VSSP2), U1.16 (VSSP1), U1.8 (VSSA)
- net LED: now also JP8.1, R1.1, R4.1, U1.22 (_LED)
- net MIC+: now also C8.1, U1.18 (MIC+)
- net MIC-: now also C9.2, U1.19 (MIC-)
- net MODE: now also S1.2 (P), U1.27 (ADDR/_DRCT)
- net REC: now also JP9.4, U1.24 (_REC)
- net ROSC: now also JP9.3, U1.20 (ROSC)
- net S0: now also JP7.4, U1.2 (S0/_M1)
- net S1: now also JP7.3, U1.3 (S1/_M2)
- net S2: now also JP7.2, U1.4 (S2/_M3)
- net S3: now also JP7.1, U1.5 (S3/_M4)
- net SP+: now also JP5.1, U1.15 (SP+), U3.RING, U3.TIP
- net SP-: now also JP5.2, U1.13 (SP-), U3.SLEEVE
- net XCLK: now also JP8.2, U1.25 (XCLK/FMC3)
- new net: C8.2, R3.1, U2.1
- new net: C10.1, R2.1, R3.2
- new net: C9.1, R4.2, U2.2
- new net: LED1.C, R1.2
