File: PROJ/SPAR/10967/STAN/01/src/kicadBoard.kicad_sch (KiCad schematic)
At the start: 12 parts

Commit message: Quickly Adding Everything
Parts:
- removed C1: (no value), symbol eagleSchem-eagle-import:CAP_POL1206
- removed C2: (no value), symbol eagleSchem-eagle-import:CAP_POL3528
- removed D1: (no value), symbol eagleSchem-eagle-import:DIODESMA
- removed FID1, FID2: (no value), symbol eagleSchem-eagle-import:FIDUCIAL1X2
- removed FRAME1: (no value), symbol eagleSchem-eagle-import:FRAME-LETTER
- removed JP1: (no value), symbol eagleSchem-eagle-import:M03PTH
- removed JP2: (no value), symbol eagleSchem-eagle-import:LOGO-SFESK
- removed L1: (no value), symbol eagleSchem-eagle-import:INDUCTORCR54
- removed U$1: (no value), symbol eagleSchem-eagle-import:OSHW-LOGOS
- removed U$2: (no value), symbol eagleSchem-eagle-import:CREATIVE_COMMONS
- removed U1: (no value), symbol eagleSchem-eagle-import:V_REG_NCP1400SOT23-5
- added C1: (no value), symbol schematicEagle-eagle-import:CAP_POL1206
- added C2: (no value), symbol schematicEagle-eagle-import:CAP_POL3528
- added D1: (no value), symbol schematicEagle-eagle-import:DIODESMA
- added FID1, FID2: (no value), symbol schematicEagle-eagle-import:FIDUCIAL1X2
- added FRAME1: (no value), symbol schematicEagle-eagle-import:FRAME-LETTER
- added JP1: (no value), symbol schematicEagle-eagle-import:M03PTH
- added JP2: (no value), symbol schematicEagle-eagle-import:LOGO-SFESK
- added L1: (no value), symbol schematicEagle-eagle-import:INDUCTORCR54
- added U$1: (no value), symbol schematicEagle-eagle-import:OSHW-LOGOS
- added U$2: (no value), symbol schematicEagle-eagle-import:CREATIVE_COMMONS
- added U1: (no value), symbol schematicEagle-eagle-import:V_REG_NCP1400SOT23-5
Connections:
- net GND: now also C1.C (-), C2.C (-), JP1.1, U1.4 (GND)
- net VIN: now also C1.A (+), JP1.3, L1.P$1 (1)
- net VOUT: now also C2.A (+), D1.C, JP1.2, U1.1 (EN), U1.2 (OUT)
- new net: D1.A, L1.P$2 (2), U1.5 (LX)
