File: PROJ/SPAR/11018/STAN/01/src/kicadBoard.kicad_sch (KiCad schematic)
At the start: 28 parts

Commit message: Quickly Adding Everything
Parts:
- removed C1: (no value), symbol eagleSchem-eagle-import:CAP_POL1206
- removed C2, C3, C4: (no value), symbol eagleSchem-eagle-import:CAP0402-CAP
- removed JP1, JP2, JP3, JP4, JP5, JP6: (no value), symbol eagleSchem-eagle-import:M01PTH
- removed JP7, JP8: (no value), symbol eagleSchem-eagle-import:FIDUCIALUFIDUCIAL
- removed LED1: (no value), symbol eagleSchem-eagle-import:LED0603
- removed R1, R2: (no value), symbol eagleSchem-eagle-import:RESISTOR0402-RES
- removed S2: (no value), symbol eagleSchem-eagle-import:SWITCH-MOMENTARY-2SMD
- removed SJ1, SJ3, SJ4: (no value), symbol eagleSchem-eagle-import:SOLDERJUMPERTRACE
- removed SJ2: (no value), symbol eagleSchem-eagle-import:SOLDERJUMPERNO
- removed U$1: (no value), symbol eagleSchem-eagle-import:OSHW-LOGOS
- removed U$3: (no value), symbol eagleSchem-eagle-import:CREATIVE_COMMONS
- removed U$7, U$8: (no value), symbol eagleSchem-eagle-import:LOGO-SFENEW
- removed U1: (no value), symbol eagleSchem-eagle-import:V_REG_LDOSMD
- removed U2: (no value), symbol eagleSchem-eagle-import:RFM22SMD
- removed U3: (no value), symbol eagleSchem-eagle-import:HEX_CONVERTER
- removed U4: (no value), symbol eagleSchem-eagle-import:ARDUINO_SHIELDNOHOLES
- added C1: (no value), symbol schematicEagle-eagle-import:CAP_POL1206
- added C2, C3, C4: (no value), symbol schematicEagle-eagle-import:CAP0402-CAP
- added JP1, JP2, JP3, JP4, JP5, JP6: (no value), symbol schematicEagle-eagle-import:M01PTH
- added JP7, JP8: (no value), symbol schematicEagle-eagle-import:FIDUCIALUFIDUCIAL
- added LED1: (no value), symbol schematicEagle-eagle-import:LED0603
- added R1, R2: (no value), symbol schematicEagle-eagle-import:RESISTOR0402-RES
- added S2: (no value), symbol schematicEagle-eagle-import:SWITCH-MOMENTARY-2SMD
- added SJ1, SJ3, SJ4: (no value), symbol schematicEagle-eagle-import:SOLDERJUMPERTRACE
- added SJ2: (no value), symbol schematicEagle-eagle-import:SOLDERJUMPERNO
- added U$1: (no value), symbol schematicEagle-eagle-import:OSHW-LOGOS
- added U$3: (no value), symbol schematicEagle-eagle-import:CREATIVE_COMMONS
- added U$7, U$8: (no value), symbol schematicEagle-eagle-import:LOGO-SFENEW
- added U1: (no value), symbol schematicEagle-eagle-import:V_REG_LDOSMD
- added U2: (no value), symbol schematicEagle-eagle-import:RFM22SMD
- added U3: (no value), symbol schematicEagle-eagle-import:HEX_CONVERTER
- added U4: (no value), symbol schematicEagle-eagle-import:ARDUINO_SHIELDNOHOLES
Connections:
- net 3.3V: now also C1.A (+), C2.1, C3.1, JP5.1, R2.2, U1.5 (OUT), U2.5 (VCC), U3.1 (VCC)
- net 3V-GPIO2: now also JP4.1, SJ3.2, U2.8 (GPIO2)
- net 3V-MISO: now also U2.10 (SDO), U4.D12
- net 3V-MOSI: now also U2.11 (SDI), U3.15 (6Y)
- net 3V-NIRQ: now also JP6.1, SJ4.2, U2.14 (NIRQ)
- net 3V-NSEL: now also U2.13 (NSEL), U3.10 (4Y)
- net 3V-SCK: now also U2.12 (SCLK), U3.12 (5Y)
- net 5V-MOSI: now also U3.14 (6A), U4.D11 (*D11)
- net 5V-NSEL: now also JP1.1, SJ1.2, U3.9 (4A)
- net 5V-SCK: now also U3.11 (5A), U4.D13
- net GND: now also C1.C (-), C2.2, C3.2, C4.2, LED1.C, R1.1, S2.1, U1.2 (GND), U2.16 (GND@3), U2.2 (GND@1), U2.9 (GND@2), U3.8 (GND), U4.GND@0, U4.GND@1, U4.GND@2
- net SDN: now also JP3.1, SJ2.1
- net VCC: now also U1.1 (IN), U1.3 (EN), U4.5V
- new net: SJ1.1, U4.D10 (*D10)
- new net: SJ4.1, U4.D2
- new net: SJ3.1, U4.D3 (*D3)
- new net: S2.3 (2), U4.RES
- new net: LED1.A, R2.1
- new net: C4.1, U1.4 (BP)
- new net: JP2.1, U2.1 (ANT)
- new net: R1.2, SJ2.2, U2.15 (SDN)
- new net: U2.3 (RXANT), U2.7 (GPIO1)
- new net: U2.4 (TXANT), U2.6 (GPIO0)
