File: PROJ/SPAR/11447/STAN/01/src/kicadBoard.kicad_sch (KiCad schematic)
At the start: 25 parts

Commit message: Quickly Adding Everything
Parts:
- removed C1, C4: (no value), symbol eagleSchem-eagle-import:0.1UF-25V(+80/-20%)(0603)
- removed C2, C3: (no value), symbol eagleSchem-eagle-import:1.0UF-16V-10%(0603)
- removed D1: (no value), symbol eagleSchem-eagle-import:RB751
- removed D2: (no value), symbol eagleSchem-eagle-import:DIODE-SCHOTTKY
- removed FID1, FID2: (no value), symbol eagleSchem-eagle-import:FIDUCIAL1X2
- removed FRAME1: (no value), symbol eagleSchem-eagle-import:FRAME-LETTER
- removed J1: (no value), symbol eagleSchem-eagle-import:AVR_SPI_PRG_6PTH
- removed JP1: (no value), symbol eagleSchem-eagle-import:FTDI_DEVICE
- removed JP2: (no value), symbol eagleSchem-eagle-import:M02-JST-2MM-SMT
- removed JP3: (no value), symbol eagleSchem-eagle-import:M03PTH
- removed JP4: (no value), symbol eagleSchem-eagle-import:LOGO-SFENW2
- removed JP5: (no value), symbol eagleSchem-eagle-import:M02PTH
- removed JP6: (no value), symbol eagleSchem-eagle-import:LOGO-SFENEW
- removed JP7: (no value), symbol eagleSchem-eagle-import:M05PTH
- removed Q1: (no value), symbol eagleSchem-eagle-import:IRF7509
- removed R1, R2: (no value), symbol eagleSchem-eagle-import:1MOHM1/10W1%(0603)
- removed R3, R4: (no value), symbol eagleSchem-eagle-import:10K-1%RES-00824
- removed U1: (no value), symbol eagleSchem-eagle-import:ADXL362ADXL362-1{colon}1
- removed U2: (no value), symbol eagleSchem-eagle-import:ATTINY2313A
- removed U3: (no value), symbol eagleSchem-eagle-import:ADP160
- added C1, C4: (no value), symbol schematicEagle-eagle-import:0.1UF-25V(+80/-20%)(0603)
- added C2, C3: (no value), symbol schematicEagle-eagle-import:1.0UF-16V-10%(0603)
- added D1: (no value), symbol schematicEagle-eagle-import:RB751
- added D2: (no value), symbol schematicEagle-eagle-import:DIODE-SCHOTTKY
- added FID1, FID2: (no value), symbol schematicEagle-eagle-import:FIDUCIAL1X2
- added FRAME1: (no value), symbol schematicEagle-eagle-import:FRAME-LETTER
- added J1: (no value), symbol schematicEagle-eagle-import:AVR_SPI_PRG_6PTH
- added JP1: (no value), symbol schematicEagle-eagle-import:FTDI_DEVICE
- added JP2: (no value), symbol schematicEagle-eagle-import:M02-JST-2MM-SMT
- added JP3: (no value), symbol schematicEagle-eagle-import:M03PTH
- added JP4: (no value), symbol schematicEagle-eagle-import:LOGO-SFENW2
- added JP5: (no value), symbol schematicEagle-eagle-import:M02PTH
- added JP6: (no value), symbol schematicEagle-eagle-import:LOGO-SFENEW
- added JP7: (no value), symbol schematicEagle-eagle-import:M05PTH
- added Q1: (no value), symbol schematicEagle-eagle-import:IRF7509
- added R1, R2: (no value), symbol schematicEagle-eagle-import:1MOHM1/10W1%(0603)
- added R3, R4: (no value), symbol schematicEagle-eagle-import:10K-1%RES-00824
- added U1: (no value), symbol schematicEagle-eagle-import:ADXL362ADXL362-1{colon}1
- added U2: (no value), symbol schematicEagle-eagle-import:ATTINY2313A
- added U3: (no value), symbol schematicEagle-eagle-import:ADP160
Connections:
- net 3.3V: now also C1.1, C3.1, C4.1, J1.2, R3.1, R4.1, U1.P$1 (VDDIO), U1.P$14 (VS), U2.20 (VCC), U3.5 (VOUT)
- net ACTIVE: now also D2.A, U2.8 (PD4)
- net GND: now also C1.2, C2.2, C3.2, C4.2, J1.6, JP1.P$6 (GND), JP2.1 (2), JP3.3, JP5.2, Q1.1 (S), R2.1, U1.P$12 (GND), U1.P$13 (GND), U1.P$16 (GND), U2.10 (GND), U3.2 (GND)
- net INT1: now also U1.P$11 (INT1), U2.7 (PD3/INT1)
- net MISO: now also J1.1, U1.P$6 (MOSI), U2.18 (PB6/MISO/DO)
- net MOSI: now also J1.4, U1.P$7 (MISO), U2.17 (PB5/MOSI/SDA/DI)
- net OVERRIDE: now also D1.A, JP3.1
- net RESET: now also J1.5, R3.2, U2.1 (PA2/~{RESET})
- net RXI: now also JP1.P$3 (RXI), R4.2, U2.2 (PD0/RXD), U2.6 (PD2/INT0)
- net SCK: now also J1.3, U1.P$4 (SCLK), U2.19 (PB7/SCK/SCL)
- net TXO: now also JP1.P$2 (TXO), U2.3 (PD1/TXD)
- net VOUT: now also JP3.2, Q1.5 (D), Q1.6 (D)
- net V_BATT: now also C2.1, JP2.2 (1), JP5.1, Q1.3 (S), R1.1, U3.1 (VIN), U3.3 (EN)
- new net: D1.C, D2.C, Q1.2 (G), R2.2
- new net: Q1.4 (G), Q1.7 (D), Q1.8 (D), R1.2
- new net: JP7.5, U2.11 (PD6)
- new net: JP7.4, U2.12 (PB0)
- new net: JP7.3, U2.13 (PB1)
- new net: JP7.2, U2.14 (PB2)
- new net: JP7.1, U2.15 (PB3)
- new net: U1.P$8 (~{CS}), U2.16 (PB4)
