File: PROJ/SPAR/11468/STAN/01/src/kicadBoard.kicad_sch (KiCad schematic)
At the start: 10 parts

Commit message: Quickly Adding Everything
Parts:
- removed FRAME1: (no value), symbol eagleSchem-eagle-import:FRAME-LETTER
- removed JP2, JP3: (no value), symbol eagleSchem-eagle-import:FIDUCIALUFIDUCIAL
- removed JP4: (no value), symbol eagleSchem-eagle-import:M11PTH
- removed LOGO0: (no value), symbol eagleSchem-eagle-import:LOGO-SFENEW
- removed SJ1: (no value), symbol eagleSchem-eagle-import:SOLDERJUMPERTRACE
- removed U$2: (no value), symbol eagleSchem-eagle-import:OSHW-LOGOS
- removed U$4: (no value), symbol eagleSchem-eagle-import:SFE_LOGO_FLAME.2_INCH
- removed U1: (no value), symbol eagleSchem-eagle-import:SD_CARD_SOCKET
- removed U2: (no value), symbol eagleSchem-eagle-import:SD_MMC_CARDSD_PCB
- added FRAME1: (no value), symbol schematicEagle-eagle-import:FRAME-LETTER
- added JP2, JP3: (no value), symbol schematicEagle-eagle-import:FIDUCIALUFIDUCIAL
- added JP4: (no value), symbol schematicEagle-eagle-import:M11PTH
- added LOGO0: (no value), symbol schematicEagle-eagle-import:LOGO-SFENEW
- added SJ1: (no value), symbol schematicEagle-eagle-import:SOLDERJUMPERTRACE
- added U$2: (no value), symbol schematicEagle-eagle-import:OSHW-LOGOS
- added U$4: (no value), symbol schematicEagle-eagle-import:SFE_LOGO_FLAME.2_INCH
- added U1: (no value), symbol schematicEagle-eagle-import:SD_CARD_SOCKET
- added U2: (no value), symbol schematicEagle-eagle-import:SD_MMC_CARDSD_PCB
Connections:
- net CD: now also JP4.5, U1.CD
- net CLK: now also JP4.7, U1.5 (CLK), U2.5 (CLK)
- net CMD: now also JP4.3, U1.2 (CMD), U2.2 (CMD)
- net D0: now also JP4.9, U1.7 (DAT0), U2.7 (DAT0)
- net D1: now also JP4.10, U1.8 (DAT1), U2.8 (DAT1)
- net D2: now also JP4.1, U1.9 (DAT2), U2.9 (DAT2)
- net D3: now also JP4.2, U1.1 (CD/DAT3), U2.1 (CD/DAT3)
- net GND: now also JP4.4, SJ1.1, U1.3 (VSS1), U1.SH@1, U1.SH@2, U2.3 (VSS1)
- net VCC: now also JP4.6, U1.4 (VDD), U2.4 (VDD)
- net VSS2: now also JP4.8, SJ1.2, U1.6 (VSS2), U2.6 (VSS2)
- net WP: now also JP4.11, U1.WP
