File: PROJ/SPAR/12581/STAN/01/src/kicadBoard.kicad_sch (KiCad schematic)
At the start: 24 parts

Commit message: Quickly Adding Everything
Parts:
- removed C1, C5: (no value), symbol eagleSchem-eagle-import:CAP0603-CAP
- removed C2, C3: (no value), symbol eagleSchem-eagle-import:CAP_POL1206
- removed C4: (no value), symbol eagleSchem-eagle-import:CAP_POL3528
- removed FRAME1: (no value), symbol eagleSchem-eagle-import:FRAME-LETTER
- removed JP1, JP3: (no value), symbol eagleSchem-eagle-import:FIDUCIALUFIDUCIAL
- removed JP2: (no value), symbol eagleSchem-eagle-import:M06SMD
- removed LOGO1: (no value), symbol eagleSchem-eagle-import:OSHW-LOGOS
- removed Q1, Q2: (no value), symbol eagleSchem-eagle-import:MOSFET-NCHANNELSMD
- removed R1, R2, R3, R4, R5, R6, R7: (no value), symbol eagleSchem-eagle-import:RESISTOR0603-RES
- removed U$1: (no value), symbol eagleSchem-eagle-import:LOGO-SFENEW
- removed U$2: (no value), symbol eagleSchem-eagle-import:REVISION
- removed U1: (no value), symbol eagleSchem-eagle-import:V_REG_317SMD
- removed U2: (no value), symbol eagleSchem-eagle-import:BLUETOOTH-RN41{dblquote}
- removed U3: (no value), symbol eagleSchem-eagle-import:V_REG_LDOSMD
- added C1, C5: (no value), symbol schematicEagle-eagle-import:CAP0603-CAP
- added C2, C3: (no value), symbol schematicEagle-eagle-import:CAP_POL1206
- added C4: (no value), symbol schematicEagle-eagle-import:CAP_POL3528
- added FRAME1: (no value), symbol schematicEagle-eagle-import:FRAME-LETTER
- added JP1, JP3: (no value), symbol schematicEagle-eagle-import:FIDUCIALUFIDUCIAL
- added JP2: (no value), symbol schematicEagle-eagle-import:M06SMD
- added LOGO1: (no value), symbol schematicEagle-eagle-import:OSHW-LOGOS
- added Q1, Q2: (no value), symbol schematicEagle-eagle-import:MOSFET-NCHANNELSMD
- added R1, R2, R3, R4, R5, R6, R7: (no value), symbol schematicEagle-eagle-import:RESISTOR0603-RES
- added U$1: (no value), symbol schematicEagle-eagle-import:LOGO-SFENEW
- added U$2: (no value), symbol schematicEagle-eagle-import:REVISION
- added U1: (no value), symbol schematicEagle-eagle-import:V_REG_317SMD
- added U2: (no value), symbol schematicEagle-eagle-import:BLUETOOTH-RN41{dblquote}
- added U3: (no value), symbol schematicEagle-eagle-import:V_REG_LDOSMD
Connections:
- net DD: now also Q2.2 (S), R3.1, U2.4 (PIO7)
- net DD_5V: now also JP2.5, Q2.3 (D), R4.1
- net GND: now also C1.2, C2.C (-), C3.C (-), C4.C (-), C5.2, JP2.3, R5.1, U2.1 (GND), U2.12 (GND1), U2.28 (GND2), U2.29 (GND3), U3.2 (GND)
- net RX: now also R7.1, U2.13 (UARTRX)
- net RX_5V: now also JP2.4, R7.2
- net TX: now also Q1.2 (S), R1.1, U2.14 (UARTTX)
- net TX_5V: now also JP2.2, Q1.3 (D), R2.1
- net VCC: now also C1.1, C2.A (+), C3.A (+), C4.A (+), C5.1, JP2.1, Q1.1 (G), Q2.1 (G), R1.2, R2.2, R3.2, R4.2, R6.2, U1.2 (OUT), U1.3 (IN), U2.11 (VDD), U3.1 (IN), U3.3 (EN), U3.5 (OUT)
- new net: R5.2, R6.1, U1.1 (ADJ)
