File: PROJ/SPAR/12634/STAN/01/src/kicadBoard.kicad_sch (KiCad schematic)
At the start: 44 parts

Commit message: Quickly Adding Everything
Parts:
- removed BAT1, BAT2: (no value), symbol eagleSchem-eagle-import:BATTERYAA-KIT
- removed C1, C2: (no value), symbol eagleSchem-eagle-import:0.1UF-50V-20%(PTH)KIT-EZ
- removed FRAME1: (no value), symbol eagleSchem-eagle-import:FRAME-LETTER
- removed JP1: (no value), symbol eagleSchem-eagle-import:M06-SFENOSILK
- removed JP2, JP5, JP6, JP7: (no value), symbol eagleSchem-eagle-import:STAND-OFF
- removed JP3: (no value), symbol eagleSchem-eagle-import:AVR_SPI_PRG_6NS
- removed JP4: (no value), symbol eagleSchem-eagle-import:M09
- removed LED0, LED1, LED2, LED3, LED4, LED5: (no value), symbol eagleSchem-eagle-import:LED5MM-KIT
- removed R1: (no value), symbol eagleSchem-eagle-import:10KOHM1/6W5%(PTH)KIT
- removed R2, R3, R4, R5: (no value), symbol eagleSchem-eagle-import:RESISTORAX-0.3-KIT
- removed S1, S2: (no value), symbol eagleSchem-eagle-import:SWITCH-SPDTKIT
- removed SG1: (no value), symbol eagleSchem-eagle-import:BUZZERPTH-KIT
- removed SJ1, SJ10, SJ11, SJ12, SJ2, SJ3, SJ4, SJ5, SJ6, SJ7, SJ8, SJ9: (no value), symbol eagleSchem-eagle-import:SOLDERJUMPER_2WAYS
- removed U$1: (no value), symbol eagleSchem-eagle-import:LOGO-SFENEW
- removed U$3: (no value), symbol eagleSchem-eagle-import:OSHW-LOGOS
- removed U$4, U$5, U$6: (no value), symbol eagleSchem-eagle-import:TILT_SENSORV5
- removed U$7: (no value), symbol eagleSchem-eagle-import:AVR-MEGA8-P-KEYED-14
- added BAT1, BAT2: (no value), symbol schematicEagle-eagle-import:BATTERYAA-KIT
- added C1, C2: (no value), symbol schematicEagle-eagle-import:0.1UF-50V-20%(PTH)KIT-EZ
- added FRAME1: (no value), symbol schematicEagle-eagle-import:FRAME-LETTER
- added JP1: (no value), symbol schematicEagle-eagle-import:M06-SFENOSILK
- added JP2, JP5, JP6, JP7: (no value), symbol schematicEagle-eagle-import:STAND-OFF
- added JP3: (no value), symbol schematicEagle-eagle-import:AVR_SPI_PRG_6NS
- added JP4: (no value), symbol schematicEagle-eagle-import:M09
- added LED0, LED1, LED2, LED3, LED4, LED5: (no value), symbol schematicEagle-eagle-import:LED5MM-KIT
- added R1: (no value), symbol schematicEagle-eagle-import:10KOHM1/6W5%(PTH)KIT
- added R2, R3, R4, R5: (no value), symbol schematicEagle-eagle-import:RESISTORAX-0.3-KIT
- added S1, S2: (no value), symbol schematicEagle-eagle-import:SWITCH-SPDTKIT
- added SG1: (no value), symbol schematicEagle-eagle-import:BUZZERPTH-KIT
- added SJ1, SJ10, SJ11, SJ12, SJ2, SJ3, SJ4, SJ5, SJ6, SJ7, SJ8, SJ9: (no value), symbol schematicEagle-eagle-import:SOLDERJUMPER_2WAYS
- added U$1: (no value), symbol schematicEagle-eagle-import:LOGO-SFENEW
- added U$3: (no value), symbol schematicEagle-eagle-import:OSHW-LOGOS
- added U$4, U$5, U$6: (no value), symbol schematicEagle-eagle-import:TILT_SENSORV5
- added U$7: (no value), symbol schematicEagle-eagle-import:AVR-MEGA8-P-KEYED-14
Connections:
- net 3.3V: now also C1.2, JP3.2, JP4.1, R1.P$2 (2), R2.P$2 (2), R3.P$2 (2), R4.P$2 (2), R5.P$2 (2), S1.3 (S), U$7.20 (AVCC), U$7.21 (AREF), U$7.7 (VCC)
- net A3: now also JP4.5, U$7.26 (PC3(ADC3))
- net A4: now also JP4.6, U$7.27 (PC4(ADC4/SDA))
- net A5: now also JP4.7, U$7.28 (PC5(ADC5/SCL))
- net D9: now also JP4.3, U$7.15 (PB1(OC1A))
- net DTR: now also C2.1, JP1.1
- net GND: now also BAT1.GND@1 (-), C1.1, JP1.5, JP1.6, JP3.6, JP4.2, U$4.D-, U$4.E-, U$5.D-, U$5.E-, U$6.D-, U$6.E-, U$7.22 (GND@2), U$7.8 (GND@1)
- net LED0: now also SJ1.3, SJ2.1, U$7.4 (PD2(INT0))
- net LED1: now also SJ3.3, SJ4.1, U$7.5 (PD3(INT1))
- net LED2: now also SJ5.3, SJ6.1, U$7.6 (PD4(XCK/T0))
- net LED3: now also SJ7.3, SJ8.1, U$7.11 (PD5(T1))
- net LED4: now also SJ10.1, SJ9.3, U$7.12 (PD6(AIN0))
- net LED5: now also SJ11.3, SJ12.1, U$7.13 (PD7(AIN1))
- net LEDS-GND: now also SJ1.1, SJ10.3, SJ11.1, SJ12.3, SJ2.3, SJ3.1, SJ4.3, SJ5.1, SJ6.3, SJ7.1, SJ8.3, SJ9.1, U$7.16 (PB2(SS/OC1B))
- net MISO: now also JP3.1, SG1.+ (1), U$7.18 (PB4(MISO))
- net MOSI: now also JP3.4, JP4.4, U$7.17 (PB3(MOSI/OC2))
- net PB6: now also JP4.9, U$7.9 (PB6(XTAL1/TOSC1))
- net PB7: now also JP4.8, U$7.10 (PB7(XTAL2/TOSC2))
- net RESET: now also C2.2, JP3.5, R1.P$1 (1), U$7.1 (PC6(/RESET))
- net RX-I: now also JP1.3, U$7.2 (PD0(RXD))
- net SCK: now also JP3.3, S2.1 (O), U$7.19 (PB5(SCK))
- net TILT-0: now also R5.P$1 (1), U$4.D+, U$7.23 (PC0(ADC0))
- net TILT-1: now also R4.P$1 (1), U$5.D+, U$7.24 (PC1(ADC1))
- net TILT-2: now also R3.P$1 (1), U$6.D+, U$7.25 (PC2(ADC2))
- net TX-O: now also JP1.2, U$7.3 (PD1(TXD))
- new net: LED3.A, SJ7.2
- new net: LED3.K (C), SJ8.2
- new net: LED0.A, SJ1.2
- new net: R2.P$1 (1), U$4.E+, U$5.E+, U$6.E+
- new net: BAT2.PWR@1 (+), S1.2 (P)
- new net: LED5.A, SJ11.2
- new net: LED5.K (C), SJ12.2
- new net: LED0.K (C), SJ2.2
- new net: S2.2 (P), SG1.- (2)
- new net: LED1.A, SJ3.2
- new net: LED2.A, SJ5.2
- new net: LED4.K (C), SJ10.2
- new net: LED1.K (C), SJ4.2
- new net: LED2.K (C), SJ6.2
- new net: LED4.A, SJ9.2
- new net: BAT1.PWR@1 (+), BAT2.GND@1 (-)
