File: PROJ/SPAR/12761/STAN/01/src/kicadBoard.kicad_sch (KiCad schematic)
At the start: 23 parts

Commit message: Quickly Adding Everything
Parts:
- removed C1, C2: (no value), symbol eagleSchem-eagle-import:0.1UF-25V-5%(0603)
- removed C3: (no value), symbol eagleSchem-eagle-import:10UF-6.3V-20%(0603)
- removed FRAME1: (no value), symbol eagleSchem-eagle-import:FRAME-LETTER
- removed J1: (no value), symbol eagleSchem-eagle-import:AVR_SPI_PRG_6NS
- removed JP1: (no value), symbol eagleSchem-eagle-import:SFE_LOGO_NAME_FLAME.1_INCH
- removed JP2, JP3: (no value), symbol eagleSchem-eagle-import:FIDUCIAL1X2
- removed JP4: (no value), symbol eagleSchem-eagle-import:M08
- removed JP5: (no value), symbol eagleSchem-eagle-import:M10{dblquote}
- removed JP6: (no value), symbol eagleSchem-eagle-import:M06SIP
- removed JP7: (no value), symbol eagleSchem-eagle-import:M081X08
- removed LED1: (no value), symbol eagleSchem-eagle-import:LED0603
- removed LOGO1: (no value), symbol eagleSchem-eagle-import:OSHW-LOGOM
- removed LOGO2: (no value), symbol eagleSchem-eagle-import:SFE_LOGO_FLAME.6_INCH
- removed R1: (no value), symbol eagleSchem-eagle-import:RESISTOR0603-RES
- removed S1: (no value), symbol eagleSchem-eagle-import:TAC_SWITCHSMD
- removed SJ1, SJ2: (no value), symbol eagleSchem-eagle-import:SOLDERJUMPERNC
- removed U$1: (no value), symbol eagleSchem-eagle-import:REVISION
- removed U1: (no value), symbol eagleSchem-eagle-import:USD-SOCKETNEW
- removed U2: (no value), symbol eagleSchem-eagle-import:ARDUINO_R3_SHIELDNOLABELS
- removed U3: (no value), symbol eagleSchem-eagle-import:HEX_CONVERTER
- added C1, C2: (no value), symbol schematicEagle-eagle-import:0.1UF-25V-5%(0603)
- added C3: (no value), symbol schematicEagle-eagle-import:10UF-6.3V-20%(0603)
- added FRAME1: (no value), symbol schematicEagle-eagle-import:FRAME-LETTER
- added J1: (no value), symbol schematicEagle-eagle-import:AVR_SPI_PRG_6NS
- added JP1: (no value), symbol schematicEagle-eagle-import:SFE_LOGO_NAME_FLAME.1_INCH
- added JP2, JP3: (no value), symbol schematicEagle-eagle-import:FIDUCIAL1X2
- added JP4: (no value), symbol schematicEagle-eagle-import:M08
- added JP5: (no value), symbol schematicEagle-eagle-import:M10{dblquote}
- added JP6: (no value), symbol schematicEagle-eagle-import:M06SIP
- added JP7: (no value), symbol schematicEagle-eagle-import:M081X08
- added LED1: (no value), symbol schematicEagle-eagle-import:LED0603
- added LOGO1: (no value), symbol schematicEagle-eagle-import:OSHW-LOGOM
- added LOGO2: (no value), symbol schematicEagle-eagle-import:SFE_LOGO_FLAME.6_INCH
- added R1: (no value), symbol schematicEagle-eagle-import:RESISTOR0603-RES
- added S1: (no value), symbol schematicEagle-eagle-import:TAC_SWITCHSMD
- added SJ1, SJ2: (no value), symbol schematicEagle-eagle-import:SOLDERJUMPERNC
- added U$1: (no value), symbol schematicEagle-eagle-import:REVISION
- added U1: (no value), symbol schematicEagle-eagle-import:USD-SOCKETNEW
- added U2: (no value), symbol schematicEagle-eagle-import:ARDUINO_R3_SHIELDNOLABELS
- added U3: (no value), symbol schematicEagle-eagle-import:HEX_CONVERTER
Connections:
- net 3.3V: now also C1.1, C2.1, C3.1, JP7.4, LED1.A, U1.4 (VCC), U2.3.3V, U3.1 (VCC)
- net 5V: now also J1.2, JP7.5, U2.5V
- net A0: now also JP6.1, U2.A0
- net A1: now also JP6.2, U2.A1
- net A2: now also JP6.3, U2.A2
- net A3: now also JP6.4, U2.A3
- net A4: now also JP6.5, SJ1.2, U2.A4
- net A5: now also JP6.6, SJ2.2, U2.A5
- net AREF: now also JP5.8, U2.AREF
- net CS: now also JP5.1, U2.D8, U3.3 (1A)
- net D10: now also JP5.3, U2.D10 (*D10)
- net D2: now also JP4.3, U2.D2
- net D3: now also JP4.4, U2.D3 (*D3)
- net D4: now also JP4.5, U2.D4
- net D5: now also JP4.6, U2.D5 (*D5)
- net D6: now also JP4.7, U2.D6 (*D6)
- net D7: now also JP4.8, U2.D7
- net D9: now also JP5.2, U2.D9 (*D9)
- net GND: now also C1.2, C2.2, C3.2, J1.6, JP5.7, JP7.6, JP7.7, R1.1, S1.1, S1.2, U1.6 (GND), U1.CD1 (SHIELD@2), U1.CD2 (SHIELD@4), U1.GND1 (SHIELD@3), U1.GND3 (SHIELD@1), U2.GND@0, U2.GND@1, U2.GND@2, U3.8 (GND)
- net IOREF: now also JP7.2, U2.IOREF
- net MISO: now also J1.1, JP5.5, U1.7 (DO), U2.D12
- net MOSI: now also J1.4, JP5.4, U2.D11 (*D11), U3.5 (2A)
- net NC: now also JP7.1
- net RES: now also J1.5, JP7.3, S1.3, S1.4, U2.RES
- net RX: now also JP4.1, U2.RX
- net SCK: now also J1.3, JP5.6, U2.D13, U3.7 (3A)
- net SCL: now also JP5.10, SJ2.1, U2.SCL
- net SDA: now also JP5.9, SJ1.1, U2.SDA
- net TX: now also JP4.2, U2.TX
- net VIN: now also JP7.8, U2.VIN
- new net: LED1.C, R1.2
- new net: U1.2 (CS), U3.2 (1Y)
- new net: U1.3 (DI), U3.4 (2Y)
- new net: U1.5 (SCK), U3.6 (3Y)
