File: PROJ/SPAR/12916/STAN/01/src/kicadBoard.kicad_sch (KiCad schematic)
At the start: 15 parts

Commit message: Quickly Adding Everything
Parts:
- removed C1: (no value), symbol eagleSchem-eagle-import:0.1UF-25V(+80/-20%)(0603)
- removed C2: (no value), symbol eagleSchem-eagle-import:1.0UF-16V-10%(0603)
- removed FID1, FID2: (no value), symbol eagleSchem-eagle-import:FIDUCIAL1X2
- removed FRAME1: (no value), symbol eagleSchem-eagle-import:FRAME-LETTER
- removed JP1: (no value), symbol eagleSchem-eagle-import:M04PTH
- removed LOGO1: (no value), symbol eagleSchem-eagle-import:SFE_LOGO_FLAME.1_INCH
- removed LOGO2: (no value), symbol eagleSchem-eagle-import:SFE_LOGO_NAME_FLAME.1_INCH
- removed LOGO3: (no value), symbol eagleSchem-eagle-import:OSHW-LOGOS
- removed R1, R2: (no value), symbol eagleSchem-eagle-import:10KOHM1/10W1%(0603)0603
- removed SJ1: (no value), symbol eagleSchem-eagle-import:SOLDERJUMPER_2WAYPASTE1&2&3
- removed STANDOFF1, STANDOFF2: (no value), symbol eagleSchem-eagle-import:STAND-OFF
- removed U1: (no value), symbol eagleSchem-eagle-import:HMC6343A
- added C1: (no value), symbol schematicEagle-eagle-import:0.1UF-25V(+80/-20%)(0603)
- added C2: (no value), symbol schematicEagle-eagle-import:1.0UF-16V-10%(0603)
- added FID1, FID2: (no value), symbol schematicEagle-eagle-import:FIDUCIAL1X2
- added FRAME1: (no value), symbol schematicEagle-eagle-import:FRAME-LETTER
- added JP1: (no value), symbol schematicEagle-eagle-import:M04PTH
- added LOGO1: (no value), symbol schematicEagle-eagle-import:SFE_LOGO_FLAME.1_INCH
- added LOGO2: (no value), symbol schematicEagle-eagle-import:SFE_LOGO_NAME_FLAME.1_INCH
- added LOGO3: (no value), symbol schematicEagle-eagle-import:OSHW-LOGOS
- added R1, R2: (no value), symbol schematicEagle-eagle-import:10KOHM1/10W1%(0603)0603
- added SJ1: (no value), symbol schematicEagle-eagle-import:SOLDERJUMPER_2WAYPASTE1&2&3
- added STANDOFF1, STANDOFF2: (no value), symbol schematicEagle-eagle-import:STAND-OFF
- added U1: (no value), symbol schematicEagle-eagle-import:HMC6343A
Connections:
- net 3.3V: now also C1.1, C2.1, JP1.2, SJ1.2, U1.11 (VDD@11), U1.21 (VDD@21), U1.3 (VDD@3)
- net GND: now also C1.2, C2.2, JP1.1, U1.25 (GND@25), U1.29 (GND@29)
- net SCL: now also JP1.4, R1.1, U1.32 (SCL)
- net SDA: now also JP1.3, R2.1, U1.36 (SDA)
- new net: U1.22 (CS), U1.35 (CSC)
- new net: R1.2, SJ1.3
- new net: R2.2, SJ1.1
