File: PROJ/SPAR/12918/STAN/01/src/kicadBoard.kicad_sch (KiCad schematic)
At the start: 16 parts

Commit message: Quickly Adding Everything
Parts:
- removed C1: (no value), symbol eagleSchem-eagle-import:CAP0603-CAP
- removed FID1, FID2: (no value), symbol eagleSchem-eagle-import:FIDUCIAL1X2
- removed FRAME2: (no value), symbol eagleSchem-eagle-import:FRAME-LETTER
- removed GND0: (no value), symbol eagleSchem-eagle-import:LOGO-SFESK
- removed JP5: (no value), symbol eagleSchem-eagle-import:M04PTH
- removed JP6: (no value), symbol eagleSchem-eagle-import:M02PTH
- removed LOGO1: (no value), symbol eagleSchem-eagle-import:OSHW-LOGOS
- removed R1, R2, R3: (no value), symbol eagleSchem-eagle-import:RESISTOR0603-RES
- removed SJ1: (no value), symbol eagleSchem-eagle-import:JUMPER-PAD-3-NC_BY_TRACE
- removed SJ2: (no value), symbol eagleSchem-eagle-import:JUMPER-PAD-3-2OF3_NC_BY_PASTE
- removed STANDOFF1, STANDOFF2: (no value), symbol eagleSchem-eagle-import:STAND-OFF
- removed U1: (no value), symbol eagleSchem-eagle-import:MCP4725SOT-23
- added C1: (no value), symbol schematicEagle-eagle-import:CAP0603-CAP
- added FID1, FID2: (no value), symbol schematicEagle-eagle-import:FIDUCIAL1X2
- added FRAME2: (no value), symbol schematicEagle-eagle-import:FRAME-LETTER
- added GND0: (no value), symbol schematicEagle-eagle-import:LOGO-SFESK
- added JP5: (no value), symbol schematicEagle-eagle-import:M04PTH
- added JP6: (no value), symbol schematicEagle-eagle-import:M02PTH
- added LOGO1: (no value), symbol schematicEagle-eagle-import:OSHW-LOGOS
- added R1, R2, R3: (no value), symbol schematicEagle-eagle-import:RESISTOR0603-RES
- added SJ1: (no value), symbol schematicEagle-eagle-import:JUMPER-PAD-3-NC_BY_TRACE
- added SJ2: (no value), symbol schematicEagle-eagle-import:JUMPER-PAD-3-2OF3_NC_BY_PASTE
- added STANDOFF1, STANDOFF2: (no value), symbol schematicEagle-eagle-import:STAND-OFF
- added U1: (no value), symbol schematicEagle-eagle-import:MCP4725SOT-23
Connections:
- net GND: now also C1.2, JP5.4, JP6.1, R3.1, U1.2 (VSS)
- net SCL: now also JP5.1, R1.1, U1.5 (SCL)
- net SDA: now also JP5.2, R2.1, U1.4 (SDA)
- net VCC: now also C1.1, JP5.3, SJ1.2, SJ2.1, U1.3 (VDD)
- new net: SJ2.2, U1.6 (AO)
- new net: R3.2, SJ2.3
- new net: R2.2, SJ1.1
- new net: R1.2, SJ1.3
- new net: JP6.2, U1.1 (VOUT)
