File: PROJ/SPAR/13268/STAN/01/src/kicadBoard.kicad_sch (KiCad schematic)
At the start: 128 parts

Commit message: Quickly Adding Everything
Parts:
- removed FRAME1: (no value), symbol eagleSchem-eagle-import:FRAME-LEDGER
- removed JP1, JP10, JP100, JP101, JP102, JP103, JP104, JP105, JP106, JP107, JP108, JP109, JP11, JP110, JP111, JP112, JP113, JP114, JP115, JP116, JP117, JP118, JP119, JP12, JP120, JP121, JP122, JP123, JP124, JP125, JP13, JP14, JP15, JP16, JP17, JP18, JP19, JP2, JP20, JP21, JP22, JP23, JP24, JP25, JP26, JP27, JP28, JP29, JP3, JP30, JP31, JP32, JP33, JP34, JP35, JP36, JP37, JP38, JP39, JP4, JP40, JP41, JP42, JP43, JP44, JP45, JP46, JP47, JP48, JP49, JP5, JP50, JP51, JP52, JP53, JP54, JP55, JP56, JP57, JP58, JP59, JP6, JP60, JP61, JP62, JP63, JP64, JP65, JP66, JP67, JP68, JP69, JP7, JP70, JP71, JP72, JP73, JP74, JP75, JP76, JP77, JP78, JP79, JP8, JP80, JP81, JP82, JP83, JP84, JP85, JP86, JP87, JP88, JP89, JP9, JP90, JP91, JP92, JP93, JP94, JP95, JP96, JP97, JP98, JP99: (no value), symbol eagleSchem-eagle-import:M10NO_SILK_PTH_FEMALE
- removed LOGO1, LOGO2: (no value), symbol eagleSchem-eagle-import:SFE_LOGO_FLAME0.05_INCH
- added FRAME1: (no value), symbol schematicEagle-eagle-import:FRAME-LEDGER
- added JP1, JP10, JP100, JP101, JP102, JP103, JP104, JP105, JP106, JP107, JP108, JP109, JP11, JP110, JP111, JP112, JP113, JP114, JP115, JP116, JP117, JP118, JP119, JP12, JP120, JP121, JP122, JP123, JP124, JP125, JP13, JP14, JP15, JP16, JP17, JP18, JP19, JP2, JP20, JP21, JP22, JP23, JP24, JP25, JP26, JP27, JP28, JP29, JP3, JP30, JP31, JP32, JP33, JP34, JP35, JP36, JP37, JP38, JP39, JP4, JP40, JP41, JP42, JP43, JP44, JP45, JP46, JP47, JP48, JP49, JP5, JP50, JP51, JP52, JP53, JP54, JP55, JP56, JP57, JP58, JP59, JP6, JP60, JP61, JP62, JP63, JP64, JP65, JP66, JP67, JP68, JP69, JP7, JP70, JP71, JP72, JP73, JP74, JP75, JP76, JP77, JP78, JP79, JP8, JP80, JP81, JP82, JP83, JP84, JP85, JP86, JP87, JP88, JP89, JP9, JP90, JP91, JP92, JP93, JP94, JP95, JP96, JP97, JP98, JP99: (no value), symbol schematicEagle-eagle-import:M10NO_SILK_PTH_FEMALE
- added LOGO1, LOGO2: (no value), symbol schematicEagle-eagle-import:SFE_LOGO_FLAME0.05_INCH
