File: PROJ/SPAR/13279/STAN/01/src/kicadBoard.kicad_sch (KiCad schematic)
At the start: 28 parts

Commit message: Quickly Adding Everything
Parts:
- removed FID1, FID2: (no value), symbol eagleSchem-eagle-import:FIDUCIAL1X2
- removed FRAME1: (no value), symbol eagleSchem-eagle-import:FRAME-LETTER
- removed JP1, JP10, JP11, JP12, JP14, JP3, JP4, JP5, JP6, JP7, JP8, JP9: (no value), symbol eagleSchem-eagle-import:M01PTH_LONGPAD
- removed JP13, JP2: (no value), symbol eagleSchem-eagle-import:M06SMD
- removed LOGO1: (no value), symbol eagleSchem-eagle-import:SFE_LOGO_NAME_FLAME.1_INCH
- removed LOGO2: (no value), symbol eagleSchem-eagle-import:OSHW-LOGOS
- removed R1, R2, R3, R4, R5, R6, R7, R8: (no value), symbol eagleSchem-eagle-import:15OHM-1/10W-1%(0603)0603
- removed U1: (no value), symbol eagleSchem-eagle-import:TPIC6C596SOIC
- added FID1, FID2: (no value), symbol schematicEagle-eagle-import:FIDUCIAL1X2
- added FRAME1: (no value), symbol schematicEagle-eagle-import:FRAME-LETTER
- added JP1, JP10, JP11, JP12, JP14, JP3, JP4, JP5, JP6, JP7, JP8, JP9: (no value), symbol schematicEagle-eagle-import:M01PTH_LONGPAD
- added JP13, JP2: (no value), symbol schematicEagle-eagle-import:M06SMD
- added LOGO1: (no value), symbol schematicEagle-eagle-import:SFE_LOGO_NAME_FLAME.1_INCH
- added LOGO2: (no value), symbol schematicEagle-eagle-import:OSHW-LOGOS
- added R1, R2, R3, R4, R5, R6, R7, R8: (no value), symbol schematicEagle-eagle-import:15OHM-1/10W-1%(0603)0603
- added U1: (no value), symbol schematicEagle-eagle-import:TPIC6C596SOIC
Connections:
- net 12V: now also JP11.1, JP12.1, JP13.1, JP2.6
- net 5V: now also JP13.2, JP2.5, U1.1 (VCC), U1.7 (~{CLR})
- net CLOCK: now also JP13.4, JP2.3, U1.15 (SRCK)
- net GND: now also JP13.6, JP2.1, U1.16 (GND), U1.8 (~{G})
- net LATCH: now also JP13.5, JP2.2, U1.10 (RCK)
- net SER_IN: now also JP13.3, U1.2 (SER_IN)
- net SER_OUT: now also JP2.4, U1.9 (SER_OUT)
- new net: JP10.1, R8.2
- new net: R3.1, U1.5 (D2)
- new net: JP5.1, R3.2
- new net: R5.1, U1.11 (D4)
- new net: JP7.1, R5.2
- new net: JP1.1, R1.2
- new net: JP4.1, R2.2
- new net: R7.1, U1.13 (D6)
- new net: JP9.1, R7.2
- new net: R6.1, U1.12 (D5)
- new net: JP8.1, R6.2
- new net: R8.1, U1.14 (D7)
- new net: R1.1, U1.3 (D0)
- new net: JP6.1, R4.2
- new net: R4.1, U1.6 (D3)
- new net: R2.1, U1.4 (D1)
