File: PROJ/SPAR/13311/STAN/01/src/kicadBoard.kicad_sch (KiCad schematic)
At the start: 35 parts

Commit message: Quickly Adding Everything
Parts:
- removed FID1, FID2: (no value), symbol eagleSchem-eagle-import:FIDUCIAL1X2
- removed FRAME1: (no value), symbol eagleSchem-eagle-import:FRAME-LETTER
- removed JP1: (no value), symbol eagleSchem-eagle-import:TEENSY-3.1NOSILK
- removed JP2, JP3: (no value), symbol eagleSchem-eagle-import:M10NO_SILK_PTH_FEMALE
- removed JP4: (no value), symbol eagleSchem-eagle-import:M14
- removed JP5: (no value), symbol eagleSchem-eagle-import:M05PTH
- removed JP6: (no value), symbol eagleSchem-eagle-import:M03PTH
- removed JP7: (no value), symbol eagleSchem-eagle-import:M18_
- removed JP8: (no value), symbol eagleSchem-eagle-import:M02PTH
- removed JP9: (no value), symbol eagleSchem-eagle-import:XBEE-1B3
- removed LED1, LED2: (no value), symbol eagleSchem-eagle-import:LED-RED0603
- removed LED3, LED4, LED5: (no value), symbol eagleSchem-eagle-import:LED-GREEN0603
- removed LOGO1: (no value), symbol eagleSchem-eagle-import:SFE_LOGO_FLAME.2_INCH
- removed LOGO2: (no value), symbol eagleSchem-eagle-import:OSHW-LOGOM
- removed LOGO3: (no value), symbol eagleSchem-eagle-import:SFE_LOGO_NAME_FLAME.2_INCH
- removed R1, R11, R2, R3, R4: (no value), symbol eagleSchem-eagle-import:1KOHM1/10W1%(0603)
- removed S2: (no value), symbol eagleSchem-eagle-import:SWITCH-DPDTAYZ0202
- removed S3: (no value), symbol eagleSchem-eagle-import:SWITCH-MOMENTARY-2SMD
- removed SJ1, SJ3: (no value), symbol eagleSchem-eagle-import:JUMPER-PAD-2-NC_BY_PASTE
- removed SJ4: (no value), symbol eagleSchem-eagle-import:JUMPER-PAD-3-2OF3_NC_BY_PASTE
- removed SJ5: (no value), symbol eagleSchem-eagle-import:JUMPER-PAD-2-NOYES_SILK
- removed STANDOFF1, STANDOFF2, STANDOFF3, STANDOFF4: (no value), symbol eagleSchem-eagle-import:STAND-OFF
- added FID1, FID2: (no value), symbol schematicEagle-eagle-import:FIDUCIAL1X2
- added FRAME1: (no value), symbol schematicEagle-eagle-import:FRAME-LETTER
- added JP1: (no value), symbol schematicEagle-eagle-import:TEENSY-3.1NOSILK
- added JP2, JP3: (no value), symbol schematicEagle-eagle-import:M10NO_SILK_PTH_FEMALE
- added JP4: (no value), symbol schematicEagle-eagle-import:M14
- added JP5: (no value), symbol schematicEagle-eagle-import:M05PTH
- added JP6: (no value), symbol schematicEagle-eagle-import:M03PTH
- added JP7: (no value), symbol schematicEagle-eagle-import:M18_
- added JP8: (no value), symbol schematicEagle-eagle-import:M02PTH
- added JP9: (no value), symbol schematicEagle-eagle-import:XBEE-1B3
- added LED1, LED2: (no value), symbol schematicEagle-eagle-import:LED-RED0603
- added LED3, LED4, LED5: (no value), symbol schematicEagle-eagle-import:LED-GREEN0603
- added LOGO1: (no value), symbol schematicEagle-eagle-import:SFE_LOGO_FLAME.2_INCH
- added LOGO2: (no value), symbol schematicEagle-eagle-import:OSHW-LOGOM
- added LOGO3: (no value), symbol schematicEagle-eagle-import:SFE_LOGO_NAME_FLAME.2_INCH
- added R1, R11, R2, R3, R4: (no value), symbol schematicEagle-eagle-import:1KOHM1/10W1%(0603)
- added S2: (no value), symbol schematicEagle-eagle-import:SWITCH-DPDTAYZ0202
- added S3: (no value), symbol schematicEagle-eagle-import:SWITCH-MOMENTARY-2SMD
- added SJ1, SJ3: (no value), symbol schematicEagle-eagle-import:JUMPER-PAD-2-NC_BY_PASTE
- added SJ4: (no value), symbol schematicEagle-eagle-import:JUMPER-PAD-3-2OF3_NC_BY_PASTE
- added SJ5: (no value), symbol schematicEagle-eagle-import:JUMPER-PAD-2-NOYES_SILK
- added STANDOFF1, STANDOFF2, STANDOFF3, STANDOFF4: (no value), symbol schematicEagle-eagle-import:STAND-OFF
Connections:
- net 13/SCK: now also JP1.13 (13/SCK), JP7.18
- net 3.3V: now also JP1.3.3V, JP5.2, SJ4.3
- net A14/DAC: now also JP1.A14/DAC, JP5.5
- net A4/18/SDA0: now also JP1.18 (A4/18/SDA0), JP7.13
- net A5/19/SCL0: now also JP1.19 (A5/19/SCL0), JP7.12
- net A6/20: now also JP1.20 (A6/20*), JP7.11, SJ3.1
- net A7/21: now also JP1.21 (A7/21*), JP7.10, SJ1.1
- net DIO5: now also JP3.5, JP9.15 (DIO5), R2.2
- net EXT_3.3V: now also JP8.1, SJ4.1, SJ5.2
- net GND: now also JP1.AGND, JP1.GND, JP1.GND1, JP2.1, JP4.1, JP5.3, JP6.1, JP6.2, JP6.3, JP7.3, JP8.2, JP9.10 (GND), LED1.C, LED4.C, LED5.C, S3.3 (2)
- net IN: now also JP2.8, JP9.3 (DIN), LED3.C, S2.5
- net OUT: now also JP2.9, JP9.2 (DOUT), LED2.C, S2.2
- net PROG: now also JP1.PROG, JP5.4
- net RESET: now also JP2.6, JP9.5 (RESET), S3.1
- net RSSI: now also JP2.5, JP9.6 (RSSI), R4.2
- net UART_RX: now also JP1.0 (0/RX1), JP4.2, S2.1
- net UART_TX: now also JP1.1 (1/TX1), JP4.3, S2.4
- net VBAT: now also JP1.VBAT, JP5.1
- net VIN: now also JP1.VIN, JP7.1, SJ5.1
- net XBEE_VDD: now also JP2.10, JP9.1 (VDD), R1.1, R11.2, R3.1, SJ4.2
- new net: LED2.A, R1.2
- new net: JP3.1, JP9.11 (DIO4)
- new net: JP3.2, JP9.12 (CTS)
- new net: JP3.3, JP9.13 (DIO9)
- new net: JP3.4, JP9.14 (RES@14)
- new net: JP3.6, JP9.16 (RTS)
- new net: JP3.7, JP9.17 (DIO3)
- new net: JP3.8, JP9.18 (DIO2)
- new net: JP3.9, JP9.19 (DIO1)
- new net: JP3.10, JP9.20 (DIO0)
- new net: JP2.7, JP9.4 (DIO12)
- new net: JP2.4, JP9.7 (DIO11)
- new net: JP2.3, JP9.8 (RES@8)
- new net: JP2.2, JP9.9 (DTR)
- new net: LED5.A, R2.1
- new net: JP1.17 (A3/17), JP7.14
- new net: JP1.16 (A2/16), JP7.15
- new net: JP1.15 (A1/15), JP7.16
- new net: JP1.14 (A0/14), JP7.17
- new net: JP1.VUSB, JP7.2
- new net: JP1.3V, JP7.4
- new net: JP1.AREF, JP7.5
- new net: JP1.A11, JP7.6
- new net: JP1.A10, JP7.7
- new net: JP1.23 (A9/23*), JP7.8
- new net: JP1.22 (A8/22*), JP7.9
- new net: S2.6, SJ1.2
- new net: JP1.10 (10*/TX2/CS), JP4.12
- new net: JP1.11 (11/DOUT), JP4.13
- new net: JP1.12 (12/DIN), JP4.14
- new net: JP1.2, JP4.4
- new net: JP1.3 (3*), JP4.5
- new net: JP1.4 (4*), JP4.6
- new net: JP1.5 (5*), JP4.7
- new net: JP1.6 (6*), JP4.8
- new net: JP1.7 (7/RX3), JP4.9
- new net: JP1.8 (8/TX3), JP4.10
- new net: JP1.9 (9*/RX2), JP4.11
- new net: S2.3, SJ3.2
- new net: LED4.A, R4.1
- new net: LED3.A, R3.2
- new net: LED1.A, R11.1
