File: PROJ/SPAR/13712/STAN/01/src/kicadBoard.kicad_sch (KiCad schematic)
At the start: 26 parts

Commit message: Quickly Adding Everything
Parts:
- removed C1: (no value), symbol eagleSchem-eagle-import:10UF-6.3V-20%(0603)(TANT){dblquote}
- removed C2, C3, C4: (no value), symbol eagleSchem-eagle-import:0.1UF-25V(+80/-20%)(0603)
- removed D1: (no value), symbol eagleSchem-eagle-import:LED-BLUE0603
- removed D3: (no value), symbol eagleSchem-eagle-import:LED-GREEN0603
- removed FID1, FID2, FID3, FID4: (no value), symbol eagleSchem-eagle-import:FIDUCIALUFIDUCIAL
- removed FRAME1: (no value), symbol eagleSchem-eagle-import:FRAME-LETTER
- removed JP2: (no value), symbol eagleSchem-eagle-import:M06NO_SILK_FEMALE_PTH
- removed LOGO1: (no value), symbol eagleSchem-eagle-import:SFE_LOGO_FLAME.1_INCH
- removed LOGO2: (no value), symbol eagleSchem-eagle-import:OSHW-LOGOMINI
- removed Q1: (no value), symbol eagleSchem-eagle-import:RESONATOR16MHZ
- removed R1: (no value), symbol eagleSchem-eagle-import:1KOHM-1/10W-1%(0603)
- removed R2: (no value), symbol eagleSchem-eagle-import:10KOHM-1/10W-1%(0603)0603
- removed R6: (no value), symbol eagleSchem-eagle-import:330OHM1/10W1%(0603)
- removed TP1, TP2, TP3, TP4, TP5: (no value), symbol eagleSchem-eagle-import:TEST-POINT3
- removed U1: (no value), symbol eagleSchem-eagle-import:ATMEGA328P_TQFP
- removed U2: (no value), symbol eagleSchem-eagle-import:MIC52053.3V
- removed U3: (no value), symbol eagleSchem-eagle-import:USD-SOCKET
- added C1: (no value), symbol schematicEagle-eagle-import:10UF-6.3V-20%(0603)(TANT){dblquote}
- added C2, C3, C4: (no value), symbol schematicEagle-eagle-import:0.1UF-25V(+80/-20%)(0603)
- added D1: (no value), symbol schematicEagle-eagle-import:LED-BLUE0603
- added D3: (no value), symbol schematicEagle-eagle-import:LED-GREEN0603
- added FID1, FID2, FID3, FID4: (no value), symbol schematicEagle-eagle-import:FIDUCIALUFIDUCIAL
- added FRAME1: (no value), symbol schematicEagle-eagle-import:FRAME-LETTER
- added JP2: (no value), symbol schematicEagle-eagle-import:M06NO_SILK_FEMALE_PTH
- added LOGO1: (no value), symbol schematicEagle-eagle-import:SFE_LOGO_FLAME.1_INCH
- added LOGO2: (no value), symbol schematicEagle-eagle-import:OSHW-LOGOMINI
- added Q1: (no value), symbol schematicEagle-eagle-import:RESONATOR16MHZ
- added R1: (no value), symbol schematicEagle-eagle-import:1KOHM-1/10W-1%(0603)
- added R2: (no value), symbol schematicEagle-eagle-import:10KOHM-1/10W-1%(0603)0603
- added R6: (no value), symbol schematicEagle-eagle-import:330OHM1/10W1%(0603)
- added TP1, TP2, TP3, TP4, TP5: (no value), symbol schematicEagle-eagle-import:TEST-POINT3
- added U1: (no value), symbol schematicEagle-eagle-import:ATMEGA328P_TQFP
- added U2: (no value), symbol schematicEagle-eagle-import:MIC52053.3V
- added U3: (no value), symbol schematicEagle-eagle-import:USD-SOCKET
Connections:
- net 3.3V: now also C1.A (+), C3.2, C4.1, R2.2, TP1.P$1 (1), U1.18 (AVCC), U1.20 (AREF), U1.4 (VCC@4), U1.6 (VCC@6), U2.5 (OUT), U3.4 (VCC)
- net CD: now also U1.25 (PC2(ADC2)), U3.CD1
- net CS: now also U1.14 (PB2(SS/OC1B)), U3.2 (CS)
- net DTR: now also C2.2, JP2.6
- net GND: now also C1.K (-), C3.1, C4.2, D1.C, D3.C, JP2.1, JP2.2, Q1.2, U1.21 (AGND), U1.3 (GND@3), U1.5 (GND@5), U2.2 (GND), U3.6 (GND), U3.GND1 (SHIELD@3), U3.GND3 (SHIELD@1)
- net MISO: now also TP2.P$1 (1), U1.16 (PB4(MISO)), U3.7 (DO)
- net MOSI: now also TP3.P$1 (1), U1.15 (PB3(MOSI/OC2)), U3.3 (DI)
- net RAW: now also JP2.3, U2.1 (IN), U2.3 (EN)
- net RST: now also C2.1, R2.1, TP5.P$1 (1), U1.29 (PC6(/RESET))
- net RXI: now also JP2.5, U1.30 (PD0(RXD))
- net SCK: now also R6.1, TP4.P$1 (1), U1.17 (PB5(SCK)), U3.5 (SCK)
- net TXO: now also JP2.4, U1.31 (PD1(TXD))
- new net: D3.A, R6.2
- new net: Q1.1, U1.8 (PB7(XTAL2/TOSC2))
- new net: Q1.3, U1.7 (PB6(XTAL1/TOSC1))
- new net: R1.1, U1.9 (PD5(T1))
- new net: D1.A, R1.2
