File: PROJ/SPAR/13963/STAN/01/src/kicadBoard.kicad_sch (KiCad schematic)
At the start: 19 parts

Commit message: Quickly Adding Everything
Parts:
- removed C1: (no value), symbol eagleSchem-eagle-import:0.1UF-0402-16V-10%
- removed C2: (no value), symbol eagleSchem-eagle-import:10UF-0603-6.3V-20%
- removed FRAME2: (no value), symbol eagleSchem-eagle-import:FRAME-LETTER
- removed J1, J2: (no value), symbol eagleSchem-eagle-import:CONN_06NO_SILK_FEMALE_PTH
- removed JP2, JP6: (no value), symbol eagleSchem-eagle-import:FIDUCIALUFIDUCIAL
- removed JP3, JP4: (no value), symbol eagleSchem-eagle-import:STAND-OFF
- removed LOGO1, LOGO2: (no value), symbol eagleSchem-eagle-import:SFE_LOGO_FLAME.1_INCH
- removed R1, R2: (no value), symbol eagleSchem-eagle-import:4.7KOHM-0603-1/10W-1%
- removed R3, R4: (no value), symbol eagleSchem-eagle-import:10KOHM-0603-1/10W-1%
- removed SJ1: (no value), symbol eagleSchem-eagle-import:SOLDERJUMPERNO
- removed SJ2: (no value), symbol eagleSchem-eagle-import:JUMPER-PAD-3-NC_BY_TRACE
- removed U$1: (no value), symbol eagleSchem-eagle-import:OSHW-LOGOS
- removed U1: (no value), symbol eagleSchem-eagle-import:LIS3DH
- added C1: (no value), symbol schematicEagle-eagle-import:0.1UF-0402-16V-10%
- added C2: (no value), symbol schematicEagle-eagle-import:10UF-0603-6.3V-20%
- added FRAME2: (no value), symbol schematicEagle-eagle-import:FRAME-LETTER
- added J1, J2: (no value), symbol schematicEagle-eagle-import:CONN_06NO_SILK_FEMALE_PTH
- added JP2, JP6: (no value), symbol schematicEagle-eagle-import:FIDUCIALUFIDUCIAL
- added JP3, JP4: (no value), symbol schematicEagle-eagle-import:STAND-OFF
- added LOGO1, LOGO2: (no value), symbol schematicEagle-eagle-import:SFE_LOGO_FLAME.1_INCH
- added R1, R2: (no value), symbol schematicEagle-eagle-import:4.7KOHM-0603-1/10W-1%
- added R3, R4: (no value), symbol schematicEagle-eagle-import:10KOHM-0603-1/10W-1%
- added SJ1: (no value), symbol schematicEagle-eagle-import:SOLDERJUMPERNO
- added SJ2: (no value), symbol schematicEagle-eagle-import:JUMPER-PAD-3-NC_BY_TRACE
- added U$1: (no value), symbol schematicEagle-eagle-import:OSHW-LOGOS
- added U1: (no value), symbol schematicEagle-eagle-import:LIS3DH
Connections:
- net ADC1: now also J2.2, U1.16 (ADC1)
- net ADC2: now also J2.3, U1.15 (ADC2)
- net ADC3: now also J2.4, U1.13 (ADC3)
- net GND: now also C1.2, C2.2, J1.1, J2.1, SJ1.1, U1.10 (RES), U1.12 (GND@12), U1.5 (GND@5)
- net INT1: now also J2.5, U1.11 (INT1)
- net INT2: now also J2.6, U1.9 (INT2)
- net SA0: now also J1.5, R3.1, SJ1.2, U1.7 (SA0/SDO)
- net SCL: now also J1.4, R1.1, U1.4 (SCL/SPC)
- net SDA: now also J1.3, R2.1, U1.6 (SDA/SDI)
- net VCC: now also C1.1, C2.1, J1.2, R3.2, R4.2, SJ2.2, U1.1 (VDDIO), U1.14 (VDD)
- net ~{CS}: now also J1.6, R4.1, U1.8 (~{CS}/MODE)
- new net: R2.2, SJ2.1
- new net: R1.2, SJ2.3
