File: PROJ/SPAR/13975/STAN/01/src/kicadBoard.kicad_sch (KiCad schematic)
At the start: 65 parts

Commit message: Quickly Adding Everything
Parts:
- removed C1, C10, C12, C14, C2, C4, C8: (no value), symbol eagleSchem-eagle-import:0.1UF-0603-25V-(+80/-20%)
- removed C13, C9: (no value), symbol eagleSchem-eagle-import:47PF-0603-50V-5%
- removed C15, C3, C6: (no value), symbol eagleSchem-eagle-import:10UF-POLAR-EIA3216-16V-10%(TANT)
- removed C5: (no value), symbol eagleSchem-eagle-import:47UF-POLAR-PANASONIC_D-35V-20%
- removed C7: (no value), symbol eagleSchem-eagle-import:1.0UF-0603-16V-10%
- removed D1: (no value), symbol eagleSchem-eagle-import:MBRA140
- removed F1: (no value), symbol eagleSchem-eagle-import:PTC-HALF_AMP
- removed FRAME2: (no value), symbol eagleSchem-eagle-import:FRAME-LETTER
- removed IC3: (no value), symbol eagleSchem-eagle-import:V_REG_LM1117ALT1
- removed J2: (no value), symbol eagleSchem-eagle-import:AVR_SPI_PROG_3X2SMD
- removed J3: (no value), symbol eagleSchem-eagle-import:POWER_JACKSUPER_BOMB_DIGITY
- removed JP1: (no value), symbol eagleSchem-eagle-import:SFE_LOGO_NAME.1_INCH
- removed JP10, JP11: (no value), symbol eagleSchem-eagle-import:M08SMD-COMBO
- removed JP12: (no value), symbol eagleSchem-eagle-import:USB-MINIB-5PIN
- removed JP13: (no value), symbol eagleSchem-eagle-import:M06SMD-STRAIGHT-COMBO
- removed JP2: (no value), symbol eagleSchem-eagle-import:M10SMD_COMBO
- removed JP3, JP4, JP5, JP6: (no value), symbol eagleSchem-eagle-import:STAND-OFF
- removed JP7: (no value), symbol eagleSchem-eagle-import:SFE_LOGO_FLAME.1_INCH
- removed JP8, JP9: (no value), symbol eagleSchem-eagle-import:FIDUCIAL1X2
- removed LED1, LED2, LED3, LED4: (no value), symbol eagleSchem-eagle-import:LED1206
- removed Q1: (no value), symbol eagleSchem-eagle-import:MOSFET-PCH-ZXMP6A13F
- removed Q2: (no value), symbol eagleSchem-eagle-import:MOSFET-NCH-2N7002PW
- removed R1, R6, R7, R8, R9: (no value), symbol eagleSchem-eagle-import:1KOHM-0603-1/10W-1%
- removed R10, R5: (no value), symbol eagleSchem-eagle-import:27OHM-0603-1/10W-1%
- removed R11, R13, R3, R4: (no value), symbol eagleSchem-eagle-import:10KOHM-0603-1/10W-1%
- removed R14: (no value), symbol eagleSchem-eagle-import:715OHM-0603-1/10W-1%
- removed R15: (no value), symbol eagleSchem-eagle-import:240OHM-0603-1/10W-1%
- removed R2: (no value), symbol eagleSchem-eagle-import:4.7KOHM-0603-1/10W-1%
- removed S1: (no value), symbol eagleSchem-eagle-import:SWITCH_SPST_4_PINSQUARE
- removed TP1, TP2, TP3, TP4, TP5, TP6: (no value), symbol eagleSchem-eagle-import:TEST-POINT3X5
- removed U$16: (no value), symbol eagleSchem-eagle-import:OSHW-LOGOS
- removed U1: (no value), symbol eagleSchem-eagle-import:FT231XS
- removed U2: (no value), symbol eagleSchem-eagle-import:MIC52053.3V
- removed U4: (no value), symbol eagleSchem-eagle-import:ATMEGA328P_TQFP
- removed Y1: (no value), symbol eagleSchem-eagle-import:RESONATOR-16MHZSMD_3.2X1.3
- added C1, C10, C12, C14, C2, C4, C8: (no value), symbol schematicEagle-eagle-import:0.1UF-0603-25V-(+80/-20%)
- added C13, C9: (no value), symbol schematicEagle-eagle-import:47PF-0603-50V-5%
- added C15, C3, C6: (no value), symbol schematicEagle-eagle-import:10UF-POLAR-EIA3216-16V-10%(TANT)
- added C5: (no value), symbol schematicEagle-eagle-import:47UF-POLAR-PANASONIC_D-35V-20%
- added C7: (no value), symbol schematicEagle-eagle-import:1.0UF-0603-16V-10%
- added D1: (no value), symbol schematicEagle-eagle-import:MBRA140
- added F1: (no value), symbol schematicEagle-eagle-import:PTC-HALF_AMP
- added FRAME2: (no value), symbol schematicEagle-eagle-import:FRAME-LETTER
- added IC3: (no value), symbol schematicEagle-eagle-import:V_REG_LM1117ALT1
- added J2: (no value), symbol schematicEagle-eagle-import:AVR_SPI_PROG_3X2SMD
- added J3: (no value), symbol schematicEagle-eagle-import:POWER_JACKSUPER_BOMB_DIGITY
- added JP1: (no value), symbol schematicEagle-eagle-import:SFE_LOGO_NAME.1_INCH
- added JP10, JP11: (no value), symbol schematicEagle-eagle-import:M08SMD-COMBO
- added JP12: (no value), symbol schematicEagle-eagle-import:USB-MINIB-5PIN
- added JP13: (no value), symbol schematicEagle-eagle-import:M06SMD-STRAIGHT-COMBO
- added JP2: (no value), symbol schematicEagle-eagle-import:M10SMD_COMBO
- added JP3, JP4, JP5, JP6: (no value), symbol schematicEagle-eagle-import:STAND-OFF
- added JP7: (no value), symbol schematicEagle-eagle-import:SFE_LOGO_FLAME.1_INCH
- added JP8, JP9: (no value), symbol schematicEagle-eagle-import:FIDUCIAL1X2
- added LED1, LED2, LED3, LED4: (no value), symbol schematicEagle-eagle-import:LED1206
- added Q1: (no value), symbol schematicEagle-eagle-import:MOSFET-PCH-ZXMP6A13F
- added Q2: (no value), symbol schematicEagle-eagle-import:MOSFET-NCH-2N7002PW
- added R1, R6, R7, R8, R9: (no value), symbol schematicEagle-eagle-import:1KOHM-0603-1/10W-1%
- added R10, R5: (no value), symbol schematicEagle-eagle-import:27OHM-0603-1/10W-1%
- added R11, R13, R3, R4: (no value), symbol schematicEagle-eagle-import:10KOHM-0603-1/10W-1%
- added R14: (no value), symbol schematicEagle-eagle-import:715OHM-0603-1/10W-1%
- added R15: (no value), symbol schematicEagle-eagle-import:240OHM-0603-1/10W-1%
- added R2: (no value), symbol schematicEagle-eagle-import:4.7KOHM-0603-1/10W-1%
- added S1: (no value), symbol schematicEagle-eagle-import:SWITCH_SPST_4_PINSQUARE
- added TP1, TP2, TP3, TP4, TP5, TP6: (no value), symbol schematicEagle-eagle-import:TEST-POINT3X5
- added U$16: (no value), symbol schematicEagle-eagle-import:OSHW-LOGOS
- added U1: (no value), symbol schematicEagle-eagle-import:FT231XS
- added U2: (no value), symbol schematicEagle-eagle-import:MIC52053.3V
- added U4: (no value), symbol schematicEagle-eagle-import:ATMEGA328P_TQFP
- added Y1: (no value), symbol schematicEagle-eagle-import:RESONATOR-16MHZSMD_3.2X1.3
Connections:
- net 3.3V: now also C6.+, C7.1, JP10.5A (5), JP10.5B (5), U2.5 (OUT)
- net 3.3V_F: now also C14.1, Q2.1 (G), R11.2, U1.13 (3V3OUT), U1.14 (~{RESET}), U1.3 (VCCIO)
- net 5V: now also C2.2, C3.+, C4.1, IC3.2 (OUT), IC3.4 (OUT@1), J2.2, JP10.4A (4), JP10.4B (4), JP10.7A (7), JP10.7B (7), Q1.2 (S), R13.2, R15.2, R2.2, R3.2, R4.2, R6.1, R7.1, TP1.P$1 (1), U2.1 (IN), U2.3 (EN), U4.18 (AVCC), U4.4 (VCC@4), U4.6 (VCC@6)
- net AD0: now also JP13.1A (1), JP13.1B (1), U4.23 (PC0(ADC0))
- net AD1: now also JP13.2A (2), JP13.2B (2), U4.24 (PC1(ADC1))
- net AD2: now also JP13.3A (3), JP13.3B (3), U4.25 (PC2(ADC2))
- net AD3: now also JP13.4A (4), JP13.4B (4), U4.26 (PC3(ADC3))
- net AD4/SDA: now also JP13.5A (5), JP13.5B (5), JP2.2A (2), JP2.2B (2), U4.27 (PC4(ADC4/SDA))
- net AD5/SCL: now also JP13.6A (6), JP13.6B (6), JP2.1A (1), JP2.1B (1), U4.28 (PC5(ADC5/SCL))
- net AREF: now also C1.1, JP2.3A (3), JP2.3B (3), U4.20 (AREF)
- net D+: now also C9.1, JP12.D+, R10.1
- net D-: now also C13.1, JP12.D-, R5.1
- net DTR: now also C8.1, Q2.3 (D), R13.1
- net GND: now also C1.2, C10.2, C12.2, C13.2, C14.2, C15.-, C2.1, C3.-, C4.2, C5.-, C6.-, C7.2, C9.2, J2.6, J3.GND (GNDBREAK), JP10.2A (2), JP10.2B (2), JP10.3A (3), JP10.3B (3), JP12.GND, JP12.MTN1 (MTN2), JP12.MTN2 (MTN3), JP12.MTN3 (MTN1), JP12.MTN4, JP2.4A (4), JP2.4B (4), LED1.C, LED2.C, R14.1, S1.1, S1.2, TP3.P$1 (1), U1.16 (GND@16), U1.6 (GND@6), U2.2 (GND), U4.21 (AGND), U4.3 (GND@3), U4.5 (GND@5), Y1.2
- net IO2: now also JP11.3A (3), JP11.3B (3), U4.32 (PD2(INT0))
- net IO3: now also JP11.4A (4), JP11.4B (4), U4.1 (PD3(INT1))
- net IO4: now also JP11.5A (5), JP11.5B (5), U4.2 (PD4(XCK/T0))
- net IO5: now also JP11.6A (6), JP11.6B (6), U4.9 (PD5(T1))
- net IO6: now also JP11.7A (7), JP11.7B (7), U4.10 (PD6(AIN0))
- net IO7: now also JP11.8A (8), JP11.8B (8), U4.11 (PD7(AIN1))
- net IO8: now also JP2.10A (10), JP2.10B (10), U4.12 (PB0(ICP))
- net IO9: now also JP2.9A (9), JP2.9B (9), U4.13 (PB1(OC1A))
- net MISO: now also J2.1, JP2.6A (6), JP2.6B (6), TP4.P$1 (1), U4.16 (PB4(MISO))
- net MOSI: now also J2.4, JP2.7A (7), JP2.7B (7), TP2.P$1 (1), U4.15 (PB3(MOSI/OC2))
- net RESET: now also C8.2, J2.5, JP10.6A (6), JP10.6B (6), R3.1, S1.3, S1.4, TP6.P$1 (1), U4.29 (PC6(/RESET))
- net RX-I: now also JP11.1A (1), JP11.1B (1), R8.1, U4.30 (PD0(RXD))
- net RXLED: now also LED4.C, U1.17 (CBUS1)
- net SCK: now also J2.3, JP2.5A (5), JP2.5B (5), R1.1, TP5.P$1 (1), U4.17 (PB5(SCK))
- net SS: now also JP2.8A (8), JP2.8B (8), U4.14 (PB2(SS/OC1B))
- net TX-O: now also JP11.2A (2), JP11.2B (2), R9.1, U4.31 (PD1(TXD))
- net TXLED: now also LED3.C, U1.10 (CBUS2)
- net USBVCC: now also C12.1, C15.+, F1.2, Q1.3 (D), U1.15 (VCC)
- net VIN: now also C5.+, D1.C, IC3.3 (IN), JP10.1A (1), JP10.1B (1)
- new net: U4.7 (PB6(XTAL1/TOSC1)), Y1.1
- new net: U4.8 (PB7(XTAL2/TOSC2)), Y1.3
- new net: Q2.2 (S), R11.1, U1.1 (~{DTR})
- new net: R5.2, U1.12 (USBDM)
- new net: J3.P$4 (GND), Q1.1 (G), R4.1
- new net: D1.A, J3.VIN0 (PWR)
- new net: LED3.A, R6.2
- new net: IC3.1 (ADJ), R14.2, R15.1
- new net: R10.2, U1.11 (USBDP)
- new net: C10.1, F1.1, JP12.VBUS
- new net: LED4.A, R7.2
- new net: LED1.A, R1.2
- new net: R8.2, U1.20 (TXD)
- new net: JP10.8A (8), JP10.8B (8)
- new net: R9.2, U1.4 (RXD)
- new net: LED2.A, R2.1
