File: PROJ/SPAR/14010/STAN/01/src/kicadBoard.kicad_sch (KiCad schematic)
At the start: 22 parts

Commit message: Quickly Adding Everything
Parts:
- removed D1, D2, D3, D4, D5: (no value), symbol eagleSchem-eagle-import:LED-WHITE1206
- removed FRAME1: (no value), symbol eagleSchem-eagle-import:FRAME-LETTER
- removed LED+1, LED+2, LED+3, LED+4, LED+5, LED-1, LED-2, LED-3, LED-4, LED-5: (no value), symbol eagleSchem-eagle-import:SEWTAP6
- removed R1, R2, R3, R4, R5: (no value), symbol eagleSchem-eagle-import:150OHM-1/10W-1%(0603)
- removed U$6: (no value), symbol eagleSchem-eagle-import:REVISION
- added D1, D2, D3, D4, D5: (no value), symbol schematicEagle-eagle-import:LED-WHITE1206
- added FRAME1: (no value), symbol schematicEagle-eagle-import:FRAME-LETTER
- added LED+1, LED+2, LED+3, LED+4, LED+5, LED-1, LED-2, LED-3, LED-4, LED-5: (no value), symbol schematicEagle-eagle-import:SEWTAP6
- added R1, R2, R3, R4, R5: (no value), symbol schematicEagle-eagle-import:150OHM-1/10W-1%(0603)
- added U$6: (no value), symbol schematicEagle-eagle-import:REVISION
Connections:
- new net: LED-5.1, R5.1
- new net: LED-3.1, R3.1
- new net: D3.C, R3.2
- new net: LED-2.1, R2.1
- new net: D2.C, R2.2
- new net: D1.A, LED+1.1
- new net: D5.A, LED+5.1
- new net: LED-4.1, R4.1
- new net: D4.C, R4.2
- new net: D4.A, LED+4.1
- new net: D3.A, LED+3.1
- new net: D5.C, R5.2
- new net: D2.A, LED+2.1
- new net: LED-1.1, R1.1
- new net: D1.C, R1.2
