File: PROJ/SPAR/14030/STAN/01/src/kicadBoard.kicad_sch (KiCad schematic)
At the start: 19 parts

Commit message: Quickly Adding Everything
Parts:
- removed C5: (no value), symbol eagleSchem-eagle-import:1.0UF-25V-+80/-20(0805){dblquote}
- removed C6: (no value), symbol eagleSchem-eagle-import:2.2UF-10V-20%(0603)
- removed D1: (no value), symbol eagleSchem-eagle-import:LED-BLUE0603
- removed FD1, FD2: (no value), symbol eagleSchem-eagle-import:FIDUCIALUFIDUCIAL
- removed FRAME1: (no value), symbol eagleSchem-eagle-import:FRAME-LETTER
- removed J1: (no value), symbol eagleSchem-eagle-import:MICROSD_TINY
- removed J2, J3: (no value), symbol eagleSchem-eagle-import:M12NO_SILK
- removed J4: (no value), symbol eagleSchem-eagle-import:M06NO_SILK_FEMALE_PTH
- removed J5: (no value), symbol eagleSchem-eagle-import:M021X02_NO_SILK
- removed LOGO1: (no value), symbol eagleSchem-eagle-import:OSHW-LOGOS
- removed LOGO3: (no value), symbol eagleSchem-eagle-import:SFE_LOGO_FLAME.1_INCH
- removed LOGO4: (no value), symbol eagleSchem-eagle-import:SFE_LOGO_NAME.1_INCH
- removed R1: (no value), symbol eagleSchem-eagle-import:470OHM1/10W1%(0603)
- removed S1: (no value), symbol eagleSchem-eagle-import:SWITCH-DPDTAYZ0202
- removed U1: (no value), symbol eagleSchem-eagle-import:GP735
- removed U2: (no value), symbol eagleSchem-eagle-import:TXB0108
- removed U3: (no value), symbol eagleSchem-eagle-import:V_REG_LDOSMD
- added C5: (no value), symbol schematicEagle-eagle-import:1.0UF-25V-+80/-20(0805){dblquote}
- added C6: (no value), symbol schematicEagle-eagle-import:2.2UF-10V-20%(0603)
- added D1: (no value), symbol schematicEagle-eagle-import:LED-BLUE0603
- added FD1, FD2: (no value), symbol schematicEagle-eagle-import:FIDUCIALUFIDUCIAL
- added FRAME1: (no value), symbol schematicEagle-eagle-import:FRAME-LETTER
- added J1: (no value), symbol schematicEagle-eagle-import:MICROSD_TINY
- added J2, J3: (no value), symbol schematicEagle-eagle-import:M12NO_SILK
- added J4: (no value), symbol schematicEagle-eagle-import:M06NO_SILK_FEMALE_PTH
- added J5: (no value), symbol schematicEagle-eagle-import:M021X02_NO_SILK
- added LOGO1: (no value), symbol schematicEagle-eagle-import:OSHW-LOGOS
- added LOGO3: (no value), symbol schematicEagle-eagle-import:SFE_LOGO_FLAME.1_INCH
- added LOGO4: (no value), symbol schematicEagle-eagle-import:SFE_LOGO_NAME.1_INCH
- added R1: (no value), symbol schematicEagle-eagle-import:470OHM1/10W1%(0603)
- added S1: (no value), symbol schematicEagle-eagle-import:SWITCH-DPDTAYZ0202
- added U1: (no value), symbol schematicEagle-eagle-import:GP735
- added U2: (no value), symbol schematicEagle-eagle-import:TXB0108
- added U3: (no value), symbol schematicEagle-eagle-import:V_REG_LDOSMD
Connections:
- net 10: now also J3.1, U2.11 (B8)
- net 11: now also J3.2, U2.12 (B7)
- net 12: now also J3.3, U2.14 (B5)
- net 13: now also J3.4, U2.13 (B6)
- net 2: now also J2.8
- net 3: now also J2.7
- net 3.3V: now also C6.1, J1.4 (VCC), J4.2, U1.2 (VCC), U2.5 (VCCA), U2.6 (OE), U3.5 (OUT)
- net 4: now also J2.6, S1.1
- net 5: now also J2.5, S1.4
- net 6: now also J2.4, U2.20 (B1)
- net 7: now also J2.3, R1.2
- net 8: now also J2.2
- net 9: now also J2.1
- net A0: now also J3.5
- net A1: now also J3.6
- net A2: now also J3.7
- net A3: now also J3.8
- net GND: now also C5.2, C6.2, D1.C, J1.6 (GND), J1.GND1 (SHIELD), J1.GND2 (SHIELD), J1.GND3 (SHIELD), J1.GND4 (SHIELD), J1.GND5 (SHIELD), J1.GND6 (SHIELD), J2.9, J3.11, J4.1, J5.1, U1.1 (GND), U2.15 (GND), U3.2 (GND)
- net GPS_CTRL: now also J4.6, U1.6 (P_CTRL), U2.1 (A1)
- net GPS_RX: now also J4.4, U1.4 (RX), U2.3 (A3)
- net GPS_TX: now also J4.3, U1.3 (TX), U2.2 (A2)
- net RX: now also S1.2, U2.19 (B2)
- net RX/0: now also J2.11, S1.3
- net SD_CS: now also J1.2 (CS), U2.10 (A8)
- net SD_DI: now also J1.3 (DI), U2.9 (A7)
- net SD_DO: now also J1.7 (DO), U2.7 (A5)
- net SD_SCK: now also J1.5 (SCK), U2.8 (A6)
- net TX: now also S1.5, U2.18 (B3)
- net TX/1: now also J2.12, S1.6
- net VCC: now also C5.1, J3.9, U2.16 (VCCB), U3.1 (IN), U3.3 (EN)
- net VIN: now also J3.12
- net V_BATT: now also J4.5, J5.2, U1.5 (VBAT)
- new net: D1.A, R1.1
- new net: J1.1 (RSV), J1.8 (RSV)
