File: PROJ/SPAR/14346/STAN/01/src/kicadBoard.kicad_sch (KiCad schematic)
At the start: 0 parts

Commit message: Quickly Adding Everything
Other:
- removed sheet eagleSchem_2
- removed sheet eagleSchem_3
- added sheet schematicEagle_2 (schematicEagle_2.kicad_sch)
- added sheet schematicEagle_3 (schematicEagle_3.kicad_sch)
