File: PROJ/SPAR/14449/STAN/01/src/kicadBoard.kicad_sch (KiCad schematic)
At the start: 55 parts

Commit message: Quickly Adding Everything
Parts:
- removed C1: (no value), symbol eagleSchem-eagle-import:2.2NF/2200PF-0603-50V-10%
- removed C10, C11, C12, C13, C14, C3: (no value), symbol eagleSchem-eagle-import:1.0UF-0402-16V-10%
- removed C2, C4, C5, C6, C7, C8, C9: (no value), symbol eagleSchem-eagle-import:0.1UF-0402-16V-10%
- removed D1: (no value), symbol eagleSchem-eagle-import:LED1206-BOTTOM
- removed F1: (no value), symbol eagleSchem-eagle-import:PPTC_HALF-AMP
- removed FD1, FD2, FD3, FD4: (no value), symbol eagleSchem-eagle-import:FIDUCIAL1X2
- removed FRAME1: (no value), symbol eagleSchem-eagle-import:FRAME-LETTER
- removed H1: (no value), symbol eagleSchem-eagle-import:6400BG_HEATSINK
- removed H2, H3, H4, H5: (no value), symbol eagleSchem-eagle-import:STAND-OFF
- removed J2: (no value), symbol eagleSchem-eagle-import:CONN_16
- removed J3: (no value), symbol eagleSchem-eagle-import:USB_MICRO-B_HALF_PTH
- removed J4: (no value), symbol eagleSchem-eagle-import:CONN_023.5MM_LOCK
- removed J5: (no value), symbol eagleSchem-eagle-import:CONN_05
- removed J6: (no value), symbol eagleSchem-eagle-import:CONN_02
- removed J7: (no value), symbol eagleSchem-eagle-import:CONN_04
- removed JP1: (no value), symbol eagleSchem-eagle-import:JUMPER-SMT_2_NC_TRACE_NO-SILK
- removed LOGO1: (no value), symbol eagleSchem-eagle-import:OSHW-LOGOM
- removed LOGO2, LOGO3: (no value), symbol eagleSchem-eagle-import:SFE_LOGO_NAME.3_INCH
- removed Q1: (no value), symbol eagleSchem-eagle-import:MOSFET-NCH-FQP30N06L
- removed R1, R12, R2, R3, R4: (no value), symbol eagleSchem-eagle-import:560OHM_0402_1%
- removed R10: (no value), symbol eagleSchem-eagle-import:8.2KOHM-0603-1/10W-5%
- removed R11: (no value), symbol eagleSchem-eagle-import:787OHM-0603-1/10W-1%
- removed R13, R9: (no value), symbol eagleSchem-eagle-import:1KOHM-0603-1/10W-1%
- removed R14: (no value), symbol eagleSchem-eagle-import:4.7KOHM-0603-1/10W-1%
- removed R18, R19: (no value), symbol eagleSchem-eagle-import:22OHM1/10W1%(0402)
- removed R5, R6: (no value), symbol eagleSchem-eagle-import:47KOHM-0603-1/10W-1%
- removed R7, R8: (no value), symbol eagleSchem-eagle-import:0.05OHM-2512-3W-1%
- removed U1: (no value), symbol eagleSchem-eagle-import:PSOC_5LP_68QFN
- removed U2: (no value), symbol eagleSchem-eagle-import:V_REG_AP2112K-3.3V
- added C1: (no value), symbol schematicEagle-eagle-import:2.2NF/2200PF-0603-50V-10%
- added C10, C11, C12, C13, C14, C3: (no value), symbol schematicEagle-eagle-import:1.0UF-0402-16V-10%
- added C2, C4, C5, C6, C7, C8, C9: (no value), symbol schematicEagle-eagle-import:0.1UF-0402-16V-10%
- added D1: (no value), symbol schematicEagle-eagle-import:LED1206-BOTTOM
- added F1: (no value), symbol schematicEagle-eagle-import:PPTC_HALF-AMP
- added FD1, FD2, FD3, FD4: (no value), symbol schematicEagle-eagle-import:FIDUCIAL1X2
- added FRAME1: (no value), symbol schematicEagle-eagle-import:FRAME-LETTER
- added H1: (no value), symbol schematicEagle-eagle-import:6400BG_HEATSINK
- added H2, H3, H4, H5: (no value), symbol schematicEagle-eagle-import:STAND-OFF
- added J2: (no value), symbol schematicEagle-eagle-import:CONN_16
- added J3: (no value), symbol schematicEagle-eagle-import:USB_MICRO-B_HALF_PTH
- added J4: (no value), symbol schematicEagle-eagle-import:CONN_023.5MM_LOCK
- added J5: (no value), symbol schematicEagle-eagle-import:CONN_05
- added J6: (no value), symbol schematicEagle-eagle-import:CONN_02
- added J7: (no value), symbol schematicEagle-eagle-import:CONN_04
- added JP1: (no value), symbol schematicEagle-eagle-import:JUMPER-SMT_2_NC_TRACE_NO-SILK
- added LOGO1: (no value), symbol schematicEagle-eagle-import:OSHW-LOGOM
- added LOGO2, LOGO3: (no value), symbol schematicEagle-eagle-import:SFE_LOGO_NAME.3_INCH
- added Q1: (no value), symbol schematicEagle-eagle-import:MOSFET-NCH-FQP30N06L
- added R1, R12, R2, R3, R4: (no value), symbol schematicEagle-eagle-import:560OHM_0402_1%
- added R10: (no value), symbol schematicEagle-eagle-import:8.2KOHM-0603-1/10W-5%
- added R11: (no value), symbol schematicEagle-eagle-import:787OHM-0603-1/10W-1%
- added R13, R9: (no value), symbol schematicEagle-eagle-import:1KOHM-0603-1/10W-1%
- added R14: (no value), symbol schematicEagle-eagle-import:4.7KOHM-0603-1/10W-1%
- added R18, R19: (no value), symbol schematicEagle-eagle-import:22OHM1/10W1%(0402)
- added R5, R6: (no value), symbol schematicEagle-eagle-import:47KOHM-0603-1/10W-1%
- added R7, R8: (no value), symbol schematicEagle-eagle-import:0.05OHM-2512-3W-1%
- added U1: (no value), symbol schematicEagle-eagle-import:PSOC_5LP_68QFN
- added U2: (no value), symbol schematicEagle-eagle-import:V_REG_AP2112K-3.3V
Connections:
- net 3.3V: now also C13.1, C5.1, U1.67 (VDDIO2), U2.5 (OUT)
- net 5V: now also C10.1, C14.1, C2.1, C3.1, C4.1, C6.1, C7.1, C8.1, C9.1, F1.2, J2.2, J5.5, J6.2, J7.3, R14.2, U1.17 (VDDIO1), U1.24 (VDDD0), U1.35 (VDDIO3), U1.44 (VDDA), U1.52 (VDDIO0), U1.59 (VDDD1), U2.1 (IN), U2.3 (EN)
- net BACK: now also R4.2
- net CONTRAST: now also J2.3, R13.2, R14.1
- net D+: now also J3.D+, R18.2
- net D-: now also J3.D-, R19.2
- net DOWN: now also R2.2
- net ENTER: now also R3.2
- net GND: now also C1.2, C10.2, C11.2, C12.2, C13.2, C14.2, C2.2, C3.2, C4.2, C5.2, C6.2, C7.2, C8.2, C9.2, J2.1, J3.GND, J5.4, J6.1, J7.4, JP1.1, R12.2, R13.1, R9.2, U1.25 (VSSD1), U1.43 (VSSA), U1.45 (VSSD2), U1.5 (VSSB), U1.58 (VSSD3), U1.69 (VSSD0), U1.7 (VBOOST), U1.8 (VBAT), U1.9 (VSSD0), U2.2 (GND)
- net GND-ISO: now also J4.2, JP1.2, R8.P$1 (1), U1.19 (P1[7])
- net I_SENSE_HIGH: now also Q1.3 (S), R7.P$2 (2), U1.18 (P1[6])
- net I_SET: now also Q1.1 (G), U1.37 (P3[7])
- net I_SET_SUM: now also R5.2, R6.2, U1.32 (P3[3])
- net LCD_D4: now also J2.11, U1.49 (P0[1])
- net LCD_D5: now also J2.12, U1.50 (P0[2])
- net LCD_D6: now also J2.13, U1.51 (P0[3])
- net LCD_D7: now also J2.14, U1.53 (P0[4])
- net LCD_E: now also J2.6, U1.54 (P0[5])
- net LCD_RS: now also J2.4, U1.55 (P0[6])
- net LCD_RW: now also J2.5, U1.56 (P0[7])
- net RXI: now also J7.2, U1.3 (P12[4])
- net SHIELD: now also J3.P$1 (SHIELD), J3.P$10 (SHIELD), J3.P$12 (SHIELD), J3.P$2 (SHIELD), J3.P$3 (SHIELD), J3.P$4 (SHIELD), J3.P$6 (SHIELD), J3.P$8 (SHIELD), J3.SHEILD2 (SHIELD), J3.SHIELD, J3.SHIELD3 (SHIELD), J3.SHIELD4 (SHIELD)
- net SWDCK: now also J5.2, U1.12 (P1[1])
- net SWDIO: now also J5.1, U1.11 (P1[0])
- net TXO: now also J7.1, U1.4 (P12[5])
- net UP: now also R1.2
- net V_SENSE: now also R11.2, R9.1, U1.33 (P3[4])
- net XRES: now also J5.3, U1.10 (~{XRES})
- new net: D1.C, R12.1
- new net: C11.1, U1.42 (VCCA)
- new net: F1.1, J3.VBUS
- new net: R5.1, U1.48 (P0[0])
- new net: D1.A, U1.29 (P3[0])
- new net: R4.1, U1.62 (P2[0])
- new net: R3.1, U1.63 (P2[1])
- new net: R2.1, U1.64 (P2[2])
- new net: R1.1, U1.65 (P2[3])
- new net: C1.1, U1.66 (P2[4])
- new net: R6.1, U1.36 (P3[6])
- new net: R19.1, U1.23 (P15[7])
- new net: J4.1, Q1.2 (D), R10.1
- new net: R18.1, U1.22 (P15[6])
- new net: C12.1, U1.26 (VCCD0), U1.57 (VCCD1)
- new net: R7.P$1 (1), R8.P$2 (2)
- new net: R10.2, R11.1
