File: PROJ/SPAR/14544/STAN/01/src/kicadBoard.kicad_sch (KiCad schematic)
At the start: 26 parts

Commit message: Quickly Adding Everything
Parts:
- removed C1: (no value), symbol eagleSchem-eagle-import:100PF-0603-50V-5%
- removed C2, C3, C4: (no value), symbol eagleSchem-eagle-import:0.1UF-0603-25V-(+80/-20%)
- removed C5: (no value), symbol eagleSchem-eagle-import:1.0NF/1000PF-0603-50V-10%
- removed FD1, FD2, FD3, FD4: (no value), symbol eagleSchem-eagle-import:FIDUCIAL1X2
- removed FRAME1: (no value), symbol eagleSchem-eagle-import:FRAME-LETTER
- removed H1: (no value), symbol eagleSchem-eagle-import:STAND-OFFTIGHT
- removed J1, J2: (no value), symbol eagleSchem-eagle-import:CONN_01SMTSO-256-ET-0.165DIA
- removed J3: (no value), symbol eagleSchem-eagle-import:CONN_021X02_NO_SILK
- removed JP1: (no value), symbol eagleSchem-eagle-import:JUMPER-SMT_2_NO_SILK
- removed JP3: (no value), symbol eagleSchem-eagle-import:M03PTH
- removed LOGO1: (no value), symbol eagleSchem-eagle-import:SFE_LOGO_NAME_FLAME.1_INCH
- removed LOGO2: (no value), symbol eagleSchem-eagle-import:OSHW-LOGOS
- removed LOGO3: (no value), symbol eagleSchem-eagle-import:SFE_LOGO_FLAME.1_INCH
- removed R1: (no value), symbol eagleSchem-eagle-import:22KOHM-0603-1/10W-1%
- removed R2: (no value), symbol eagleSchem-eagle-import:1KOHM-0603-1/10W-1%
- removed R5: (no value), symbol eagleSchem-eagle-import:4.7KOHM-0603-1/10W-1%
- removed U1: (no value), symbol eagleSchem-eagle-import:ACS723
- removed U2: (no value), symbol eagleSchem-eagle-import:OPA344
- removed VR1, VR2: (no value), symbol eagleSchem-eagle-import:TRIMPOT-SMD-3MM-OPEN-1/10W-25%
- added C1: (no value), symbol schematicEagle-eagle-import:100PF-0603-50V-5%
- added C2, C3, C4: (no value), symbol schematicEagle-eagle-import:0.1UF-0603-25V-(+80/-20%)
- added C5: (no value), symbol schematicEagle-eagle-import:1.0NF/1000PF-0603-50V-10%
- added FD1, FD2, FD3, FD4: (no value), symbol schematicEagle-eagle-import:FIDUCIAL1X2
- added FRAME1: (no value), symbol schematicEagle-eagle-import:FRAME-LETTER
- added H1: (no value), symbol schematicEagle-eagle-import:STAND-OFFTIGHT
- added J1, J2: (no value), symbol schematicEagle-eagle-import:CONN_01SMTSO-256-ET-0.165DIA
- added J3: (no value), symbol schematicEagle-eagle-import:CONN_021X02_NO_SILK
- added JP1: (no value), symbol schematicEagle-eagle-import:JUMPER-SMT_2_NO_SILK
- added JP3: (no value), symbol schematicEagle-eagle-import:M03PTH
- added LOGO1: (no value), symbol schematicEagle-eagle-import:SFE_LOGO_NAME_FLAME.1_INCH
- added LOGO2: (no value), symbol schematicEagle-eagle-import:OSHW-LOGOS
- added LOGO3: (no value), symbol schematicEagle-eagle-import:SFE_LOGO_FLAME.1_INCH
- added R1: (no value), symbol schematicEagle-eagle-import:22KOHM-0603-1/10W-1%
- added R2: (no value), symbol schematicEagle-eagle-import:1KOHM-0603-1/10W-1%
- added R5: (no value), symbol schematicEagle-eagle-import:4.7KOHM-0603-1/10W-1%
- added U1: (no value), symbol schematicEagle-eagle-import:ACS723
- added U2: (no value), symbol schematicEagle-eagle-import:OPA344
- added VR1, VR2: (no value), symbol schematicEagle-eagle-import:TRIMPOT-SMD-3MM-OPEN-1/10W-25%
Connections:
- net BW_SEL: now also JP1.2, R5.1, U1.6 (BW_SEL)
- net GND: now also C2.2, C3.2, C4.1, C5.2, JP1.1, JP3.3, U1.5 (GND), U2.2 (P$V-), VR2.1 (CW)
- net VCC: now also C3.1, C4.2, JP3.1, R5.2, U1.8 (VCC), U2.5 (P$V+), VR2.3 (CCW)
- net VIOUT: now also C5.1, R2.2, U1.7 (VIOUT)
- net VO: now also C1.1, JP3.2, R1.1, U2.1 (OUT)
- new net: J1.P$1 (1), J3.2, U1.1 (IP+@1), U1.2 (IP+@2)
- new net: J2.P$1 (1), J3.1, U1.3 (IP-@1), U1.4 (IP-@2)
- new net: C2.1, U2.3 (+IN), VR2.2 (WIPER)
- new net: R2.1, VR1.1 (CW)
- new net: C1.2, R1.2, U2.4 (-IN), VR1.2 (WIPER), VR1.3 (CCW)
