File: PROJ/SPAR/14571/STAN/01/src/kicadBoard.kicad_sch (KiCad schematic)
At the start: 24 parts

Commit message: Quickly Adding Everything
Parts:
- removed C1, C4: (no value), symbol eagleSchem-eagle-import:0.1UF-0603-25V-(+80/-20%)
- removed FD1, FD2, FD3, FD4: (no value), symbol eagleSchem-eagle-import:FIDUCIALUFIDUCIAL
- removed FRAME2: (no value), symbol eagleSchem-eagle-import:FRAME-LETTER
- removed J1, J2: (no value), symbol eagleSchem-eagle-import:CONN_06NO_SILK_FEMALE_PTH
- removed J3, J4: (no value), symbol eagleSchem-eagle-import:QWIIC_CONNECTORJS-1MM
- removed JP3, JP4: (no value), symbol eagleSchem-eagle-import:STAND-OFF
- removed LOGO1: (no value), symbol eagleSchem-eagle-import:SFE_LOGO_NAME_FLAME.1_INCH
- removed LOGO2: (no value), symbol eagleSchem-eagle-import:SFE_LOGO_FLAME.1_INCH
- removed LOGO3: (no value), symbol eagleSchem-eagle-import:REVISION
- removed R1, R2: (no value), symbol eagleSchem-eagle-import:10KOHM-0603-1/10W-1%
- removed SJ1: (no value), symbol eagleSchem-eagle-import:JUMPER-SMT_2_NC_TRACE_SILK
- removed SJ2: (no value), symbol eagleSchem-eagle-import:JUMPER-PAD-3-NC_BY_TRACE
- removed SJ3, SJ4: (no value), symbol eagleSchem-eagle-import:JUMPER-SMT_3_1-NC_TRACE_SILK
- removed U$1: (no value), symbol eagleSchem-eagle-import:OSHW-LOGOS
- removed U1: (no value), symbol eagleSchem-eagle-import:MLX90393_MAGNETOMETER
- added C1, C4: (no value), symbol schematicEagle-eagle-import:0.1UF-0603-25V-(+80/-20%)
- added FD1, FD2, FD3, FD4: (no value), symbol schematicEagle-eagle-import:FIDUCIALUFIDUCIAL
- added FRAME2: (no value), symbol schematicEagle-eagle-import:FRAME-LETTER
- added J1, J2: (no value), symbol schematicEagle-eagle-import:CONN_06NO_SILK_FEMALE_PTH
- added J3, J4: (no value), symbol schematicEagle-eagle-import:QWIIC_CONNECTORJS-1MM
- added JP3, JP4: (no value), symbol schematicEagle-eagle-import:STAND-OFF
- added LOGO1: (no value), symbol schematicEagle-eagle-import:SFE_LOGO_NAME_FLAME.1_INCH
- added LOGO2: (no value), symbol schematicEagle-eagle-import:SFE_LOGO_FLAME.1_INCH
- added LOGO3: (no value), symbol schematicEagle-eagle-import:REVISION
- added R1, R2: (no value), symbol schematicEagle-eagle-import:10KOHM-0603-1/10W-1%
- added SJ1: (no value), symbol schematicEagle-eagle-import:JUMPER-SMT_2_NC_TRACE_SILK
- added SJ2: (no value), symbol schematicEagle-eagle-import:JUMPER-PAD-3-NC_BY_TRACE
- added SJ3, SJ4: (no value), symbol schematicEagle-eagle-import:JUMPER-SMT_3_1-NC_TRACE_SILK
- added U$1: (no value), symbol schematicEagle-eagle-import:OSHW-LOGOS
- added U1: (no value), symbol schematicEagle-eagle-import:MLX90393_MAGNETOMETER
Connections:
- net 3.3V: now also C1.1, C4.1, J1.2, J2.2, J3.2, J4.2, SJ1.2, SJ2.2, SJ3.1, SJ4.1, U1.15 (VDD), U1.8 (VDDIO)
- net A0: now also SJ3.2, U1.12 (A0)
- net A1: now also SJ4.2, U1.11 (A1)
- net CS: now also J2.6, SJ1.1, U1.2 (SENB/CS)
- net GND: now also C1.2, C4.2, J1.1, J2.1, J3.1, J4.1, SJ3.3, SJ4.3, U1.13 (GND)
- net INT: now also J1.5, U1.1 (INT)
- net MISO: now also J2.4, U1.6 (MISO)
- net SCL: now also J1.4, J2.3, J3.4, J4.4, R1.1, U1.3 (SCL/SCLK)
- net SDA: now also J1.3, J2.5, J3.3, J4.3, R2.1, U1.5 (SDA/MOSI)
- net TRIG: now also J1.6, U1.7 (INT/TRIG)
- new net: R2.2, SJ2.1
- new net: R1.2, SJ2.3
