File: PROJ/SPAR/15332/STAN/01/src/kicadBoard.kicad_sch (KiCad schematic)
At the start: 87 parts

Commit message: Quickly Adding Everything
Parts:
- removed A1: (no value), symbol eagleSchem-eagle-import:ANTENNA2.4GHZ-8.0X1.0MM
- removed C1: (no value), symbol eagleSchem-eagle-import:470NF-0402_TIGHT-6.3V-10%-X5R
- removed C11: (no value), symbol eagleSchem-eagle-import:47NF-0402_TIGHT-25V-10%-X7R
- removed C12, C13, C14, C15, C4: (no value), symbol eagleSchem-eagle-import:1.0UF-0402-TIGHT-16V-10%
- removed C16, C3, C5, C8: (no value), symbol eagleSchem-eagle-import:2.2UF-0402_TIGHT-10V-10%-X5R
- removed C17: (no value), symbol eagleSchem-eagle-import:DNP-CAP-0402-TIGHT
- removed C18: (no value), symbol eagleSchem-eagle-import:0.5PF-0402_TIGHT-20V-PM0.05PF-NP0
- removed C2: (no value), symbol eagleSchem-eagle-import:4.7UF-0402_TIGHT-6.3V-20%-X5R
- removed C6, C7: (no value), symbol eagleSchem-eagle-import:6PF-0402-TIGHT-50V-0.5%
- removed FD3, FD4: (no value), symbol eagleSchem-eagle-import:FIDUCIAL0.2MM
- removed FRAME1: (no value), symbol eagleSchem-eagle-import:FRAME-LETTER
- removed J1, J10, J11, J12, J13, J14, J15, J16, J17, J18, J19, J2, J20, J21, J23, J24, J25, J26, J27, J28, J29, J3, J30, J31, J32, J33, J34, J35, J36, J37, J39, J4, J40, J41, J42, J43, J44, J45, J46, J47, J48, J49, J5, J50, J51, J52, J53, J54, J55, J56, J57, J58, J59, J6, J7, J8, J9: (no value), symbol eagleSchem-eagle-import:PAD.4X.6
- removed J22, J38: (no value), symbol eagleSchem-eagle-import:PAD.35X.35
- removed L1: (no value), symbol eagleSchem-eagle-import:2.2μH-0805_WIDE-2.2μH-1.7A-0.14OHM
- removed L2: (no value), symbol eagleSchem-eagle-import:1.0μH-0805_WIDE-1.0μH-1.45A-0.106OHM-1.0MM_H
- removed L3: (no value), symbol eagleSchem-eagle-import:INDUCTOR-0402_TIGHT-2.7NH
- removed L4: (no value), symbol eagleSchem-eagle-import:INDUCTOR-0402_TIGHT-2.0NH
- removed LOGO1: (no value), symbol eagleSchem-eagle-import:SFE_LOGO_FLAME.05_INCH_INTERNAL
- removed R2: (no value), symbol eagleSchem-eagle-import:0OHM-0402T-1/10W
- removed U1: (no value), symbol eagleSchem-eagle-import:AMBIQ-APOLLO3KBR
- removed Y1: (no value), symbol eagleSchem-eagle-import:CRYSTAL-32MHZ-SMD-2.0X1.6MM
- added A1: (no value), symbol schematicEagle-eagle-import:ANTENNA2.4GHZ-8.0X1.0MM
- added C1: (no value), symbol schematicEagle-eagle-import:470NF-0402_TIGHT-6.3V-10%-X5R
- added C11: (no value), symbol schematicEagle-eagle-import:47NF-0402_TIGHT-25V-10%-X7R
- added C12, C13, C14, C15, C4: (no value), symbol schematicEagle-eagle-import:1.0UF-0402-TIGHT-16V-10%
- added C16, C3, C5, C8: (no value), symbol schematicEagle-eagle-import:2.2UF-0402_TIGHT-10V-10%-X5R
- added C17: (no value), symbol schematicEagle-eagle-import:DNP-CAP-0402-TIGHT
- added C18: (no value), symbol schematicEagle-eagle-import:0.5PF-0402_TIGHT-20V-PM0.05PF-NP0
- added C2: (no value), symbol schematicEagle-eagle-import:4.7UF-0402_TIGHT-6.3V-20%-X5R
- added C6, C7: (no value), symbol schematicEagle-eagle-import:6PF-0402-TIGHT-50V-0.5%
- added FD3, FD4: (no value), symbol schematicEagle-eagle-import:FIDUCIAL0.2MM
- added FRAME1: (no value), symbol schematicEagle-eagle-import:FRAME-LETTER
- added J1, J10, J11, J12, J13, J14, J15, J16, J17, J18, J19, J2, J20, J21, J23, J24, J25, J26, J27, J28, J29, J3, J30, J31, J32, J33, J34, J35, J36, J37, J39, J4, J40, J41, J42, J43, J44, J45, J46, J47, J48, J49, J5, J50, J51, J52, J53, J54, J55, J56, J57, J58, J59, J6, J7, J8, J9: (no value), symbol schematicEagle-eagle-import:PAD.4X.6
- added J22, J38: (no value), symbol schematicEagle-eagle-import:PAD.35X.35
- added L1: (no value), symbol schematicEagle-eagle-import:2.2μH-0805_WIDE-2.2μH-1.7A-0.14OHM
- added L2: (no value), symbol schematicEagle-eagle-import:1.0μH-0805_WIDE-1.0μH-1.45A-0.106OHM-1.0MM_H
- added L3: (no value), symbol schematicEagle-eagle-import:INDUCTOR-0402_TIGHT-2.7NH
- added L4: (no value), symbol schematicEagle-eagle-import:INDUCTOR-0402_TIGHT-2.0NH
- added LOGO1: (no value), symbol schematicEagle-eagle-import:SFE_LOGO_FLAME.05_INCH_INTERNAL
- added R2: (no value), symbol schematicEagle-eagle-import:0OHM-0402T-1/10W
- added U1: (no value), symbol schematicEagle-eagle-import:AMBIQ-APOLLO3KBR
- added Y1: (no value), symbol schematicEagle-eagle-import:CRYSTAL-32MHZ-SMD-2.0X1.6MM
Connections:
- net AD16: now also J42.1, U1.D4 (GPIO16)
- net AD34: now also J31.1, U1.C6 (GPIO34)
- net BOOTLOAD: now also J7.1, U1.H9 (GPIO47)
- net D0: now also J51.1, U1.H4 (GPIO0)
- net D1: now also J49.1, U1.G4 (GPIO1)
- net D10: now also J8.1, U1.G8 (GPIO10)
- net D14: now also J20.1, U1.D7 (GPIO14)
- net D15: now also J29.1, U1.C7 (GPIO15)
- net D17: now also J43.1, U1.D3 (GPIO17)
- net D2: now also J48.1, U1.F4 (GPIO2)
- net D3: now also J54.1, U1.G5 (GPIO3)
- net D36: now also J55.1, U1.H6 (GPIO36)
- net D38: now also J56.1, U1.J6 (GPIO38)
- net D40: now also J5.1, U1.J9 (GPIO40)
- net D41: now also J45.1, U1.E5 (GPIO41)
- net D7: now also J13.1, U1.F9 (GPIO7)
- net D8: now also J11.1, U1.F8 (GPIO8)
- net D9: now also J6.1, U1.G7 (GPIO9)
- net DVDD: now also C11.1, U1.H3 (DVDD)
- net GND: now also C1.2, C11.2, C12.2, C13.2, C14.2, C15.2, C16.2, C17.2, C18.2, C2.2, C3.2, C4.2, C5.2, C6.1, C7.1, C8.2, J1.1, J22.1, J38.1, J39.1, J47.1, J59.1, U1.B3 (VSSP), U1.C2 (VSSB), U1.E2 (VSS), U1.E3 (VSSA), U1.F2 (VSSBA), U1.H1 (VSSVCO), U1.H2 (VSSS), U1.J2 (RFIOM)
- net RFIOP: now also C17.1, L3.1, U1.J1 (RFIOP)
- net RXI-0: now also J3.1, U1.H8 (GPIO49)
- net SWDCK: now also J2.1, U1.G6 (GPIO20/SWDCK)
- net SWDIO: now also J10.1, U1.F7 (GPIO21/SWDIO)
- net TXO-0: now also J9.1, U1.G9 (GPIO48)
- net VDD: now also C12.1, C13.1, C14.1, C15.1, C16.1, J36.1, J37.1, U1.B1 (VDDB), U1.B2 (VDDP), U1.C4 (VDDA), U1.F3 (VDDH), U1.J4 (VCC)
- net XI: now also J35.1, U1.B4 (XI)
- net XO: now also J34.1, U1.A4 (XO)
- net ~{AD11}: now also J32.1, U1.B5 (GPIO11)
- net ~{AD12}: now also J26.1, U1.A7 (GPIO12)
- net ~{AD13}: now also J28.1, U1.B7 (GPIO13)
- net ~{AD29}: now also J33.1, U1.A5 (GPIO29)
- net ~{AD31}: now also J44.1, U1.D5 (GPIO31)
- net ~{AD32}: now also J24.1, U1.E6 (GPIO32)
- net ~{AD33/SWO}: now also J30.1, U1.B6 (GPIO33)
- net ~{AD35}: now also J14.1, U1.D6 (GPIO35)
- net ~{D18}: now also J41.1, U1.C5 (GPIO18)
- net ~{D19}: now also J40.1, U1.C3 (GPIO19)
- net ~{D22}: now also J17.1, U1.C9 (GPIO22)
- net ~{D23}: now also J18.1, U1.D8 (GPIO23)
- net ~{D24}: now also J16.1, U1.C8 (GPIO24)
- net ~{D25}: now also J25.1, U1.A8 (GPIO25)
- net ~{D26}: now also J27.1, U1.B8 (GPIO26)
- net ~{D27}: now also J19.1, U1.B9 (GPIO27)
- net ~{D28}: now also J21.1, U1.A9 (GPIO28)
- net ~{D37}: now also J57.1, U1.H7 (GPIO37)
- net ~{D39}: now also J4.1, U1.J8 (GPIO39)
- net ~{D42}: now also J53.1, U1.H5 (GPIO42)
- net ~{D43}: now also J52.1, U1.J5 (GPIO43)
- net ~{D44}: now also J58.1, U1.J7 (GPIO44)
- net ~{D45}: now also J46.1, U1.F5 (GPIO45)
- net ~{D4}: now also J15.1, U1.D9 (GPIO4)
- net ~{D5}: now also J12.1, U1.E9 (GPIO5)
- net ~{D6}: now also J23.1, U1.E8 (GPIO6)
- net ~{RST}: now also J50.1, U1.G3 (NRST)
- new net: C8.1, U1.E1 (VDDS)
- new net: C2.1, L2.2, R2.1, U1.C1 (VDDBH)
- new net: C4.1, R2.2, U1.G2 (VDCDCRF)
- new net: C5.1, U1.D2 (VDDF)
- new net: L1.1, U1.A1 (SIMOBUCK_SW)
- new net: L1.2, U1.A2 (SIMOBUCK_SWSEL)
- new net: C6.2, U1.F1 (XO32MP), Y1.3 (2)
- new net: C3.1, U1.A3 (VDDC)
- new net: C1.1, U1.A6 (ADC_VREF)
- new net: L2.1, U1.D1 (VDDBH_SW)
- new net: C7.2, U1.G1 (XO32MM), Y1.1
- new net: C18.1, L3.2, L4.1
- new net: A1.FEED (SIGNAL), L4.2
