File: PROJ/SPAR/15440/STAN/01/src/kicadBoard.kicad_sch (KiCad schematic)
At the start: 27 parts

Commit message: Quickly Adding Everything
Parts:
- removed C1, C2: (no value), symbol eagleSchem-eagle-import:0.1UF-0603-25V-(+80/-20%)
- removed D1: (no value), symbol eagleSchem-eagle-import:LED-RED0603
- removed FD1, FD2, FD3, FD4: (no value), symbol eagleSchem-eagle-import:FIDUCIAL1X2
- removed FRAME1: (no value), symbol eagleSchem-eagle-import:FRAME-LETTER
- removed H1, H2, H4: (no value), symbol eagleSchem-eagle-import:STAND-OFF
- removed J1, J2: (no value), symbol eagleSchem-eagle-import:I2C_STANDARDQWIIC
- removed J3: (no value), symbol eagleSchem-eagle-import:I2C_STANDARD_NO_SILK
- removed J4: (no value), symbol eagleSchem-eagle-import:CONN_021X02_NO_SILK
- removed JP1: (no value), symbol eagleSchem-eagle-import:JUMPER-SMT_2_NC_TRACE_NO-SILK
- removed JP2: (no value), symbol eagleSchem-eagle-import:JUMPER-PAD-2-NC_BY_TRACENO_SILK
- removed JP3: (no value), symbol eagleSchem-eagle-import:JUMPER-SMT_3_1-NC_TRACE_NO-SILK
- removed JP4: (no value), symbol eagleSchem-eagle-import:JUMPER-SMT_3_2-NC_TRACE_NO-SILK
- removed LOGO1: (no value), symbol eagleSchem-eagle-import:SFE_LOGO_NAME.1_INCH
- removed LOGO4: (no value), symbol eagleSchem-eagle-import:OSHW-LOGOS
- removed R1, R2, R3, R4: (no value), symbol eagleSchem-eagle-import:4.7KOHM-0603-1/10W-1%
- removed R5: (no value), symbol eagleSchem-eagle-import:1KOHM-0603-1/10W-1%
- removed U1: (no value), symbol eagleSchem-eagle-import:BME280
- added C1, C2: (no value), symbol schematicEagle-eagle-import:0.1UF-0603-25V-(+80/-20%)
- added D1: (no value), symbol schematicEagle-eagle-import:LED-RED0603
- added FD1, FD2, FD3, FD4: (no value), symbol schematicEagle-eagle-import:FIDUCIAL1X2
- added FRAME1: (no value), symbol schematicEagle-eagle-import:FRAME-LETTER
- added H1, H2, H4: (no value), symbol schematicEagle-eagle-import:STAND-OFF
- added J1, J2: (no value), symbol schematicEagle-eagle-import:I2C_STANDARDQWIIC
- added J3: (no value), symbol schematicEagle-eagle-import:I2C_STANDARD_NO_SILK
- added J4: (no value), symbol schematicEagle-eagle-import:CONN_021X02_NO_SILK
- added JP1: (no value), symbol schematicEagle-eagle-import:JUMPER-SMT_2_NC_TRACE_NO-SILK
- added JP2: (no value), symbol schematicEagle-eagle-import:JUMPER-PAD-2-NC_BY_TRACENO_SILK
- added JP3: (no value), symbol schematicEagle-eagle-import:JUMPER-SMT_3_1-NC_TRACE_NO-SILK
- added JP4: (no value), symbol schematicEagle-eagle-import:JUMPER-SMT_3_2-NC_TRACE_NO-SILK
- added LOGO1: (no value), symbol schematicEagle-eagle-import:SFE_LOGO_NAME.1_INCH
- added LOGO4: (no value), symbol schematicEagle-eagle-import:OSHW-LOGOS
- added R1, R2, R3, R4: (no value), symbol schematicEagle-eagle-import:4.7KOHM-0603-1/10W-1%
- added R5: (no value), symbol schematicEagle-eagle-import:1KOHM-0603-1/10W-1%
- added U1: (no value), symbol schematicEagle-eagle-import:BME280
Connections:
- net 3.3V: now also C1.1, C2.1, J1.2, J2.2, J3.2, JP1.2, JP2.2, JP4.2, R2.2, U1.6 (VDDIO), U1.8 (VDD)
- net GND: now also C1.2, C2.2, D1.C, J1.1, J2.1, J3.1, JP3.1, U1.1 (GND), U1.7 (GND)
- net SCK/SCL: now also J1.4, J2.4, J3.4, R4.1, U1.4 (SCK/SCL)
- net SDI/SDA: now also J1.3, J2.3, J3.3, R3.1, U1.3 (SDI/SDA)
- net SDO/ADR: now also J4.2, JP3.2, U1.5 (SDO/ADR)
- net ~{CS}: now also J4.1, R1.1, U1.2 (~{CS})
- new net: JP4.1, R4.2
- new net: JP4.3, R3.2
- new net: D1.A, R5.1
- new net: JP1.1, R5.2
- new net: JP2.1, R1.2
- new net: JP3.3, R2.1
