File: PROJ/SPAR/17119/STAN/01/src/kicadBoard.kicad_sch (KiCad schematic)
At the start: 22 parts

Commit message: Quickly Adding Everything
Parts:
- removed D1: (no value), symbol eagleSchem-eagle-import:DIODE-SCHOTTKY-BAT60A
- removed D1_BP0: (no value), symbol eagleSchem-eagle-import:JUMPER-SMT_2_NO_SILK
- removed FD1, FD2, FD3, FD4: (no value), symbol eagleSchem-eagle-import:FIDUCIAL1X2
- removed FRAME1: (no value), symbol eagleSchem-eagle-import:FRAME-LETTER
- removed I2C0: (no value), symbol eagleSchem-eagle-import:JUMPER-SMT_3_NO_SILK
- removed J1: (no value), symbol eagleSchem-eagle-import:TEENSYNOSILK
- removed J2, J3: (no value), symbol eagleSchem-eagle-import:QWIIC_CONNECTORJS-1MM
- removed J4, J5: (no value), symbol eagleSchem-eagle-import:QWIIC_CONNECTOR
- removed J6: (no value), symbol eagleSchem-eagle-import:CONN_021X02_NO_SILK
- removed LOGO1: (no value), symbol eagleSchem-eagle-import:SFE_LOGO_NAME_FLAME.1_INCH
- removed LOGO2: (no value), symbol eagleSchem-eagle-import:SFE_LOGO_FLAME.1_INCH
- removed LOGO3: (no value), symbol eagleSchem-eagle-import:OSHW-LOGOS
- removed LOGO4: (no value), symbol eagleSchem-eagle-import:QWIIC_LOGO_5MM
- removed R3, R4: (no value), symbol eagleSchem-eagle-import:4.7KOHM-0603-1/10W-1%
- removed S1: (no value), symbol eagleSchem-eagle-import:MOMENTARY-SWITCH-SPST-SMD-5.2MM-TALL
- removed UNK3V3_ISO0: (no value), symbol eagleSchem-eagle-import:JUMPER-SMT_2_NC_TRACE_SILK
- added D1: (no value), symbol schematicEagle-eagle-import:DIODE-SCHOTTKY-BAT60A
- added D1_BP0: (no value), symbol schematicEagle-eagle-import:JUMPER-SMT_2_NO_SILK
- added FD1, FD2, FD3, FD4: (no value), symbol schematicEagle-eagle-import:FIDUCIAL1X2
- added FRAME1: (no value), symbol schematicEagle-eagle-import:FRAME-LETTER
- added I2C0: (no value), symbol schematicEagle-eagle-import:JUMPER-SMT_3_NO_SILK
- added J1: (no value), symbol schematicEagle-eagle-import:TEENSYNOSILK
- added J2, J3: (no value), symbol schematicEagle-eagle-import:QWIIC_CONNECTORJS-1MM
- added J4, J5: (no value), symbol schematicEagle-eagle-import:QWIIC_CONNECTOR
- added J6: (no value), symbol schematicEagle-eagle-import:CONN_021X02_NO_SILK
- added LOGO1: (no value), symbol schematicEagle-eagle-import:SFE_LOGO_NAME_FLAME.1_INCH
- added LOGO2: (no value), symbol schematicEagle-eagle-import:SFE_LOGO_FLAME.1_INCH
- added LOGO3: (no value), symbol schematicEagle-eagle-import:OSHW-LOGOS
- added LOGO4: (no value), symbol schematicEagle-eagle-import:QWIIC_LOGO_5MM
- added R3, R4: (no value), symbol schematicEagle-eagle-import:4.7KOHM-0603-1/10W-1%
- added S1: (no value), symbol schematicEagle-eagle-import:MOMENTARY-SWITCH-SPST-SMD-5.2MM-TALL
- added UNK3V3_ISO0: (no value), symbol schematicEagle-eagle-import:JUMPER-SMT_2_NC_TRACE_SILK
Connections:
- net 3.3V: now also D1.C, D1_BP0.2, I2C0.2, J2.2, J3.2, J4.2, J5.2, UNK3V3_ISO0.1
- net GND: now also J1.AGND, J1.GND, J1.GND1, J2.1, J3.1, J4.1, J5.1, J6.1, S1.3 (2)
- net NC: now also J1.3.3V
- net SCL: now also J1.19 (A5/19/SCL0), J2.4, J3.4, J4.4, J5.4, R3.1
- net SDA: now also J1.18 (A4/18/SDA0), J2.3, J3.3, J4.3, J5.3, R4.1
- net VBAT: now also J1.VBAT
- net VIN: now also J1.VIN
- net VUSB: now also J1.VUSB
- new net: D1.A, D1_BP0.1, J6.2
- new net: J1.3V, UNK3V3_ISO0.2
- new net: J1.PROG, S1.1
- new net: I2C0.3, R4.2
- new net: I2C0.1, R3.2
