File: PROJ/SPAR/18521/STAN/01/src/kicadBoard.kicad_sch (KiCad schematic)
At the start: 30 parts

Commit message: Quickly Adding Everything
Parts:
- removed C1: (no value), symbol eagleSchem-eagle-import:0.1UF-0603-25V-(+80/-20%)
- removed D1: (no value), symbol eagleSchem-eagle-import:LED-RED0603
- removed FD1, FD2, FD3, FD4: (no value), symbol eagleSchem-eagle-import:FIDUCIALUFIDUCIAL
- removed FRAME1: (no value), symbol eagleSchem-eagle-import:FRAME-LETTER
- removed I2C0: (no value), symbol eagleSchem-eagle-import:JUMPER-SMT_3_2-NC_TRACE_SILK
- removed J1: (no value), symbol eagleSchem-eagle-import:I2C_STANDARD_NO_SILK
- removed J2, J3: (no value), symbol eagleSchem-eagle-import:QWIIC_CONNECTORJS-1MM
- removed J4, J5: (no value), symbol eagleSchem-eagle-import:CONN_01PTH_NO_SILK_YES_STOP
- removed JP1: (no value), symbol eagleSchem-eagle-import:JUMPER-SMT_2_NC_TRACE_SILK
- removed JP10, JP4: (no value), symbol eagleSchem-eagle-import:JUMPER-SMT_3_1-NC_TRACE_NO-SILK
- removed JP11, JP5: (no value), symbol eagleSchem-eagle-import:JUMPER-SMT_3_NO_NO_SILK
- removed JP2, JP3, JP8, JP9: (no value), symbol eagleSchem-eagle-import:STAND-OFF
- removed LOGO1: (no value), symbol eagleSchem-eagle-import:OSHW-LOGOMINI
- removed LOGO4: (no value), symbol eagleSchem-eagle-import:SFE_LOGO_NAME_FLAME.1_INCH
- removed R1: (no value), symbol eagleSchem-eagle-import:1KOHM-0603-1/10W-1%
- removed R2, R6: (no value), symbol eagleSchem-eagle-import:10KOHM-0603-1/10W-1%
- removed R4, R5: (no value), symbol eagleSchem-eagle-import:2.2KOHM-0603-1/10W-1%
- removed U2: (no value), symbol eagleSchem-eagle-import:AS6212WLCSP
- added C1: (no value), symbol schematicEagle-eagle-import:0.1UF-0603-25V-(+80/-20%)
- added D1: (no value), symbol schematicEagle-eagle-import:LED-RED0603
- added FD1, FD2, FD3, FD4: (no value), symbol schematicEagle-eagle-import:FIDUCIALUFIDUCIAL
- added FRAME1: (no value), symbol schematicEagle-eagle-import:FRAME-LETTER
- added I2C0: (no value), symbol schematicEagle-eagle-import:JUMPER-SMT_3_2-NC_TRACE_SILK
- added J1: (no value), symbol schematicEagle-eagle-import:I2C_STANDARD_NO_SILK
- added J2, J3: (no value), symbol schematicEagle-eagle-import:QWIIC_CONNECTORJS-1MM
- added J4, J5: (no value), symbol schematicEagle-eagle-import:CONN_01PTH_NO_SILK_YES_STOP
- added JP1: (no value), symbol schematicEagle-eagle-import:JUMPER-SMT_2_NC_TRACE_SILK
- added JP10, JP4: (no value), symbol schematicEagle-eagle-import:JUMPER-SMT_3_1-NC_TRACE_NO-SILK
- added JP11, JP5: (no value), symbol schematicEagle-eagle-import:JUMPER-SMT_3_NO_NO_SILK
- added JP2, JP3, JP8, JP9: (no value), symbol schematicEagle-eagle-import:STAND-OFF
- added LOGO1: (no value), symbol schematicEagle-eagle-import:OSHW-LOGOMINI
- added LOGO4: (no value), symbol schematicEagle-eagle-import:SFE_LOGO_NAME_FLAME.1_INCH
- added R1: (no value), symbol schematicEagle-eagle-import:1KOHM-0603-1/10W-1%
- added R2, R6: (no value), symbol schematicEagle-eagle-import:10KOHM-0603-1/10W-1%
- added R4, R5: (no value), symbol schematicEagle-eagle-import:2.2KOHM-0603-1/10W-1%
- added U2: (no value), symbol schematicEagle-eagle-import:AS6212WLCSP
Connections:
- net 3.3V: now also C1.1, I2C0.2, J1.2, J2.2, J3.2, JP1.2, R2.1, R6.1, U2.B1 (VCC)
- net ADD0: now also J5.1, JP4.2, JP5.2, U2.B2 (ADD0)
- net ALERT/ADD1: now also J4.1, JP10.2, JP11.2, U2.A2 (ALERT/ADD1)
- net GND: now also C1.2, D1.C, J1.1, J2.1, J3.1, JP11.3, JP4.3, U2.A1 (GND)
- net SCL: now also J1.4, J2.4, J3.4, JP10.1, JP5.3, R5.1, U2.A3 (SCL)
- net SDA: now also J1.3, J2.3, J3.3, JP11.1, JP4.1, R4.1, U2.B3 (SDA)
- new net: JP10.3, R6.2
- new net: I2C0.3, R4.2
- new net: I2C0.1, R5.2
- new net: JP5.1, R2.2
- new net: JP1.1, R1.1
- new net: D1.A, R1.2
