File: PROJ/SPAR/18721/STAN/01/src/kicadBoard.kicad_sch (KiCad schematic)
At the start: 78 parts

Commit message: Quickly Adding Everything
Parts:
- removed C1, C17, C18, C2, C20, C21, C22, C23, C24, C25, C29, C3: (no value), symbol eagleSchem-eagle-import:0.1UF-0402T-6.3V-10%-X7R
- removed C10, C7: (no value), symbol eagleSchem-eagle-import:4.7UF-0402_TIGHT-6.3V-20%-X5R
- removed C16, C5: (no value), symbol eagleSchem-eagle-import:15PF-0402T-50V-5%
- removed C26, C27, C28, C4, C9: (no value), symbol eagleSchem-eagle-import:2.2UF-0402_TIGHT-10V-10%-X5R
- removed C8: (no value), symbol eagleSchem-eagle-import:1.0UF-0402T-16V-10%
- removed D1: (no value), symbol eagleSchem-eagle-import:LED-YELLOW0603
- removed D2: (no value), symbol eagleSchem-eagle-import:DIODE-SCHOTTKY-BAT20J
- removed D3: (no value), symbol eagleSchem-eagle-import:LED-RED0603
- removed D4: (no value), symbol eagleSchem-eagle-import:LED-BLUE0603
- removed D5: (no value), symbol eagleSchem-eagle-import:WS2812_2020
- removed FD1, FD2, FD3, FD4: (no value), symbol eagleSchem-eagle-import:FIDUCIALUFIDUCIAL
- removed FRAME1: (no value), symbol eagleSchem-eagle-import:FRAME-LEDGER
- removed H1, H2, H3, H4: (no value), symbol eagleSchem-eagle-import:STAND-OFF
- removed I2C0: (no value), symbol eagleSchem-eagle-import:JUMPER-SMT_3_2-NC_TRACE_SILK
- removed J1: (no value), symbol eagleSchem-eagle-import:CORTEX_JTAG_DEBUG_MINIMUM_PTH
- removed J3: (no value), symbol eagleSchem-eagle-import:QWIIC_CONNECTORJS-1MM
- removed J4: (no value), symbol eagleSchem-eagle-import:JST_2MM_MALE
- removed J5: (no value), symbol eagleSchem-eagle-import:USB_C_4-LAYER-ISOLATED
- removed J6: (no value), symbol eagleSchem-eagle-import:MICRO-SD-PUSH-PUSH-EXT-PIN
- removed J7: (no value), symbol eagleSchem-eagle-import:CONN_161X16_NO_SILK
- removed J8: (no value), symbol eagleSchem-eagle-import:CONN_12NO_SILK
- removed J9: (no value), symbol eagleSchem-eagle-import:MIKROBUS_SMD_BLACK1
- removed LOGO1: (no value), symbol eagleSchem-eagle-import:OSHW-LOGOS
- removed LOGO2: (no value), symbol eagleSchem-eagle-import:SFE_LOGO_NAME.1_INCH
- removed PWR0: (no value), symbol eagleSchem-eagle-import:JUMPER-SMT_2_NC_TRACE_SILK
- removed Q1: (no value), symbol eagleSchem-eagle-import:MOSFET_PCH-DMG2305UX-7
- removed R1, R4: (no value), symbol eagleSchem-eagle-import:5.1KOHM-0402T-1/16W-1%
- removed R10, R17: (no value), symbol eagleSchem-eagle-import:2.2KOHM-0402T-1/16W-1%
- removed R11, R2, R3, R5, R8: (no value), symbol eagleSchem-eagle-import:1KOHM-0402T-1/16W-1%
- removed R12, R13: (no value), symbol eagleSchem-eagle-import:27OHM
- removed R15, R16, R9: (no value), symbol eagleSchem-eagle-import:10KOHM-0402T-1/16W-1%
- removed R6: (no value), symbol eagleSchem-eagle-import:2.0KOHM-0603-1/10W-5%
- removed R7: (no value), symbol eagleSchem-eagle-import:200OHM-0402T-1/16W-1%
- removed S1, S2: (no value), symbol eagleSchem-eagle-import:MOMENTARY-SWITCH-SPST-SMD-5.2MM-TALL
- removed TP1, TP2, TP3: (no value), symbol eagleSchem-eagle-import:TEST-POINT3X4
- removed U$17, U$73: (no value), symbol eagleSchem-eagle-import:RASPI_RP2040_LOGO_10MM
- removed U2: (no value), symbol eagleSchem-eagle-import:MAX17048DFN8
- removed U3: (no value), symbol eagleSchem-eagle-import:MCP73831
- removed U4: (no value), symbol eagleSchem-eagle-import:W25QXX128MBIT-6X5-SKINNY_CENTER
- removed U5: (no value), symbol eagleSchem-eagle-import:RP2040
- removed U7: (no value), symbol eagleSchem-eagle-import:V_REG_AP2112K-3.3V
- removed Y2: (no value), symbol eagleSchem-eagle-import:CRYSTAL-12MHZ
- added C1, C17, C18, C2, C20, C21, C22, C23, C24, C25, C29, C3: (no value), symbol schematicEagle-eagle-import:0.1UF-0402T-6.3V-10%-X7R
- added C10, C7: (no value), symbol schematicEagle-eagle-import:4.7UF-0402_TIGHT-6.3V-20%-X5R
- added C16, C5: (no value), symbol schematicEagle-eagle-import:15PF-0402T-50V-5%
- added C26, C27, C28, C4, C9: (no value), symbol schematicEagle-eagle-import:2.2UF-0402_TIGHT-10V-10%-X5R
- added C8: (no value), symbol schematicEagle-eagle-import:1.0UF-0402T-16V-10%
- added D1: (no value), symbol schematicEagle-eagle-import:LED-YELLOW0603
- added D2: (no value), symbol schematicEagle-eagle-import:DIODE-SCHOTTKY-BAT20J
- added D3: (no value), symbol schematicEagle-eagle-import:LED-RED0603
- added D4: (no value), symbol schematicEagle-eagle-import:LED-BLUE0603
- added D5: (no value), symbol schematicEagle-eagle-import:WS2812_2020
- added FD1, FD2, FD3, FD4: (no value), symbol schematicEagle-eagle-import:FIDUCIALUFIDUCIAL
- added FRAME1: (no value), symbol schematicEagle-eagle-import:FRAME-LEDGER
- added H1, H2, H3, H4: (no value), symbol schematicEagle-eagle-import:STAND-OFF
- added I2C0: (no value), symbol schematicEagle-eagle-import:JUMPER-SMT_3_2-NC_TRACE_SILK
- added J1: (no value), symbol schematicEagle-eagle-import:CORTEX_JTAG_DEBUG_MINIMUM_PTH
- added J3: (no value), symbol schematicEagle-eagle-import:QWIIC_CONNECTORJS-1MM
- added J4: (no value), symbol schematicEagle-eagle-import:JST_2MM_MALE
- added J5: (no value), symbol schematicEagle-eagle-import:USB_C_4-LAYER-ISOLATED
- added J6: (no value), symbol schematicEagle-eagle-import:MICRO-SD-PUSH-PUSH-EXT-PIN
- added J7: (no value), symbol schematicEagle-eagle-import:CONN_161X16_NO_SILK
- added J8: (no value), symbol schematicEagle-eagle-import:CONN_12NO_SILK
- added J9: (no value), symbol schematicEagle-eagle-import:MIKROBUS_SMD_BLACK1
- added LOGO1: (no value), symbol schematicEagle-eagle-import:OSHW-LOGOS
- added LOGO2: (no value), symbol schematicEagle-eagle-import:SFE_LOGO_NAME.1_INCH
- added PWR0: (no value), symbol schematicEagle-eagle-import:JUMPER-SMT_2_NC_TRACE_SILK
- added Q1: (no value), symbol schematicEagle-eagle-import:MOSFET_PCH-DMG2305UX-7
- added R1, R4: (no value), symbol schematicEagle-eagle-import:5.1KOHM-0402T-1/16W-1%
- added R10, R17: (no value), symbol schematicEagle-eagle-import:2.2KOHM-0402T-1/16W-1%
- added R11, R2, R3, R5, R8: (no value), symbol schematicEagle-eagle-import:1KOHM-0402T-1/16W-1%
- added R12, R13: (no value), symbol schematicEagle-eagle-import:27OHM
- added R15, R16, R9: (no value), symbol schematicEagle-eagle-import:10KOHM-0402T-1/16W-1%
- added R6: (no value), symbol schematicEagle-eagle-import:2.0KOHM-0603-1/10W-5%
- added R7: (no value), symbol schematicEagle-eagle-import:200OHM-0402T-1/16W-1%
- added S1, S2: (no value), symbol schematicEagle-eagle-import:MOMENTARY-SWITCH-SPST-SMD-5.2MM-TALL
- added TP1, TP2, TP3: (no value), symbol schematicEagle-eagle-import:TEST-POINT3X4
- added U$17, U$73: (no value), symbol schematicEagle-eagle-import:RASPI_RP2040_LOGO_10MM
- added U2: (no value), symbol schematicEagle-eagle-import:MAX17048DFN8
- added U3: (no value), symbol schematicEagle-eagle-import:MCP73831
- added U4: (no value), symbol schematicEagle-eagle-import:W25QXX128MBIT-6X5-SKINNY_CENTER
- added U5: (no value), symbol schematicEagle-eagle-import:RP2040
- added U7: (no value), symbol schematicEagle-eagle-import:V_REG_AP2112K-3.3V
- added Y2: (no value), symbol schematicEagle-eagle-import:CRYSTAL-12MHZ
Connections:
- net 1.1V: now also C24.1, C25.1, C26.1, U5.23 (VDD_1V1), U5.45 (LDO_OUT), U5.50 (VDD_1V1)
- net 3.3V: now also C17.1, C18.1, C2.1, C20.1, C21.1, C22.1, C23.1, C27.1, C29.1, C3.1, C4.1, C9.1, D5.VCC, I2C0.2, J1.1 (VCC), J3.2, J6.4 (VCC), J7.2, J9.7 (+3.3V), PWR0.2, R7.2, R9.2, U4.8 (VDD), U5.1 (VDDIO), U5.10 (VDDIO), U5.22 (VDDIO), U5.33 (VDDIO), U5.42 (VDDIO), U5.44 (LDO_IN), U5.48 (USB_VDD), U5.49 (VDDIO), U7.5 (OUT)
- net ADC0: now also J7.5, J9.1 (AN), U5.38 (GPIO26/ADC0)
- net ADC1: now also J7.6, U5.39 (GPIO27/ADC1)
- net ADC2: now also J7.7, U5.40 (GPIO28/ADC2)
- net ADC3: now also J7.8, U5.41 (GPIO29/ADC3)
- net AVDD: now also C28.1, J7.3, R7.1, U5.43 (ADC_VDD)
- net EN: now also J8.2, R16.1, U7.3 (EN)
- net GND: now also C1.2, C10.2, C16.1, C17.2, C18.2, C2.2, C20.2, C21.2, C22.2, C23.2, C24.2, C25.2, C26.2, C27.2, C28.2, C29.2, C3.2, C4.2, C5.1, C7.2, C8.2, C9.2, D5.GND, J1.3 (GND), J1.5 (GND), J1.9 (GND), J3.1, J4.1 (-), J5.GND, J5.GND2 (GND), J6.10 (GND), J6.11 (GND), J6.12 (GND), J6.13 (GND), J6.6 (GND), J6.9 (DET), J7.4, J9.8 (GND), J9.9 (GND2), R1.2, R15.1, R3.1, R4.2, R6.1, R8.1, S1.1, S2.1, U2.1 (CTG), U2.4 (GND), U2.6 (QSTRT), U2.9 (GND), U3.2 (VSS), U4.4 (GND), U5.19 (TESTEN), U5.EPAD (GND), U7.2 (GND)
- net GPIO13: now also J9.2 (RST), U5.16 (GPIO13)
- net GPIO16: now also J8.4, J9.16 (PWM), U5.27 (GPIO16)
- net GPIO17: now also J8.5, J9.15 (INT), U5.28 (GPIO17)
- net GPIO18: now also J8.6, U5.29 (GPIO18)
- net GPIO19: now also J8.7, U5.30 (GPIO19)
- net GPIO20: now also J8.8, U5.31 (GPIO20)
- net GPIO21: now also J8.9, U5.32 (GPIO21)
- net GPIO22: now also J8.10, U5.34 (GPIO22)
- net I2C1_SCL/GPIO23: now also J3.4, J8.11, J9.12 (SCL), R10.1, U2.7 (SCL), U5.35 (GPIO23), U5.9 (GPIO7)
- net I2C1_SDA: now also J3.3, J8.12, J9.11 (SDA), R17.1, U2.8 (SDA), U5.8 (GPIO6)
- net LED_BUILTIN: now also D4.A, U5.37 (GPIO25)
- net QSPI-0: now also U4.5 (D0/DI), U5.53 (QSPI_SD0)
- net QSPI-1: now also U4.2 (D1/DO), U5.55 (QSPI_SD1)
- net QSPI-2: now also U4.3 (D2/~{WP}), U5.54 (QSPI_SD2)
- net QSPI-3: now also U4.7 (D3/~{HOLD}), U5.51 (QSPI_SD3)
- net QSPI-CLK: now also U4.6 (CLK), U5.52 (QSPI_SCLK)
- net SDIO_DAT1: now also J6.8 (DAT1), U5.14 (GPIO11)
- net SDIO_DAT2: now also J6.1 (DAT2), U5.13 (GPIO10)
- net SPI0_CIPO: now also J7.13, J9.5 (CIPO), U5.6 (GPIO4)
- net SPI0_COPI: now also J7.12, J9.6 (COPI), U5.5 (GPIO3)
- net SPI0_SCK: now also J7.11, J9.4 (SCK), U5.4 (GPIO2)
- net SPI_CIPO1/SDIO_DAT0: now also J6.7 (DAT0/SDO), U5.15 (GPIO12)
- net SPI_COPI1/SDIO_CMD: now also J6.3 (CMD/SDI), U5.18 (GPIO15)
- net SPI_SCK1/SDIO_CLK: now also J6.5 (CLK/SCK), U5.17 (GPIO14)
- net SPI_~{CS1}/SDIO_DAT3: now also J6.2 (DAT3/~{CS}), U5.12 (GPIO9)
- net SWDCK: now also J1.4 (SWDCLK), TP1.1, U5.24 (SWCLK)
- net SWDIO: now also J1.2 (SWDIO), TP2.1, U5.25 (SWDIO)
- net UART0_RX: now also J7.14, J9.14 (RX), U5.3 (GPIO1)
- net UART0_TX: now also J7.15, J9.13 (TX), U5.2 (GPIO0)
- net USB_N: now also J5.A7 (D-), J5.B7 (D-), R12.1
- net USB_P: now also J5.A6 (D+), J5.B6 (D+), R13.1
- net V_BATT: now also C1.1, C10.1, J4.2 (+), J8.1, Q1.3 (D), U2.2 (CELL), U2.3 (VDD), U3.3 (VBAT)
- net V_USB: now also C7.1, D2.A, J5.VBUS1 (VBUS), J5.VBUS2 (VBUS), J8.3, J9.10 (+5V), Q1.1 (G), R15.2, R2.2, U3.4 (VIN)
- net WS2812_DI: now also D5.DI, U5.11 (GPIO8)
- net WS2812_DO: now also D5.DO, J7.16
- net ~{BATT_ALERT}: now also U2.5 (~{ALRT}), U5.36 (GPIO24)
- net ~{BOOT}: now also R5.2, S1.3 (2)
- net ~{QSPI-CS}: now also R5.1, R9.1, U4.1 (~{CS}), U5.56 (QSPI_~{CS})
- net ~{RESET}: now also J1.10 (~{RESET}), J7.1, S2.3 (2), TP3.1, U5.26 (RUN)
- net ~{SPI0_CS}: now also J9.3 (CS), U5.7 (GPIO5)
- new net: I2C0.3, R10.2
- new net: I2C0.1, R17.2
- new net: D3.A, PWR0.1
- new net: D3.C, R8.2
- new net: R12.2, U5.46 (USB_D-)
- new net: R13.2, U5.47 (USB_D+)
- new net: C5.2, R11.1, Y2.P1 (1)
- new net: R6.2, U3.5 (PROG)
- new net: R11.2, U5.21 (XOUT)
- new net: C16.2, U5.20 (XIN), Y2.P3 (2)
- new net: J5.A5 (CC1), R1.1
- new net: J5.B5 (CC2), R4.1
- new net: J5.SHLD1 (SHLD), J5.SHLD2 (SHLD), J5.SHLD3 (SHLD), J5.SHLD4 (SHLD), J5.SHLD5 (SHLD), J5.SHLD6 (SHLD), J5.SHLD7 (SHLD), J5.SHLD8 (SHLD)
- new net: C8.1, D2.C, Q1.2 (S), R16.2, U7.1 (IN)
- new net: D4.C, R3.2
- new net: D1.A, R2.1
- new net: D1.C, U3.1 (STAT)
