File: PROJ/SPAR/19389/STAN/01/src/kicadBoard.kicad_sch (KiCad schematic)
At the start: 19 parts

Commit message: Quickly Adding Everything
Parts:
- removed C1: (no value), symbol eagleSchem-eagle-import:4.7UF-0603-6.3V-(10%)
- removed C2: (no value), symbol eagleSchem-eagle-import:1.0UF-0603-16V-10%
- removed C3: (no value), symbol eagleSchem-eagle-import:27PF-0603-50V-5%
- removed C4: (no value), symbol eagleSchem-eagle-import:0.1UF-0603-25V-(+80/-20%)
- removed FD1, FD2, FD3, FD4: (no value), symbol eagleSchem-eagle-import:FIDUCIALUFIDUCIAL
- removed FRAME2: (no value), symbol eagleSchem-eagle-import:FRAME-LETTER
- removed JP1: (no value), symbol eagleSchem-eagle-import:CONN_031X03_NO_SILK
- removed LOGO1: (no value), symbol eagleSchem-eagle-import:SFE_LOGO_FLAME.1_INCH
- removed LOGO2: (no value), symbol eagleSchem-eagle-import:OSHW-LOGOMINI
- removed OUT-0: (no value), symbol eagleSchem-eagle-import:TEST-POINTTP_15TH_THRU
- removed R1, R2: (no value), symbol eagleSchem-eagle-import:10KOHM-0603-1/10W-1%
- removed R3: (no value), symbol eagleSchem-eagle-import:4.7KOHM-0603-1/10W-1%
- removed R4: (no value), symbol eagleSchem-eagle-import:300KOHM-0603-1/10W-1%
- removed U1: (no value), symbol eagleSchem-eagle-import:OPA344
- removed U3: (no value), symbol eagleSchem-eagle-import:SPH8878LR5H-1
- added C1: (no value), symbol schematicEagle-eagle-import:4.7UF-0603-6.3V-(10%)
- added C2: (no value), symbol schematicEagle-eagle-import:1.0UF-0603-16V-10%
- added C3: (no value), symbol schematicEagle-eagle-import:27PF-0603-50V-5%
- added C4: (no value), symbol schematicEagle-eagle-import:0.1UF-0603-25V-(+80/-20%)
- added FD1, FD2, FD3, FD4: (no value), symbol schematicEagle-eagle-import:FIDUCIALUFIDUCIAL
- added FRAME2: (no value), symbol schematicEagle-eagle-import:FRAME-LETTER
- added JP1: (no value), symbol schematicEagle-eagle-import:CONN_031X03_NO_SILK
- added LOGO1: (no value), symbol schematicEagle-eagle-import:SFE_LOGO_FLAME.1_INCH
- added LOGO2: (no value), symbol schematicEagle-eagle-import:OSHW-LOGOMINI
- added OUT-0: (no value), symbol schematicEagle-eagle-import:TEST-POINTTP_15TH_THRU
- added R1, R2: (no value), symbol schematicEagle-eagle-import:10KOHM-0603-1/10W-1%
- added R3: (no value), symbol schematicEagle-eagle-import:4.7KOHM-0603-1/10W-1%
- added R4: (no value), symbol schematicEagle-eagle-import:300KOHM-0603-1/10W-1%
- added U1: (no value), symbol schematicEagle-eagle-import:OPA344
- added U3: (no value), symbol schematicEagle-eagle-import:SPH8878LR5H-1
Connections:
- net GND: now also C2.2, C4.1, JP1.2, R2.1, U1.2 (P$V-), U3.2 (GND), U3.3 (GND), U3.4 (GND)
- net VCC: now also C4.2, JP1.1, R1.2, U1.5 (P$V+), U3.5 (VDD)
- new net: C3.2, JP1.3, R4.1, U1.1 (OUT)
- new net: C2.1, R1.1, R2.2, U1.3 (+IN)
- new net: C3.1, R3.1, R4.2, U1.4 (-IN)
- new net: C1.1, U3.1 (OUT+)
- new net: C1.2, R3.2
- new net: OUT-0.1, U3.6 (OUT-)
