File: PROJ/SPAR/19921/STAN/01/src/kicadBoard.kicad_sch (KiCad schematic)
At the start: 26 parts

Commit message: Quickly Adding Everything
Parts:
- removed C2: (no value), symbol eagleSchem-eagle-import:1.0UF-0402T-16V-10%
- removed C5: (no value), symbol eagleSchem-eagle-import:10UF-0402T-6.3V-20%
- removed D1: (no value), symbol eagleSchem-eagle-import:LED-RED_0402
- removed FD1, FD2, FID1, FID2: (no value), symbol eagleSchem-eagle-import:FIDUCIALUFIDUCIAL
- removed FRAME1: (no value), symbol eagleSchem-eagle-import:FRAME-LETTER
- removed I2C_PU0: (no value), symbol eagleSchem-eagle-import:JUMPER-SMT_3_2-NC_TRACE_SILK
- removed J1: (no value), symbol eagleSchem-eagle-import:QWIIC_CONNECTORJS-1MM
- removed J2, J4: (no value), symbol eagleSchem-eagle-import:CONN_01_1MM
- removed LED0: (no value), symbol eagleSchem-eagle-import:JUMPER-SMT_2_NC_TRACE_SILK
- removed LOGO1: (no value), symbol eagleSchem-eagle-import:QWIIC_LOGO_4MM
- removed LOGO2: (no value), symbol eagleSchem-eagle-import:OSHW-LOGOMINI
- removed LOGO3: (no value), symbol eagleSchem-eagle-import:SFE_LOGO_NAMEBLANK
- removed R1, R2: (no value), symbol eagleSchem-eagle-import:2.2KOHM-0402T-1/16W-1%
- removed R4: (no value), symbol eagleSchem-eagle-import:1KOHM-0402T-1/16W-1%
- removed R7: (no value), symbol eagleSchem-eagle-import:100KOHM-0402T-1/16W-1%
- removed STANDOFF3: (no value), symbol eagleSchem-eagle-import:STAND-OFFTIGHT
- removed TP1, TP2, TP3, TP5: (no value), symbol eagleSchem-eagle-import:TEST-POINT3
- removed U2: (no value), symbol eagleSchem-eagle-import:MMC5983MA_QFN16
- added C2: (no value), symbol schematicEagle-eagle-import:1.0UF-0402T-16V-10%
- added C5: (no value), symbol schematicEagle-eagle-import:10UF-0402T-6.3V-20%
- added D1: (no value), symbol schematicEagle-eagle-import:LED-RED_0402
- added FD1, FD2, FID1, FID2: (no value), symbol schematicEagle-eagle-import:FIDUCIALUFIDUCIAL
- added FRAME1: (no value), symbol schematicEagle-eagle-import:FRAME-LETTER
- added I2C_PU0: (no value), symbol schematicEagle-eagle-import:JUMPER-SMT_3_2-NC_TRACE_SILK
- added J1: (no value), symbol schematicEagle-eagle-import:QWIIC_CONNECTORJS-1MM
- added J2, J4: (no value), symbol schematicEagle-eagle-import:CONN_01_1MM
- added LED0: (no value), symbol schematicEagle-eagle-import:JUMPER-SMT_2_NC_TRACE_SILK
- added LOGO1: (no value), symbol schematicEagle-eagle-import:QWIIC_LOGO_4MM
- added LOGO2: (no value), symbol schematicEagle-eagle-import:OSHW-LOGOMINI
- added LOGO3: (no value), symbol schematicEagle-eagle-import:SFE_LOGO_NAMEBLANK
- added R1, R2: (no value), symbol schematicEagle-eagle-import:2.2KOHM-0402T-1/16W-1%
- added R4: (no value), symbol schematicEagle-eagle-import:1KOHM-0402T-1/16W-1%
- added R7: (no value), symbol schematicEagle-eagle-import:100KOHM-0402T-1/16W-1%
- added STANDOFF3: (no value), symbol schematicEagle-eagle-import:STAND-OFFTIGHT
- added TP1, TP2, TP3, TP5: (no value), symbol schematicEagle-eagle-import:TEST-POINT3
- added U2: (no value), symbol schematicEagle-eagle-import:MMC5983MA_QFN16
Connections:
- net 3.3V: now also C2.1, I2C_PU0.2, J1.2, R4.2, R7.2, TP1.1, U2.13 (VDDIO), U2.2 (VDD)
- net GND: now also C2.2, C5.2, J1.1, J4.1, LED0.1, TP5.1, U2.11 (GND), U2.9 (GND)
- net INT: now also J2.1, U2.15 (INT)
- net SCL: now also J1.4, R1.1, TP3.1, U2.1 (SCL/SCK)
- net SDA: now also J1.3, R2.1, TP2.1, U2.16 (SDA/SDI)
- new net: I2C_PU0.1, R1.2
- new net: I2C_PU0.3, R2.2
- new net: D1.A, R4.1
- new net: D1.C, LED0.2
- new net: C5.1, U2.10 (CAP)
- new net: U2.12 (NC), U2.14 (NC), U2.3 (NC), U2.6 (NC), U2.7 (NC), U2.8 (NC)
- new net: R7.1, U2.4 (~{SPI_CS})
