File: PROJ/ADAF/1438/STAN/01/src/kicadBoard.kicad_sch (KiCad schematic)
At the start: 50 parts

Commit message: Quickly Adding Everything
Parts:
- removed A0, A1, A2, A3, A4: (no value), symbol eagleSchem-eagle-import:SOLDERJUMPERREFLOW_NOPASTE
- removed C1, C10, C2, C3, C6: (no value), symbol eagleSchem-eagle-import:CAP_CERAMIC0805-NOOUTLINE
- removed C4, C5: (no value), symbol eagleSchem-eagle-import:CAP_ELECTROLYTICPANASONIC_C
- removed C9: (no value), symbol eagleSchem-eagle-import:CPOL-USC
- removed CN1: (no value), symbol eagleSchem-eagle-import:1X4-CLEANBIG
- removed D0-7, JP2: (no value), symbol eagleSchem-eagle-import:PINHD-1X8CLEANBIG
- removed IC1, IC3: (no value), symbol eagleSchem-eagle-import:TB6612FNG
- removed J1, J2: (no value), symbol eagleSchem-eagle-import:1X5
- removed JP1: (no value), symbol eagleSchem-eagle-import:HEADER-1X476MIL
- removed JP3: (no value), symbol eagleSchem-eagle-import:HEADER-1X1070MIL
- removed JP4: (no value), symbol eagleSchem-eagle-import:HEADER-1X2ROUND
- removed LED1: (no value), symbol eagleSchem-eagle-import:LED0805_NOOUTLINE
- removed MPOWER0, SERPWR0: (no value), symbol eagleSchem-eagle-import:1X2-3.5MM
- removed PWR0: (no value), symbol eagleSchem-eagle-import:JP1E
- removed Q1: (no value), symbol eagleSchem-eagle-import:IRF?5305R
- removed R1, R2, R3, R4, R5, R6, R7, R8: (no value), symbol eagleSchem-eagle-import:RESISTOR0805_NOOUTLINE
- removed SERVO1, SERVO2: (no value), symbol eagleSchem-eagle-import:PINHD-1X3
- removed SJ1: (no value), symbol eagleSchem-eagle-import:SOLDERJUMPER_2WAY
- removed SW1: (no value), symbol eagleSchem-eagle-import:SPST_TACT-EVQQ2
- removed TP1, TP2, TP3, TP4, TP5: (no value), symbol eagleSchem-eagle-import:TESTPOINTROUND2MM
- removed U$1: (no value), symbol eagleSchem-eagle-import:ARDUINO_R3_ICSP
- removed U$2, U$3, U$4: (no value), symbol eagleSchem-eagle-import:FIDUCIAL
- removed U2: (no value), symbol eagleSchem-eagle-import:PCA9685
- added A0, A1, A2, A3, A4: (no value), symbol schematicEagle-eagle-import:SJ
- added C1, C10, C2, C3, C6: (no value), symbol schematicEagle-eagle-import:C-USC0805K
- added C4, C5: (no value), symbol schematicEagle-eagle-import:CAP_ELECTROLYTICPANASONIC_C
- added C9: (no value), symbol schematicEagle-eagle-import:CPOL-USC
- added CN1: (no value), symbol schematicEagle-eagle-import:1X4-CLEANBIG
- added D0-7, JP2: (no value), symbol schematicEagle-eagle-import:PINHD-1X8CLEANBIG
- added IC1, IC3: (no value), symbol schematicEagle-eagle-import:TB6612FNG
- added J1, J2: (no value), symbol schematicEagle-eagle-import:1X5
- added JP1: (no value), symbol schematicEagle-eagle-import:HEADER-1X476MIL
- added JP3: (no value), symbol schematicEagle-eagle-import:HEADER-1X1070MIL
- added LED1: (no value), symbol schematicEagle-eagle-import:LEDCHIP-LED0805
- added MPOWER0, SERPWR0: (no value), symbol schematicEagle-eagle-import:1X2-3.5MM
- added PWR0: (no value), symbol schematicEagle-eagle-import:JP1E
- added Q1: (no value), symbol schematicEagle-eagle-import:IRF?5305R
- added R1, R2, R3, R4, R5, R6, R7, R8: (no value), symbol schematicEagle-eagle-import:R-US_R0805
- added SERVO1, SERVO2: (no value), symbol schematicEagle-eagle-import:PINHD-1X3
- added SJ1: (no value), symbol schematicEagle-eagle-import:SOLDERJUMPER_2WAY
- added TP1, TP2, TP3, TP4, TP5: (no value), symbol schematicEagle-eagle-import:TESTPOINTROUND2MM
- added U$1, U$5: (no value), symbol schematicEagle-eagle-import:ARDUINO_R3_ICSP
- added U$2, U$3, U$4: (no value), symbol schematicEagle-eagle-import:FIDUCIAL
- added U2: (no value), symbol schematicEagle-eagle-import:PCA9685
Connections:
- net +12V: now also C4.+, C5.+, IC1.13 (VM2), IC1.14 (VM3), IC1.24 (VM1), IC3.13 (VM2), IC3.14 (VM3), IC3.24 (VM1), LED1.A, PWR0.1, Q1.4 (D)
- net +3V3: now also JP2.5, SJ1.3, U$1.3V, U$5.3V
- net +5V: now also C9.+, JP2.4, SERPWR0.1, SERVO1.2, SERVO2.2, SJ1.1, U$1.5V_ICSP (5V), U$5.5V_ICSP (5V)
- net /RST: now also JP2.6, U$1.RESET (/RESET), U$5.RESET (/RESET)
- net A0: now also A0.2, R1.2, TP5.P$1, U2.1 (A0)
- net A1: now also A1.2, R2.2, TP4.P$1, U2.2 (A1)
- net A2: now also A2.2, R3.2, TP3.P$1, U2.3 (A2)
- net A3: now also A3.1, R5.2, TP2.P$1, U2.4 (A3)
- net A4: now also A4.1, R6.2, TP1.P$1, U2.5 (A4)
- net GND: now also C1.2, C10.2, C2.2, C3.2, C4.-, C5.-, C6.2, C9.-, IC1.10 (PGND2'), IC1.18 (GND), IC1.3 (PGND1), IC1.4 (PGND1'), IC1.9 (PGND2), IC3.10 (PGND2'), IC3.18 (GND), IC3.3 (PGND1), IC3.4 (PGND1'), IC3.9 (PGND2), J1.3, J2.3, JP2.2, JP2.3, JP3.4, MPOWER0.1, Q1.1 (G), R1.1, R2.1, R3.1, R4.1, R5.1, R6.1, SERPWR0.2, SERVO1.1, SERVO2.1, U$1.GND, U$1.GND@1, U$1.GND@2, U$5.GND, U$5.GND@1, U$5.GND@2, U2.14 (GND), U2.23 (#OE), U2.25 (EXTCLK)
- net PWM0: now also JP1.1, U2.6 (PWM0)
- net PWM1: now also JP1.2, U2.7 (PWM1)
- net PWM10: now also IC1.21 (AIN1), U2.17 (PWM10)
- net PWM11: now also IC1.17 (BIN1), U2.18 (PWM11)
- net PWM12: now also IC1.16 (BIN2), U2.19 (PWM12)
- net PWM13: now also IC1.15 (PWMB), U2.20 (PWM13)
- net PWM14: now also JP1.3, U2.21 (PWM14)
- net PWM15: now also JP1.4, U2.22 (PWM15)
- net PWM2: now also IC3.23 (PWMA), U2.8 (PWM2)
- net PWM3: now also IC3.22 (AIN2), U2.9 (PWM3)
- net PWM4: now also IC3.21 (AIN1), U2.10 (PWM4)
- net PWM5: now also IC3.17 (BIN1), U2.11 (PWM5)
- net PWM6: now also IC3.16 (BIN2), U2.12 (PWM6)
- net PWM7: now also IC3.15 (PWMB), U2.13 (PWM7)
- net PWM8: now also IC1.23 (PWMA), U2.15 (PWM8)
- net PWM9: now also IC1.22 (AIN2), U2.16 (PWM9)
- net VCC: now also A0.1, A1.1, A2.1, A3.2, A4.2, C1.1, C10.1, C2.1, C3.1, C6.1, IC1.19 (STBY), IC1.20 (VCC), IC3.19 (STBY), IC3.20 (VCC), R7.2, R8.2, SJ1.2, U2.24 (A5), U2.28 (VDD)
- net VIN: now also JP2.1, PWR0.2, U$1.VIN, U$5.VIN
- new net: D0-7.1, U$1.D0, U$5.D0
- new net: D0-7.2, U$1.D1, U$5.D1
- new net: D0-7.3, U$1.D2, U$5.D2
- new net: D0-7.4, U$1.D3, U$5.D3
- new net: D0-7.5, U$1.D4, U$5.D4
- new net: D0-7.6, U$1.D5, U$5.D5
- new net: D0-7.7, U$1.D6, U$5.D6
- new net: D0-7.8, U$1.D7, U$5.D7
- new net: MPOWER0.2, Q1.3 (S)
- new net: IC1.1 (AO1), IC1.2 (AO1'), J1.5
- new net: IC1.11 (BO1), IC1.12 (BO1'), J1.1
- new net: IC1.5 (AO2), IC1.6 (AO2'), J1.4
- new net: IC1.7 (BO2), IC1.8 (BO2'), J1.2
- new net: LED1.C, R4.2
- new net: IC3.1 (AO1), IC3.2 (AO1'), J2.1
- new net: IC3.5 (AO2), IC3.6 (AO2'), J2.2
- new net: IC3.7 (BO2), IC3.8 (BO2'), J2.4
- new net: IC3.11 (BO1), IC3.12 (BO1'), J2.5
- new net: U$1.5V (5V@1), U$5.5V (5V@1)
- new net: CN1.4, U$1.A0, U$5.A0
- new net: CN1.3, U$1.A1, U$5.A1
- new net: CN1.2, U$1.A2, U$5.A2
- new net: CN1.1, U$1.A3, U$5.A3
- new net: JP3.3, U$1.AREF, U$5.AREF
- new net: JP3.7, U$1.D11, U$5.D11
- new net: JP3.6, U$1.D12, U$5.D12
- new net: JP3.5, U$1.D13, U$5.D13
- new net: JP3.10, U$1.D8, U$5.D8
- new net: U$1.GND@3, U$5.GND@3
- new net: JP2.7, U$1.IOREF, U$5.IOREF
- new net: U$1.MISO, U$5.MISO
- new net: U$1.MOSI, U$5.MOSI
- new net: JP2.8, U$1.RESERVED, U$5.RESERVED
- new net: U$1.RESET_ICSP (RST), U$5.RESET_ICSP (RST)
- new net: U$1.SCK, U$5.SCK
- new net PWM1A: JP3.9, SERVO2.3, U$1.D9, U$5.D9
- new net PWM1B: JP3.8, SERVO1.3, U$1.D10, U$5.D10
- new net SCL: JP3.1, R8.1, U$1.A5 (A5/SCL), U$1.SCL, U$5.A5 (A5/SCL), U$5.SCL, U2.26 (SCL)
- new net SDA: JP3.2, R7.1, U$1.A4 (A4/SDA), U$1.SDA, U$5.A4 (A4/SDA), U$5.SDA, U2.27 (SDA)

Commit message: Quickly Adding Everything
Parts:
- removed A0, A1, A2, A3, A4: (no value), symbol schematicEagle-eagle-import:SJ
- removed C1, C10, C2, C3, C6: (no value), symbol schematicEagle-eagle-import:C-USC0805K
- removed C4, C5: (no value), symbol schematicEagle-eagle-import:CAP_ELECTROLYTICPANASONIC_C
- removed C9: (no value), symbol schematicEagle-eagle-import:CPOL-USC
- removed CN1: (no value), symbol schematicEagle-eagle-import:1X4-CLEANBIG
- removed D0-7, JP2: (no value), symbol schematicEagle-eagle-import:PINHD-1X8CLEANBIG
- removed IC1, IC3: (no value), symbol schematicEagle-eagle-import:TB6612FNG
- removed J1, J2: (no value), symbol schematicEagle-eagle-import:1X5
- removed JP1: (no value), symbol schematicEagle-eagle-import:HEADER-1X476MIL
- removed JP3: (no value), symbol schematicEagle-eagle-import:HEADER-1X1070MIL
- removed LED1: (no value), symbol schematicEagle-eagle-import:LEDCHIP-LED0805
- removed MPOWER0, SERPWR0: (no value), symbol schematicEagle-eagle-import:1X2-3.5MM
- removed PWR0: (no value), symbol schematicEagle-eagle-import:JP1E
- removed Q1: (no value), symbol schematicEagle-eagle-import:IRF?5305R
- removed R1, R2, R3, R4, R5, R6, R7, R8: (no value), symbol schematicEagle-eagle-import:R-US_R0805
- removed SERVO1, SERVO2: (no value), symbol schematicEagle-eagle-import:PINHD-1X3
- removed SJ1: (no value), symbol schematicEagle-eagle-import:SOLDERJUMPER_2WAY
- removed TP1, TP2, TP3, TP4, TP5: (no value), symbol schematicEagle-eagle-import:TESTPOINTROUND2MM
- removed U$1, U$5: (no value), symbol schematicEagle-eagle-import:ARDUINO_R3_ICSP
- removed U$2, U$3, U$4: (no value), symbol schematicEagle-eagle-import:FIDUCIAL
- removed U2: (no value), symbol schematicEagle-eagle-import:PCA9685
- added A0, A1, A2, A3, A4: (no value), symbol eagleSchem-eagle-import:SOLDERJUMPERREFLOW_NOPASTE
- added C1, C10, C2, C3, C6: (no value), symbol eagleSchem-eagle-import:CAP_CERAMIC0805-NOOUTLINE
- added C4, C5: (no value), symbol eagleSchem-eagle-import:CAP_ELECTROLYTICPANASONIC_C
- added C9: (no value), symbol eagleSchem-eagle-import:CPOL-USC
- added CN1: (no value), symbol eagleSchem-eagle-import:1X4-CLEANBIG
- added D0-7, JP2: (no value), symbol eagleSchem-eagle-import:PINHD-1X8CLEANBIG
- added IC1, IC3: (no value), symbol eagleSchem-eagle-import:TB6612FNG
- added J1, J2: (no value), symbol eagleSchem-eagle-import:1X5
- added JP1: (no value), symbol eagleSchem-eagle-import:HEADER-1X476MIL
- added JP3: (no value), symbol eagleSchem-eagle-import:HEADER-1X1070MIL
- added JP4: (no value), symbol eagleSchem-eagle-import:HEADER-1X2ROUND
- added LED1: (no value), symbol eagleSchem-eagle-import:LED0805_NOOUTLINE
- added MPOWER0, SERPWR0: (no value), symbol eagleSchem-eagle-import:1X2-3.5MM
- added PWR0: (no value), symbol eagleSchem-eagle-import:JP1E
- added Q1: (no value), symbol eagleSchem-eagle-import:IRF?5305R
- added R1, R2, R3, R4, R5, R6, R7, R8: (no value), symbol eagleSchem-eagle-import:RESISTOR0805_NOOUTLINE
- added SERVO1, SERVO2: (no value), symbol eagleSchem-eagle-import:PINHD-1X3
- added SJ1: (no value), symbol eagleSchem-eagle-import:SOLDERJUMPER_2WAY
- added SW1: (no value), symbol eagleSchem-eagle-import:SPST_TACT-EVQQ2
- added TP1, TP2, TP3, TP4, TP5: (no value), symbol eagleSchem-eagle-import:TESTPOINTROUND2MM
- added U$1: (no value), symbol eagleSchem-eagle-import:ARDUINO_R3_ICSP
- added U$2, U$3, U$4: (no value), symbol eagleSchem-eagle-import:FIDUCIAL
- added U2: (no value), symbol eagleSchem-eagle-import:PCA9685
Connections:
- net +12V: now also C4.+, C5.+, IC1.13 (VM2), IC1.14 (VM3), IC1.24 (VM1), IC3.13 (VM2), IC3.14 (VM3), IC3.24 (VM1), LED1.A, PWR0.1, Q1.3 (S)
- net +3V3: now also JP2.5, SJ1.3, U$1.3V
- net +5V: now also C9.+, JP2.4, SERPWR0.1, SERVO1.2, SERVO2.2, SJ1.1, U$1.5V, U$1.5V_ICSP (5V@1)
- net /RST: now also JP2.6, SW1.B (S), SW1.B' (S1), U$1.RESET (/RESET), U$1.RESET_ICSP (RST)
- net A0: now also A0.2, R1.2, TP5.P$1, U2.1 (A0)
- net A1: now also A1.2, R2.2, TP4.P$1, U2.2 (A1)
- net A2: now also A2.2, R3.2, TP3.P$1, U2.3 (A2)
- net A3: now also A3.1, R5.2, TP2.P$1, U2.4 (A3)
- net A4: now also A4.1, R6.2, TP1.P$1, U2.5 (A4)
- net GND: now also C1.2, C10.2, C2.2, C3.2, C4.-, C5.-, C6.2, C9.-, IC1.10 (PGND2'), IC1.18 (GND), IC1.3 (PGND1), IC1.4 (PGND1'), IC1.9 (PGND2), IC3.10 (PGND2'), IC3.18 (GND), IC3.3 (PGND1), IC3.4 (PGND1'), IC3.9 (PGND2), J1.3, J2.3, JP2.2, JP2.3, JP3.4, MPOWER0.1, Q1.1 (G), R1.1, R2.1, R3.1, R4.1, R5.1, R6.1, SERPWR0.2, SERVO1.1, SERVO2.1, SW1.A (P), SW1.A' (P1), U$1.GND, U$1.GND@1 (GND@2), U$1.GND@2 (GND@3), U$1.GND@3 (GND@1), U2.14 (GND), U2.23 (#OE), U2.25 (EXTCLK)
- net PWM0: now also JP1.1, U2.6 (PWM0)
- net PWM1: now also JP1.2, U2.7 (PWM1)
- net PWM10: now also IC1.21 (AIN1), U2.17 (PWM10)
- net PWM11: now also IC1.17 (BIN1), U2.18 (PWM11)
- net PWM12: now also IC1.16 (BIN2), U2.19 (PWM12)
- net PWM13: now also IC1.15 (PWMB), U2.20 (PWM13)
- net PWM14: now also JP1.3, U2.21 (PWM14)
- net PWM15: now also JP1.4, U2.22 (PWM15)
- net PWM2: now also IC3.23 (PWMA), U2.8 (PWM2)
- net PWM3: now also IC3.22 (AIN2), U2.9 (PWM3)
- net PWM4: now also IC3.21 (AIN1), U2.10 (PWM4)
- net PWM5: now also IC3.17 (BIN1), U2.11 (PWM5)
- net PWM6: now also IC3.16 (BIN2), U2.12 (PWM6)
- net PWM7: now also IC3.15 (PWMB), U2.13 (PWM7)
- net PWM8: now also IC1.23 (PWMA), U2.15 (PWM8)
- net PWM9: now also IC1.22 (AIN2), U2.16 (PWM9)
- net VCC: now also A0.1, A1.1, A2.1, A3.2, A4.2, C1.1, C10.1, C2.1, C3.1, C6.1, IC1.19 (STBY), IC1.20 (VCC), IC3.19 (STBY), IC3.20 (VCC), R7.2, R8.2, SJ1.2, U2.24 (A5), U2.28 (VDD)
- net VIN: now also JP2.1, PWR0.2, U$1.VIN
- new net: IC1.1 (AO1), IC1.2 (AO1'), J1.5
- new net: IC1.11 (BO1), IC1.12 (BO1'), J1.1
- new net: IC1.5 (AO2), IC1.6 (AO2'), J1.4
- new net: IC1.7 (BO2), IC1.8 (BO2'), J1.2
- new net: CN1.1, U$1.A3
- new net: CN1.2, U$1.A2
- new net: CN1.3, U$1.A1
- new net: CN1.4, U$1.A0
- new net: IC3.1 (AO1), IC3.2 (AO1'), J2.1
- new net: IC3.11 (BO1), IC3.12 (BO1'), J2.5
- new net: IC3.5 (AO2), IC3.6 (AO2'), J2.2
- new net: IC3.7 (BO2), IC3.8 (BO2'), J2.4
- new net: MPOWER0.2, Q1.4 (D)
- new net: D0-7.1, U$1.D0
- new net: D0-7.2, U$1.D1
- new net: D0-7.3, U$1.D2
- new net: D0-7.4, U$1.D3
- new net: D0-7.5, U$1.D4
- new net: D0-7.6, U$1.D5
- new net: D0-7.7, U$1.D6
- new net: D0-7.8, U$1.D7
- new net: LED1.C, R4.2
- new net: JP3.10, U$1.D8
- new net: JP3.3, U$1.AREF
- new net: JP3.5, U$1.D13
- new net: JP3.6, U$1.D12
- new net: JP3.7, U$1.D11
- new net: JP2.7, U$1.IOREF
- new net: JP2.8, U$1.RESERVED
- new net AD4/SDA: JP3.2, JP4.2, R7.1, U$1.A4 (A4/SDA), U$1.SDA, U2.27 (SDA)
- new net AD5/SCL: JP3.1, JP4.1, R8.1, U$1.A5 (A5/SCL), U$1.SCL, U2.26 (SCL)
- new net D10: JP3.8, SERVO1.3, U$1.D10
- new net D9: JP3.9, SERVO2.3, U$1.D9
