File: PROJ/ADAF/1601/STAN/01/src/kicadBoard.kicad_sch (KiCad schematic)
At the start: 33 parts

Commit message: Quickly Adding Everything
Parts:
- removed C1, C2, C3, C4, C5: (no value), symbol eagleSchem-eagle-import:C-USC0805K
- removed IC4: (no value), symbol eagleSchem-eagle-import:LP298XS
- removed IC5: (no value), symbol eagleSchem-eagle-import:AXP083-SAG
- removed JP1: (no value), symbol eagleSchem-eagle-import:HEADER-2X13
- removed Q1: (no value), symbol eagleSchem-eagle-import:-NPN-SOT23-BEC
- removed R1, R10, R11, R2, R3, R4, R5, R6, R7, R8, R9: (no value), symbol eagleSchem-eagle-import:R-US_R0805
- removed SW1, SW2, SW3, SW4: (no value), symbol eagleSchem-eagle-import:SWITCH_PUSHBUTTONEVQ-PE
- removed U$10, U$11, U$18: (no value), symbol eagleSchem-eagle-import:FIDUCIAL
- removed U$15, U$16, U$17: (no value), symbol eagleSchem-eagle-import:MOUNTINGHOLE2.5_THICK
- removed U$2: (no value), symbol eagleSchem-eagle-import:DISP_LCD_1.28IN_240X320_50PIN
- removed U$3: (no value), symbol eagleSchem-eagle-import:RASPBERRYPI_B_MODELB_V2
- removed U2: (no value), symbol eagleSchem-eagle-import:STMPE610
- added C1, C2, C3, C4, C5: (no value), symbol schematicEagle-eagle-import:C-USC0805K
- added IC4: (no value), symbol schematicEagle-eagle-import:LP298XS
- added IC5: (no value), symbol schematicEagle-eagle-import:AXP083-SAG
- added JP1: (no value), symbol schematicEagle-eagle-import:HEADER-2X13
- added Q1: (no value), symbol schematicEagle-eagle-import:-NPN-SOT23-BEC
- added R1, R10, R11, R2, R3, R4, R5, R6, R7, R8, R9: (no value), symbol schematicEagle-eagle-import:R-US_R0805
- added SW1, SW2, SW3, SW4: (no value), symbol schematicEagle-eagle-import:SWITCH_PUSHBUTTONEVQ-PE
- added U$10, U$11, U$18: (no value), symbol schematicEagle-eagle-import:FIDUCIAL
- added U$15, U$16, U$17: (no value), symbol schematicEagle-eagle-import:MOUNTINGHOLE2.5_THICK
- added U$2: (no value), symbol schematicEagle-eagle-import:DISP_LCD_1.28IN_240X320_50PIN
- added U$3: (no value), symbol schematicEagle-eagle-import:RASPBERRYPI_B_MODELB_V2
- added U2: (no value), symbol schematicEagle-eagle-import:STMPE610
Connections:
- net +5V: now also C5.1, IC4.1 (VIN), IC4.3 (EN), JP1.2, JP1.4, R1.1, R2.1, R3.1, R4.1, U$3.2 (5.0V), U$3.4 (5.0V@1)
- net GND: now also C1.2, C2.2, C3.2, C4.2, C5.2, IC4.2 (GND), IC5.1 (GND), JP1.14, JP1.20, JP1.25, JP1.9, Q1.E, SW1.P$2, SW2.P$2, SW3.P$2, SW4.P$2, U$2.43 (GND@1), U$2.48 (GND@2), U$2.49 (GND@3), U$2.50 (GND@4), U$2.6 (IM0), U$3.14 (GND@1), U$3.20 (GND@2), U$3.25 (GND@3), U$3.6 (GND), U$3.9 (GND@4), U2.P$10 (GND)
- net GPIO18: now also JP1.12, SW4.P$1, U$3.12 (GPIO18)
- net GPIO21: now also JP1.13, SW3.P$1, U$3.13 (GPIO21)
- net GPIO22: now also JP1.15, SW2.P$1, U$3.15 (GPIO22_27)
- net GPIO23: now also JP1.16, SW1.P$1, U$3.16 (GPIO23)
- net MISO: now also JP1.21, U$2.33 (SDO), U$3.21 (SPI_MISO), U2.P$3 (A0/MISO)
- net MOSI: now also R11.2, U$2.34 (SDI), U2.P$7 (MOSI)
- net MOSI_3V: now also JP1.19, R11.1, U$3.19 (SPI_MOSI)
- net RT_CS_3V: now also JP1.26, R7.1, U$3.26 (#SPI_CE1), U2.P$5 (SDA/CS)
- net RT_INT: now also JP1.18, R8.2, U$3.18 (GPIO24), U2.P$2 (INT)
- net SCLK: now also R10.2, U$2.37 (RS), U2.P$4 (SCLK)
- net SCLK_3V: now also JP1.23, R10.1, U$3.23 (SPI_SCLK)
- net TFT_CS_3V: now also JP1.24, U$2.38 (#CS), U$3.24 (#SPI_CE0)
- net TFT_DC_3V: now also JP1.22, U$2.36 (#WR), U$3.22 (GPIO25)
- net TFT_RST: now also IC5.2 (/RESET), R6.1, U$2.10 (RESET)
- net VCC: now also C1.1, C2.1, C3.1, C4.1, IC4.5 (VOUT), IC5.3 (VCC), R6.2, R7.2, R8.1, R9.2, U$2.40 (IOVCC@1), U$2.41 (IOVCC@2), U$2.42 (VCI), U$2.7 (IM1), U$2.8 (IM2), U$2.9 (IM3), U2.P$14 (VIO), U2.P$6 (VCC), U2.P$9 (MODE)
- net XL: now also U$2.46 (XL), U2.P$16 (X-)
- net XR: now also U$2.44 (XR), U2.P$13 (X+)
- net YD: now also U$2.45 (YD), U2.P$15 (Y+)
- net YU: now also U$2.47 (YU), U2.P$1 (Y-)
- new net: R1.2, U$2.2 (LEDA@1)
- new net: Q1.C, U$2.1 (LEDK)
- new net: U$2.15 (DB17), U$2.16 (DB16), U$2.17 (DB15), U$2.18 (DB14), U$2.19 (DB13), U$2.20 (DB12), U$2.21 (DB11), U$2.22 (DB10), U$2.23 (DB9), U$2.24 (DB8), U$2.25 (DB7), U$2.26 (DB6), U$2.27 (DB5), U$2.28 (DB4), U$2.29 (DB3), U$2.30 (DB2), U$2.31 (DB1), U$2.32 (DB0)
- new net: R2.2, U$2.3 (LEDA@2)
- new net: R3.2, U$2.4 (LEDA@3)
- new net: R4.2, U$2.5 (LEDA@4)
- new net: R5.1, R9.1, U2.P$11 (IN2/GPIO2)
- new net: Q1.B, R5.2
- new net: JP1.1, U$3.1 (3.3V)
- new net: JP1.10, U$3.10 (RXD)
- new net: JP1.11, U$3.11 (GPIO17)
- new net: JP1.17, U$3.17 (3.3V@1)
- new net: JP1.3, U$3.3 (SDA)
- new net: JP1.5, U$3.5 (SCL)
- new net: JP1.7, U$3.7 (GPIO4)
- new net: JP1.8, U$3.8 (TXD)

Commit message: Quickly Adding Everything
Parts:
- removed C1, C2, C3, C4, C5: (no value), symbol schematicEagle-eagle-import:C-USC0805K
- removed IC4: (no value), symbol schematicEagle-eagle-import:LP298XS
- removed IC5: (no value), symbol schematicEagle-eagle-import:AXP083-SAG
- removed JP1: (no value), symbol schematicEagle-eagle-import:HEADER-2X13
- removed Q1: (no value), symbol schematicEagle-eagle-import:-NPN-SOT23-BEC
- removed R1, R10, R11, R2, R3, R4, R5, R6, R7, R8, R9: (no value), symbol schematicEagle-eagle-import:R-US_R0805
- removed SW1, SW2, SW3, SW4: (no value), symbol schematicEagle-eagle-import:SWITCH_PUSHBUTTONEVQ-PE
- removed U$10, U$11, U$18: (no value), symbol schematicEagle-eagle-import:FIDUCIAL
- removed U$15, U$16, U$17: (no value), symbol schematicEagle-eagle-import:MOUNTINGHOLE2.5_THICK
- removed U$2: (no value), symbol schematicEagle-eagle-import:DISP_LCD_1.28IN_240X320_50PIN
- removed U$3: (no value), symbol schematicEagle-eagle-import:RASPBERRYPI_B_MODELB_V2
- removed U2: (no value), symbol schematicEagle-eagle-import:STMPE610
- added C1, C2, C3, C4, C5: (no value), symbol eagleSchem-eagle-import:C-USC0805K
- added IC4: (no value), symbol eagleSchem-eagle-import:LP298XS
- added IC5: (no value), symbol eagleSchem-eagle-import:AXP083-SAG
- added JP1: (no value), symbol eagleSchem-eagle-import:HEADER-2X13
- added Q1: (no value), symbol eagleSchem-eagle-import:-NPN-SOT23-BEC
- added R1, R10, R11, R2, R3, R4, R5, R6, R7, R8, R9: (no value), symbol eagleSchem-eagle-import:R-US_R0805
- added SW1, SW2, SW3, SW4: (no value), symbol eagleSchem-eagle-import:SWITCH_PUSHBUTTONEVQ-PE
- added U$10, U$11, U$18: (no value), symbol eagleSchem-eagle-import:FIDUCIAL
- added U$15, U$16, U$17: (no value), symbol eagleSchem-eagle-import:MOUNTINGHOLE2.5_THICK
- added U$2: (no value), symbol eagleSchem-eagle-import:DISP_LCD_1.28IN_240X320_50PIN
- added U$3: (no value), symbol eagleSchem-eagle-import:RASPBERRYPI_B_MODELB_V2
- added U2: (no value), symbol eagleSchem-eagle-import:STMPE610
Connections:
- net +5V: now also C5.1, IC4.1 (VIN), IC4.3 (EN), JP1.2, JP1.4, R1.1, R2.1, R3.1, R4.1, U$3.2 (5.0V), U$3.4 (5.0V@1)
- net GND: now also C1.2, C2.2, C3.2, C4.2, C5.2, IC4.2 (GND), IC5.1 (GND), JP1.14, JP1.20, JP1.25, JP1.9, Q1.E, SW1.P$2, SW2.P$2, SW3.P$2, SW4.P$2, U$2.43 (GND@1), U$2.48 (GND@2), U$2.49 (GND@3), U$2.50 (GND@4), U$2.6 (IM0), U$3.14 (GND@1), U$3.20 (GND@2), U$3.25 (GND@3), U$3.6 (GND), U$3.9 (GND@4), U2.P$10 (GND)
- net GPIO18: now also JP1.12, SW4.P$1, U$3.12 (GPIO18)
- net GPIO21: now also JP1.13, SW3.P$1, U$3.13 (GPIO21)
- net GPIO22: now also JP1.15, SW2.P$1, U$3.15 (GPIO22_27)
- net GPIO23: now also JP1.16, SW1.P$1, U$3.16 (GPIO23)
- net MISO: now also JP1.21, U$2.33 (SDO), U$3.21 (SPI_MISO), U2.P$3 (A0/MISO)
- net MOSI: now also R11.2, U$2.34 (SDI), U2.P$7 (MOSI)
- net MOSI_3V: now also JP1.19, R11.1, U$3.19 (SPI_MOSI)
- net RT_CS_3V: now also JP1.26, R7.1, U$3.26 (#SPI_CE1), U2.P$5 (SDA/CS)
- net RT_INT: now also JP1.18, R8.2, U$3.18 (GPIO24), U2.P$2 (INT)
- net SCLK: now also R10.2, U$2.37 (RS), U2.P$4 (SCLK)
- net SCLK_3V: now also JP1.23, R10.1, U$3.23 (SPI_SCLK)
- net TFT_CS_3V: now also JP1.24, U$2.38 (#CS), U$3.24 (#SPI_CE0)
- net TFT_DC_3V: now also JP1.22, U$2.36 (#WR), U$3.22 (GPIO25)
- net TFT_RST: now also IC5.2 (/RESET), R6.1, U$2.10 (RESET)
- net VCC: now also C1.1, C2.1, C3.1, C4.1, IC4.5 (VOUT), IC5.3 (VCC), R6.2, R7.2, R8.1, R9.2, U$2.40 (IOVCC@1), U$2.41 (IOVCC@2), U$2.42 (VCI), U$2.7 (IM1), U$2.8 (IM2), U$2.9 (IM3), U2.P$14 (VIO), U2.P$6 (VCC), U2.P$9 (MODE)
- net XL: now also U$2.46 (XL), U2.P$16 (X-)
- net XR: now also U$2.44 (XR), U2.P$13 (X+)
- net YD: now also U$2.45 (YD), U2.P$15 (Y+)
- net YU: now also U$2.47 (YU), U2.P$1 (Y-)
- new net: JP1.1, U$3.1 (3.3V)
- new net: JP1.10, U$3.10 (RXD)
- new net: JP1.11, U$3.11 (GPIO17)
- new net: JP1.17, U$3.17 (3.3V@1)
- new net: JP1.3, U$3.3 (SDA)
- new net: JP1.5, U$3.5 (SCL)
- new net: JP1.7, U$3.7 (GPIO4)
- new net: JP1.8, U$3.8 (TXD)
- new net: R2.2, U$2.3 (LEDA@2)
- new net: R4.2, U$2.5 (LEDA@4)
- new net: Q1.B, R5.2
- new net: Q1.C, U$2.1 (LEDK)
- new net: R3.2, U$2.4 (LEDA@3)
- new net: R5.1, R9.1, U2.P$11 (IN2/GPIO2)
- new net: U$2.15 (DB17), U$2.16 (DB16), U$2.17 (DB15), U$2.18 (DB14), U$2.19 (DB13), U$2.20 (DB12), U$2.21 (DB11), U$2.22 (DB10), U$2.23 (DB9), U$2.24 (DB8), U$2.25 (DB7), U$2.26 (DB6), U$2.27 (DB5), U$2.28 (DB4), U$2.29 (DB3), U$2.30 (DB2), U$2.31 (DB1), U$2.32 (DB0)
- new net: R1.2, U$2.2 (LEDA@1)
