File: PROJ/ADAF/1743/STAN/01/src/kicadBoard.kicad_sch (KiCad schematic)
At the start: 39 parts

Commit message: Quickly Adding Everything
Parts:
- removed C1, C2, C3, C4, C5: (no value), symbol eagleSchem-eagle-import:CAP_CERAMIC0805-NOOUTLINE
- removed IC1: (no value), symbol eagleSchem-eagle-import:LP298XS
- removed IC2, IC3: (no value), symbol eagleSchem-eagle-import:74245DW
- removed IC4: (no value), symbol eagleSchem-eagle-import:AXP083-SAG
- removed JP1, JP2: (no value), symbol eagleSchem-eagle-import:HEADER-1X20ROUND
- removed Q1: (no value), symbol eagleSchem-eagle-import:-NPN-SOT23-BEC
- removed R1, R10, R11, R12, R13, R14, R2, R3, R4, R5, R7, R8, R9: (no value), symbol eagleSchem-eagle-import:RESISTOR0805_NOOUTLINE
- removed R6: (no value), symbol eagleSchem-eagle-import:R-US_R0805
- removed SJ1, SJ2, SJ3, SJ4: (no value), symbol eagleSchem-eagle-import:SOLDERJUMPER
- removed U$11, U$23, U$9: (no value), symbol eagleSchem-eagle-import:FIDUCIAL{dblquote}{dblquote}
- removed U$15, U$16, U$17, U$7: (no value), symbol eagleSchem-eagle-import:MOUNTINGHOLE3.0THIN
- removed U$24: (no value), symbol eagleSchem-eagle-import:DISP_LCD_6LED_240X320_50PIN
- removed X1: (no value), symbol eagleSchem-eagle-import:MICROSD
- added C1, C2, C3, C4, C5: (no value), symbol schematicEagle-eagle-import:CAP_CERAMIC0805-NOOUTLINE
- added IC1: (no value), symbol schematicEagle-eagle-import:LP298XS
- added IC2, IC3: (no value), symbol schematicEagle-eagle-import:74245DW
- added IC4: (no value), symbol schematicEagle-eagle-import:AXP083-SAG
- added JP1, JP2: (no value), symbol schematicEagle-eagle-import:HEADER-1X20ROUND
- added Q1: (no value), symbol schematicEagle-eagle-import:-NPN-SOT23-BEC
- added R1, R10, R11, R12, R13, R14, R2, R3, R4, R5, R7, R8, R9: (no value), symbol schematicEagle-eagle-import:RESISTOR0805_NOOUTLINE
- added R6: (no value), symbol schematicEagle-eagle-import:R-US_R0805
- added SJ1, SJ2, SJ3, SJ4: (no value), symbol schematicEagle-eagle-import:SOLDERJUMPER
- added U$11, U$23, U$9: (no value), symbol schematicEagle-eagle-import:FIDUCIAL{dblquote}{dblquote}
- added U$15, U$16, U$17, U$7: (no value), symbol schematicEagle-eagle-import:MOUNTINGHOLE3.0THIN
- added U$24: (no value), symbol schematicEagle-eagle-import:DISP_LCD_6LED_240X320_50PIN
- added X1: (no value), symbol schematicEagle-eagle-import:MICROSD
Connections:
- net +5V: now also C2.1, C5.1, IC1.1 (VIN), IC1.3 (EN), JP1.2, JP2.2, R7.2
- net CARDDET: now also JP2.20, X1.CD2 (CARD_DETECT1)
- net GND: now also C1.2, C2.2, C3.2, C4.2, C5.2, IC1.2 (GND), IC2.19 (G), IC3.19 (G), IC4.1 (GND), JP1.1, JP2.1, Q1.E, R10.2, R11.2, R12.1, R8.1, R9.1, U$24.43 (GND@1), U$24.50 (GND@2), X1.6 (GND@3), X1.MT1 (GND@2), X1.MT2 (GND@1)
- net IM0: now also SJ1.1, U$24.6 (IM0)
- net IM1: now also SJ2.1, U$24.7 (IM1)
- net IM2: now also SJ3.2, U$24.8 (IM2)
- net IM3: now also SJ4.2, U$24.9 (IM3)
- net LCD_CS: now also IC3.15 (B4), U$24.38 (#CS)
- net LCD_CS_5V: now also IC3.5 (A4), JP1.3, JP2.7
- net LCD_DATA0: now also IC2.18 (B1), U$24.32 (DB0)
- net LCD_DATA0_5V: now also IC2.2 (A1), JP1.13
- net LCD_DATA1: now also IC2.17 (B2), U$24.31 (DB1)
- net LCD_DATA1_5V: now also IC2.3 (A2), JP1.14
- net LCD_DATA2: now also IC2.16 (B3), U$24.30 (DB2)
- net LCD_DATA2_5V: now also IC2.4 (A3), JP1.15
- net LCD_DATA3: now also IC2.15 (B4), U$24.29 (DB3)
- net LCD_DATA3_5V: now also IC2.5 (A4), JP1.16
- net LCD_DATA4: now also IC2.14 (B5), U$24.28 (DB4)
- net LCD_DATA4_5V: now also IC2.6 (A5), JP1.17
- net LCD_DATA5: now also IC2.13 (B6), U$24.27 (DB5)
- net LCD_DATA5_5V: now also IC2.7 (A6), JP1.18
- net LCD_DATA6: now also IC2.12 (B7), U$24.26 (DB6)
- net LCD_DATA6_5V: now also IC2.8 (A7), JP1.19
- net LCD_DATA7: now also IC2.11 (B8), U$24.25 (DB7)
- net LCD_DATA7_5V: now also IC2.9 (A8), JP1.20
- net LCD_LITE: now also JP1.8, JP2.10, R5.1, R7.1
- net LCD_RD: now also IC3.12 (B7), U$24.35 (#RD)
- net LCD_RD_5V: now also IC2.1 (DIR), IC3.8 (A7), JP1.6, R12.2
- net LCD_RS: now also IC3.14 (B5), U$24.37 (RS), X1.5 (SCLK)
- net LCD_RST: now also IC3.11 (B8), U$24.10 (RESET)
- net LCD_RST_5V: now also IC3.9 (A8), IC4.2 (/RESET), JP1.7, JP2.9, R6.1
- net LCD_RS_5V: now also IC3.6 (A5), JP1.4, JP2.4
- net LCD_WR: now also IC3.13 (B6), U$24.36 (#WR)
- net LCD_WR_5V: now also IC3.7 (A6), JP1.5, JP2.8
- net LCD_X+: now also JP1.9, JP2.12, U$24.46 (XL)
- net LCD_X-: now also JP1.11, JP2.14, U$24.44 (XR)
- net LCD_Y+: now also JP1.10, JP2.11, U$24.47 (YU)
- net LCD_Y-: now also JP1.12, JP2.13, U$24.45 (YD)
- net MISO: now also JP2.5, U$24.33 (SDO), X1.7 (DATA_OUT)
- net MOSI_3V: now also IC3.16 (B3), U$24.34 (SDI), X1.3 (DATA_IN)
- net MOSI_5V: now also IC3.4 (A3), JP2.6
- net SD_CS_3V: now also IC3.17 (B2), X1.2 (CS)
- net SD_CS_5V: now also IC3.3 (A2), JP2.19
- net VCC: now also C1.1, C3.1, C4.1, IC1.5 (VOUT), IC3.1 (DIR), IC4.3 (VCC), JP2.3, R1.1, R13.1, R14.1, R2.1, R3.1, R4.1, R6.2, SJ1.2, SJ2.2, SJ3.1, SJ4.1, U$24.40 (IOVCC@1), U$24.41 (IOVCC@2), U$24.42 (VCI), X1.4 (SD_VDD)
- new net: Q1.B, R5.2
- new net: Q1.C, U$24.1 (LEDK)
- new net: JP2.16, R11.1
- new net: JP2.15, R10.1
- new net: JP2.17, R9.2
- new net: JP2.18, R8.2
- new net: R2.2, U$24.4 (LEDA@3)
- new net: R13.2, U$24.2 (LEDA@1)
- new net: R1.2, U$24.3 (LEDA@2)
- new net: R4.2, U$24.48 (LEDA@5)
- new net: R14.2, U$24.49 (LEDA@6)
- new net: R3.2, U$24.5 (LEDA@4)

Commit message: Quickly Adding Everything
Parts:
- removed C1, C2, C3, C4, C5: (no value), symbol schematicEagle-eagle-import:CAP_CERAMIC0805-NOOUTLINE
- removed IC1: (no value), symbol schematicEagle-eagle-import:LP298XS
- removed IC2, IC3: (no value), symbol schematicEagle-eagle-import:74245DW
- removed IC4: (no value), symbol schematicEagle-eagle-import:AXP083-SAG
- removed JP1, JP2: (no value), symbol schematicEagle-eagle-import:HEADER-1X20ROUND
- removed Q1: (no value), symbol schematicEagle-eagle-import:-NPN-SOT23-BEC
- removed R1, R10, R11, R12, R13, R14, R2, R3, R4, R5, R7, R8, R9: (no value), symbol schematicEagle-eagle-import:RESISTOR0805_NOOUTLINE
- removed R6: (no value), symbol schematicEagle-eagle-import:R-US_R0805
- removed SJ1, SJ2, SJ3, SJ4: (no value), symbol schematicEagle-eagle-import:SOLDERJUMPER
- removed U$11, U$23, U$9: (no value), symbol schematicEagle-eagle-import:FIDUCIAL{dblquote}{dblquote}
- removed U$15, U$16, U$17, U$7: (no value), symbol schematicEagle-eagle-import:MOUNTINGHOLE3.0THIN
- removed U$24: (no value), symbol schematicEagle-eagle-import:DISP_LCD_6LED_240X320_50PIN
- removed X1: (no value), symbol schematicEagle-eagle-import:MICROSD
- added C1, C2, C3, C4, C5: (no value), symbol eagleSchem-eagle-import:CAP_CERAMIC0805-NOOUTLINE
- added IC1: (no value), symbol eagleSchem-eagle-import:LP298XS
- added IC2, IC3: (no value), symbol eagleSchem-eagle-import:74245DW
- added IC4: (no value), symbol eagleSchem-eagle-import:AXP083-SAG
- added JP1, JP2: (no value), symbol eagleSchem-eagle-import:HEADER-1X20ROUND
- added Q1: (no value), symbol eagleSchem-eagle-import:-NPN-SOT23-BEC
- added R1, R10, R11, R12, R13, R14, R2, R3, R4, R5, R7, R8, R9: (no value), symbol eagleSchem-eagle-import:RESISTOR0805_NOOUTLINE
- added R6: (no value), symbol eagleSchem-eagle-import:R-US_R0805
- added SJ1, SJ2, SJ3, SJ4: (no value), symbol eagleSchem-eagle-import:SOLDERJUMPER
- added U$11, U$23, U$9: (no value), symbol eagleSchem-eagle-import:FIDUCIAL{dblquote}{dblquote}
- added U$15, U$16, U$17, U$7: (no value), symbol eagleSchem-eagle-import:MOUNTINGHOLE3.0THIN
- added U$24: (no value), symbol eagleSchem-eagle-import:DISP_LCD_6LED_240X320_50PIN
- added X1: (no value), symbol eagleSchem-eagle-import:MICROSD
Connections:
- net +5V: now also C2.1, C5.1, IC1.1 (VIN), IC1.3 (EN), JP1.2, JP2.2, R7.2
- net CARDDET: now also JP2.20, X1.CD2 (CARD_DETECT1)
- net GND: now also C1.2, C2.2, C3.2, C4.2, C5.2, IC1.2 (GND), IC2.19 (G), IC3.19 (G), IC4.1 (GND), JP1.1, JP2.1, Q1.E, R10.2, R11.2, R12.1, R8.1, R9.1, U$24.43 (GND@1), U$24.50 (GND@2), X1.6 (GND@3), X1.MT1 (GND@2), X1.MT2 (GND@1)
- net IM0: now also SJ1.1, U$24.6 (IM0)
- net IM1: now also SJ2.1, U$24.7 (IM1)
- net IM2: now also SJ3.2, U$24.8 (IM2)
- net IM3: now also SJ4.2, U$24.9 (IM3)
- net LCD_CS: now also IC3.15 (B4), U$24.38 (#CS)
- net LCD_CS_5V: now also IC3.5 (A4), JP1.3, JP2.7
- net LCD_DATA0: now also IC2.18 (B1), U$24.32 (DB0)
- net LCD_DATA0_5V: now also IC2.2 (A1), JP1.13
- net LCD_DATA1: now also IC2.17 (B2), U$24.31 (DB1)
- net LCD_DATA1_5V: now also IC2.3 (A2), JP1.14
- net LCD_DATA2: now also IC2.16 (B3), U$24.30 (DB2)
- net LCD_DATA2_5V: now also IC2.4 (A3), JP1.15
- net LCD_DATA3: now also IC2.15 (B4), U$24.29 (DB3)
- net LCD_DATA3_5V: now also IC2.5 (A4), JP1.16
- net LCD_DATA4: now also IC2.14 (B5), U$24.28 (DB4)
- net LCD_DATA4_5V: now also IC2.6 (A5), JP1.17
- net LCD_DATA5: now also IC2.13 (B6), U$24.27 (DB5)
- net LCD_DATA5_5V: now also IC2.7 (A6), JP1.18
- net LCD_DATA6: now also IC2.12 (B7), U$24.26 (DB6)
- net LCD_DATA6_5V: now also IC2.8 (A7), JP1.19
- net LCD_DATA7: now also IC2.11 (B8), U$24.25 (DB7)
- net LCD_DATA7_5V: now also IC2.9 (A8), JP1.20
- net LCD_LITE: now also JP1.8, JP2.10, R5.1, R7.1
- net LCD_RD: now also IC3.12 (B7), U$24.35 (#RD)
- net LCD_RD_5V: now also IC2.1 (DIR), IC3.8 (A7), JP1.6, R12.2
- net LCD_RS: now also IC3.14 (B5), U$24.37 (RS), X1.5 (SCLK)
- net LCD_RST: now also IC3.11 (B8), U$24.10 (RESET)
- net LCD_RST_5V: now also IC3.9 (A8), IC4.2 (/RESET), JP1.7, JP2.9, R6.1
- net LCD_RS_5V: now also IC3.6 (A5), JP1.4, JP2.4
- net LCD_WR: now also IC3.13 (B6), U$24.36 (#WR)
- net LCD_WR_5V: now also IC3.7 (A6), JP1.5, JP2.8
- net LCD_X+: now also JP1.9, JP2.12, U$24.46 (XL)
- net LCD_X-: now also JP1.11, JP2.14, U$24.44 (XR)
- net LCD_Y+: now also JP1.10, JP2.11, U$24.47 (YU)
- net LCD_Y-: now also JP1.12, JP2.13, U$24.45 (YD)
- net MISO: now also JP2.5, U$24.33 (SDO), X1.7 (DATA_OUT)
- net MOSI_3V: now also IC3.16 (B3), U$24.34 (SDI), X1.3 (DATA_IN)
- net MOSI_5V: now also IC3.4 (A3), JP2.6
- net SD_CS_3V: now also IC3.17 (B2), X1.2 (CS)
- net SD_CS_5V: now also IC3.3 (A2), JP2.19
- net VCC: now also C1.1, C3.1, C4.1, IC1.5 (VOUT), IC3.1 (DIR), IC4.3 (VCC), JP2.3, R1.1, R13.1, R14.1, R2.1, R3.1, R4.1, R6.2, SJ1.2, SJ2.2, SJ3.1, SJ4.1, U$24.40 (IOVCC@1), U$24.41 (IOVCC@2), U$24.42 (VCI), X1.4 (SD_VDD)
- new net: Q1.B, R5.2
- new net: Q1.C, U$24.1 (LEDK)
- new net: R13.2, U$24.2 (LEDA@1)
- new net: R2.2, U$24.4 (LEDA@3)
- new net: R3.2, U$24.5 (LEDA@4)
- new net: JP2.18, R8.2
- new net: JP2.15, R10.1
- new net: JP2.16, R11.1
- new net: JP2.17, R9.2
- new net: R1.2, U$24.3 (LEDA@2)
- new net: R4.2, U$24.48 (LEDA@5)
- new net: R14.2, U$24.49 (LEDA@6)
