File: PROJ/ADAF/1778/STAN/01/src/kicadBoard.kicad_sch (KiCad schematic)
At the start: 17 parts

Commit message: Quickly Adding Everything
Parts:
- removed C1, C2, C3, C4: (no value), symbol eagleSchem-eagle-import:CAP_CERAMIC0805-NOOUTLINE
- removed D1: (no value), symbol eagleSchem-eagle-import:SHUNT-VREF
- removed FB1: (no value), symbol eagleSchem-eagle-import:FERRITE0805
- removed FID1, FID2: (no value), symbol eagleSchem-eagle-import:FIDUCIAL{dblquote}{dblquote}
- removed JP1: (no value), symbol eagleSchem-eagle-import:HEADER-1X4ROUND
- removed R1, R2, R3, R4: (no value), symbol eagleSchem-eagle-import:RESISTOR0805_NOOUTLINE
- removed U$11, U$12: (no value), symbol eagleSchem-eagle-import:MOUNTINGHOLE2.5
- removed U1: (no value), symbol eagleSchem-eagle-import:AD849X
- removed X1: (no value), symbol eagleSchem-eagle-import:TERMBLOCK_1X2
- added C1, C2, C3, C4: (no value), symbol schematicEagle-eagle-import:CAP_CERAMIC0805-NOOUTLINE
- added D1: (no value), symbol schematicEagle-eagle-import:SHUNT-VREF
- added FB1: (no value), symbol schematicEagle-eagle-import:FERRITE0805
- added FID1, FID2: (no value), symbol schematicEagle-eagle-import:FIDUCIAL{dblquote}{dblquote}
- added JP1: (no value), symbol schematicEagle-eagle-import:HEADER-1X4ROUND
- added R1, R2, R3, R4: (no value), symbol schematicEagle-eagle-import:RESISTOR0805_NOOUTLINE
- added U$11, U$12: (no value), symbol schematicEagle-eagle-import:MOUNTINGHOLE2.5
- added U1: (no value), symbol schematicEagle-eagle-import:AD849X
- added X1: (no value), symbol schematicEagle-eagle-import:TERMBLOCK_1X2
Connections:
- net GND: now also C1.1, C2.2, C4.1, D1.3 (A), JP1.2, JP1.4, R3.1, U1.3 (VS-)
- net VCC: now also C1.2, FB1.1 (P$1), R4.1, U1.7 (VS+)
- net VOUT: now also JP1.3, U1.5 (SENSE), U1.6 (OUT)
- new net: FB1.2 (P$2), JP1.1
- new net: C2.1, C3.2, R2.2, U1.1 (IN-)
- new net: D1.1 (VREF), D1.2 (C), R4.2, U1.2 (REF)
- new net: C3.1, C4.2, R1.2, U1.8 (IN+)
- new net: R1.1, X1.2
- new net: R2.1, R3.2, X1.1

Commit message: Quickly Adding Everything
Parts:
- removed C1, C2, C3, C4: (no value), symbol schematicEagle-eagle-import:CAP_CERAMIC0805-NOOUTLINE
- removed D1: (no value), symbol schematicEagle-eagle-import:SHUNT-VREF
- removed FB1: (no value), symbol schematicEagle-eagle-import:FERRITE0805
- removed FID1, FID2: (no value), symbol schematicEagle-eagle-import:FIDUCIAL{dblquote}{dblquote}
- removed JP1: (no value), symbol schematicEagle-eagle-import:HEADER-1X4ROUND
- removed R1, R2, R3, R4: (no value), symbol schematicEagle-eagle-import:RESISTOR0805_NOOUTLINE
- removed U$11, U$12: (no value), symbol schematicEagle-eagle-import:MOUNTINGHOLE2.5
- removed U1: (no value), symbol schematicEagle-eagle-import:AD849X
- removed X1: (no value), symbol schematicEagle-eagle-import:TERMBLOCK_1X2
- added C1, C2, C3, C4: (no value), symbol eagleSchem-eagle-import:CAP_CERAMIC0805-NOOUTLINE
- added D1: (no value), symbol eagleSchem-eagle-import:SHUNT-VREF
- added FB1: (no value), symbol eagleSchem-eagle-import:FERRITE0805
- added FID1, FID2: (no value), symbol eagleSchem-eagle-import:FIDUCIAL{dblquote}{dblquote}
- added JP1: (no value), symbol eagleSchem-eagle-import:HEADER-1X4ROUND
- added R1, R2, R3, R4: (no value), symbol eagleSchem-eagle-import:RESISTOR0805_NOOUTLINE
- added U$11, U$12: (no value), symbol eagleSchem-eagle-import:MOUNTINGHOLE2.5
- added U1: (no value), symbol eagleSchem-eagle-import:AD849X
- added X1: (no value), symbol eagleSchem-eagle-import:TERMBLOCK_1X2
Connections:
- net GND: now also C1.1, C2.2, C4.1, D1.3 (A), JP1.2, JP1.4, R3.1, U1.3 (VS-)
- net VCC: now also C1.2, FB1.1 (P$1), R4.1, U1.7 (VS+)
- net VOUT: now also JP1.3, U1.5 (SENSE), U1.6 (OUT)
- new net: C2.1, C3.2, R2.2, U1.1 (IN-)
- new net: D1.1 (VREF), D1.2 (C), R4.2, U1.2 (REF)
- new net: C3.1, C4.2, R1.2, U1.8 (IN+)
- new net: FB1.2 (P$2), JP1.1
- new net: R2.1, R3.2, X1.1
- new net: R1.1, X1.2
