File: PROJ/ADAF/2107/STAN/01/src/kicadBoard.kicad_sch (KiCad schematic)
At the start: 28 parts

Commit message: Quickly Adding Everything
Parts:
- removed C1, C10, C2, C3, C4, C5, C6, C7, C8, C9: (no value), symbol eagleSchem-eagle-import:CAP_CERAMIC0805-NOOUTLINE
- removed D1: (no value), symbol eagleSchem-eagle-import:LED0805_NOOUTLINE
- removed FID1, FID2, FID3: (no value), symbol eagleSchem-eagle-import:FIDUCIAL{dblquote}{dblquote}
- removed R1, R2, R3, R5: (no value), symbol eagleSchem-eagle-import:RESISTOR0805_NOOUTLINE
- removed R4: (no value), symbol eagleSchem-eagle-import:RESISTOR_0805MP
- removed SW1: (no value), symbol eagleSchem-eagle-import:SWITCH_DPDTEG1390
- removed U$10, U$7, U$8, U$9: (no value), symbol eagleSchem-eagle-import:MOUNTINGHOLE2.5_THICK
- removed U1: (no value), symbol eagleSchem-eagle-import:ADUM4160
- removed U2: (no value), symbol eagleSchem-eagle-import:ADUM5000
- removed X2: (no value), symbol eagleSchem-eagle-import:USB_TYPEAPTHFML
- removed X3: (no value), symbol eagleSchem-eagle-import:USBMINIBLARGE
- added C1, C10, C2, C3, C4, C5, C6, C7, C8, C9: (no value), symbol schematicEagle-eagle-import:CAP_CERAMIC0805-NOOUTLINE
- added D1: (no value), symbol schematicEagle-eagle-import:LED0805_NOOUTLINE
- added FID1, FID2, FID3: (no value), symbol schematicEagle-eagle-import:FIDUCIAL{dblquote}{dblquote}
- added R1, R2, R3, R5: (no value), symbol schematicEagle-eagle-import:RESISTOR0805_NOOUTLINE
- added R4: (no value), symbol schematicEagle-eagle-import:RESISTOR_0805MP
- added SW1: (no value), symbol schematicEagle-eagle-import:SWITCH_DPDTEG1390
- added U$10, U$7, U$8, U$9: (no value), symbol schematicEagle-eagle-import:MOUNTINGHOLE2.5_THICK
- added U1: (no value), symbol schematicEagle-eagle-import:ADUM4160
- added U2: (no value), symbol schematicEagle-eagle-import:ADUM5000
- added X2: (no value), symbol schematicEagle-eagle-import:USB_TYPEAPTHFML
- added X3: (no value), symbol schematicEagle-eagle-import:USBMINIBLARGE
Connections:
- net AGND: now also C3.1, C4.1, C5.2, C6.2, C7.1, R5.2, SW1.O2, U1.15 (GND2@1), U1.9 (GND2@2), U2.15 (GND2@1), U2.9 (GND2@2), X2.GND
- net AVCC: now also C3.2, C5.1, C6.1, C7.2, D1.A, U1.16 (VBUS2), U2.10 (VISO@2), U2.13 (VSEL), U2.16 (VISO@1), X2.VBUS
- net GND: now also C1.2, C10.1, C2.2, C8.2, C9.2, SW1.O1, U1.2 (GND1@1), U1.8 (GND1@2), U2.2 (GND1@1), U2.8 (GND1@2), X3.GND, X3.GND1 (GND), X3.GND2 (GND), X3.GND3 (GND), X3.GND4 (GND)
- net SPD: now also SW1.P2, U1.13 (SPD)
- net SPU: now also SW1.P1, U1.5 (SPU)
- net VCC: now also C1.1, C10.2, C8.1, C9.1, U1.1 (VBUS1), U2.1 (VDD@1), U2.6 (RCSEL), U2.7 (VDD@2), X3.VBUS
- net VDD1: now also C2.1, SW1.S1, U1.3 (VDD1), U1.4 (PDEN)
- net VDD2: now also C4.2, SW1.S2, U1.12 (PIN), U1.14 (VDD2)
- new net: R4.1, U1.10 (DD+)
- new net: R3.1, U1.11 (DD-)
- new net: R1.2, U1.6 (UD-)
- new net: R2.2, U1.7 (UD+)
- new net: R4.2, X2.D+
- new net: D1.C, R5.1
- new net: R3.2, X2.D-
- new net: R2.1, X3.D+
- new net: R1.1, X3.D-

Commit message: Quickly Adding Everything
Parts:
- removed C1, C10, C2, C3, C4, C5, C6, C7, C8, C9: (no value), symbol schematicEagle-eagle-import:CAP_CERAMIC0805-NOOUTLINE
- removed D1: (no value), symbol schematicEagle-eagle-import:LED0805_NOOUTLINE
- removed FID1, FID2, FID3: (no value), symbol schematicEagle-eagle-import:FIDUCIAL{dblquote}{dblquote}
- removed R1, R2, R3, R5: (no value), symbol schematicEagle-eagle-import:RESISTOR0805_NOOUTLINE
- removed R4: (no value), symbol schematicEagle-eagle-import:RESISTOR_0805MP
- removed SW1: (no value), symbol schematicEagle-eagle-import:SWITCH_DPDTEG1390
- removed U$10, U$7, U$8, U$9: (no value), symbol schematicEagle-eagle-import:MOUNTINGHOLE2.5_THICK
- removed U1: (no value), symbol schematicEagle-eagle-import:ADUM4160
- removed U2: (no value), symbol schematicEagle-eagle-import:ADUM5000
- removed X2: (no value), symbol schematicEagle-eagle-import:USB_TYPEAPTHFML
- removed X3: (no value), symbol schematicEagle-eagle-import:USBMINIBLARGE
- added C1, C10, C2, C3, C4, C5, C6, C7, C8, C9: (no value), symbol eagleSchem-eagle-import:CAP_CERAMIC0805-NOOUTLINE
- added D1: (no value), symbol eagleSchem-eagle-import:LED0805_NOOUTLINE
- added FID1, FID2, FID3: (no value), symbol eagleSchem-eagle-import:FIDUCIAL{dblquote}{dblquote}
- added R1, R2, R3, R5: (no value), symbol eagleSchem-eagle-import:RESISTOR0805_NOOUTLINE
- added R4: (no value), symbol eagleSchem-eagle-import:RESISTOR_0805MP
- added SW1: (no value), symbol eagleSchem-eagle-import:SWITCH_DPDTEG1390
- added U$10, U$7, U$8, U$9: (no value), symbol eagleSchem-eagle-import:MOUNTINGHOLE2.5_THICK
- added U1: (no value), symbol eagleSchem-eagle-import:ADUM4160
- added U2: (no value), symbol eagleSchem-eagle-import:ADUM5000
- added X2: (no value), symbol eagleSchem-eagle-import:USB_TYPEAPTHFML
- added X3: (no value), symbol eagleSchem-eagle-import:USBMINIBLARGE
Connections:
- net AGND: now also C3.1, C4.1, C5.2, C6.2, C7.1, R5.2, SW1.O2, U1.15 (GND2@1), U1.9 (GND2@2), U2.15 (GND2@1), U2.9 (GND2@2), X2.GND
- net AVCC: now also C3.2, C5.1, C6.1, C7.2, D1.A, U1.16 (VBUS2), U2.10 (VISO@2), U2.13 (VSEL), U2.16 (VISO@1), X2.VBUS
- net GND: now also C1.2, C10.1, C2.2, C8.2, C9.2, SW1.O1, U1.2 (GND1@1), U1.8 (GND1@2), U2.2 (GND1@1), U2.8 (GND1@2), X3.GND, X3.GND1 (GND), X3.GND2 (GND), X3.GND3 (GND), X3.GND4 (GND)
- net SPD: now also SW1.P2, U1.13 (SPD)
- net SPU: now also SW1.P1, U1.5 (SPU)
- net VCC: now also C1.1, C10.2, C8.1, C9.1, U1.1 (VBUS1), U2.1 (VDD@1), U2.6 (RCSEL), U2.7 (VDD@2), X3.VBUS
- net VDD1: now also C2.1, SW1.S1, U1.3 (VDD1), U1.4 (PDEN)
- net VDD2: now also C4.2, SW1.S2, U1.12 (PIN), U1.14 (VDD2)
- new net: R3.1, U1.11 (DD-)
- new net: R3.2, X2.D-
- new net: R2.1, X3.D+
- new net: R1.1, X3.D-
- new net: R1.2, U1.6 (UD-)
- new net: D1.C, R5.1
- new net: R4.1, U1.10 (DD+)
- new net: R4.2, X2.D+
- new net: R2.2, U1.7 (UD+)
