File: PROJ/ADAF/2130/STAN/01/src/kicadBoard.kicad_sch (KiCad schematic)
At the start: 18 parts

Commit message: Quickly Adding Everything
Parts:
- removed C1, C2, C3, C4, C5: (no value), symbol eagleSchem-eagle-import:CAP_CERAMIC0805-NOOUTLINE
- removed FB1, FB2: (no value), symbol eagleSchem-eagle-import:FERRITE_0805
- removed FID1, FID2: (no value), symbol eagleSchem-eagle-import:FIDUCIAL{dblquote}{dblquote}
- removed JP1: (no value), symbol eagleSchem-eagle-import:HEADER-1X570MIL
- removed R1, R2, R3: (no value), symbol eagleSchem-eagle-import:RESISTOR0805_NOOUTLINE
- removed U$10, U$11: (no value), symbol eagleSchem-eagle-import:MOUNTINGHOLE2.0
- removed U1: (no value), symbol eagleSchem-eagle-import:AUDIOAMP_PAM8302A
- removed VR1: (no value), symbol eagleSchem-eagle-import:TRIMPOT3303W/X
- removed X1: (no value), symbol eagleSchem-eagle-import:TERMBLOCK_1X2
- added C1, C2, C3, C4, C5: (no value), symbol schematicEagle-eagle-import:CAP_CERAMIC0805-NOOUTLINE
- added FB1, FB2: (no value), symbol schematicEagle-eagle-import:FERRITE_0805
- added FID1, FID2: (no value), symbol schematicEagle-eagle-import:FIDUCIAL{dblquote}{dblquote}
- added JP1: (no value), symbol schematicEagle-eagle-import:HEADER-1X570MIL
- added R1, R2, R3: (no value), symbol schematicEagle-eagle-import:RESISTOR0805_NOOUTLINE
- added U$10, U$11: (no value), symbol schematicEagle-eagle-import:MOUNTINGHOLE2.0
- added U1: (no value), symbol schematicEagle-eagle-import:AUDIOAMP_PAM8302A
- added VR1: (no value), symbol schematicEagle-eagle-import:TRIMPOT3303W/X
- added X1: (no value), symbol schematicEagle-eagle-import:TERMBLOCK_1X2
Connections:
- net AIN+: now also JP1.5, VR1.3 (E)
- net AIN-: now also C2.2, JP1.4, VR1.1 (A)
- net GND: now also C3.2, C4.2, C5.2, JP1.1, U1.7 (GND)
- net SD: now also JP1.3, R3.2, U1.1 (/SD)
- net VCC: now also C3.1, JP1.2, R3.1, U1.6 (VDD)
- net VO+: now also C5.1, FB1.2 (P$2), X1.1
- net VO-: now also C4.1, FB2.2 (P$2), X1.2
- new net: R1.2, U1.3 (IN_P)
- new net: R2.2, U1.4 (IN_N)
- new net: FB1.1 (P$1), U1.5 (VO_P)
- new net: FB2.1 (P$1), U1.8 (VO_N)
- new net: C1.1, R1.1
- new net: C2.1, R2.1
- new net: C1.2, VR1.2 (S)

Commit message: Quickly Adding Everything
Parts:
- removed C1, C2, C3, C4, C5: (no value), symbol schematicEagle-eagle-import:CAP_CERAMIC0805-NOOUTLINE
- removed FB1, FB2: (no value), symbol schematicEagle-eagle-import:FERRITE_0805
- removed FID1, FID2: (no value), symbol schematicEagle-eagle-import:FIDUCIAL{dblquote}{dblquote}
- removed JP1: (no value), symbol schematicEagle-eagle-import:HEADER-1X570MIL
- removed R1, R2, R3: (no value), symbol schematicEagle-eagle-import:RESISTOR0805_NOOUTLINE
- removed U$10, U$11: (no value), symbol schematicEagle-eagle-import:MOUNTINGHOLE2.0
- removed U1: (no value), symbol schematicEagle-eagle-import:AUDIOAMP_PAM8302A
- removed VR1: (no value), symbol schematicEagle-eagle-import:TRIMPOT3303W/X
- removed X1: (no value), symbol schematicEagle-eagle-import:TERMBLOCK_1X2
- added C1, C2, C3, C4, C5: (no value), symbol eagleSchem-eagle-import:CAP_CERAMIC0805-NOOUTLINE
- added FB1, FB2: (no value), symbol eagleSchem-eagle-import:FERRITE_0805
- added FID1, FID2: (no value), symbol eagleSchem-eagle-import:FIDUCIAL{dblquote}{dblquote}
- added JP1: (no value), symbol eagleSchem-eagle-import:HEADER-1X570MIL
- added R1, R2, R3: (no value), symbol eagleSchem-eagle-import:RESISTOR0805_NOOUTLINE
- added U$10, U$11: (no value), symbol eagleSchem-eagle-import:MOUNTINGHOLE2.0
- added U1: (no value), symbol eagleSchem-eagle-import:AUDIOAMP_PAM8302A
- added VR1: (no value), symbol eagleSchem-eagle-import:TRIMPOT3303W/X
- added X1: (no value), symbol eagleSchem-eagle-import:TERMBLOCK_1X2
Connections:
- net AIN+: now also JP1.5, VR1.3 (E)
- net AIN-: now also C2.2, JP1.4, VR1.1 (A)
- net GND: now also C3.2, C4.2, C5.2, JP1.1, U1.7 (GND)
- net SD: now also JP1.3, R3.2, U1.1 (/SD)
- net VCC: now also C3.1, JP1.2, R3.1, U1.6 (VDD)
- net VO+: now also C5.1, FB1.2 (P$2), X1.1
- net VO-: now also C4.1, FB2.2 (P$2), X1.2
- new net: C2.1, R2.1
- new net: R2.2, U1.4 (IN_N)
- new net: C1.1, R1.1
- new net: C1.2, VR1.2 (S)
- new net: FB1.1 (P$1), U1.5 (VO_P)
- new net: R1.2, U1.3 (IN_P)
- new net: FB2.1 (P$1), U1.8 (VO_N)
